Commit message: fix(baracuda): tuned weights manually

File: duatic_dynaarm_description/urdf/common/baracuda12/dynaarm_parameters.urdf.xacro (robot description, xacro)
@@ -156,5 +156,5 @@
     <inertial>
       <!-- Original - <mass value="1.72040464" /> -->
-      <mass value="2.12040464" />
+      <mass value="1.22040464" />
       <origin xyz="0.20391301 -0.00000528 -0.00015224"
         rpy="0 0 0" />
@@ -188,5 +188,5 @@
     <inertial>
       <!-- The mass here is 100g more than the value in CAD, but through testing we found out that freedrive works better with the increased value (09.12.25 Antonis & Marc)-->
-      <mass value="1.337246" />
+      <mass value="2.037246" />
       <origin xyz="-0.001568 0.000046 0.292163" rpy="0 0 0" />
       <inertia ixx="0.033872" iyy="0.033868"
@@ -199,5 +199,5 @@
     <inertial>
       <!-- <mass value="0.75007482" />  original value but doesn't work well - Needs to include the cables inside the forearm tube?-->
-      <mass value="1.15007482" />
+      <mass value="0.95007482" />
       <origin xyz="0.07972553 -0.00005038 0.02334747" rpy="0 0 0" />
       <inertia ixx="0.00065953" iyy="0.00088282"
@@ -219,5 +219,5 @@
   <xacro:property name="link06_inertial">
     <inertial>
-      <mass value="0.0478406" />
+      <mass value="0.0978406" />
       <origin xyz="0.00045711 0.00000557 0.00344945" rpy="0 0 0" />
       <inertia ixx="0.00001366" iyy="0.00001419"
