Commit message: fix: remove added weight on forearm

File: duatic_dynaarm_description/urdf/common/baracuda12/dynaarm_parameters.urdf.xacro (robot description, xacro)
@@ -169,6 +169,5 @@
   <xacro:property name="link04_inertial">
     <inertial>
-      <!-- The mass here is 100g more than the value in CAD, but through testing we found out that freedrive works better with the increased value (09.12.25 Antonis & Marc)-->
-      <mass value="1.337246" />
+      <mass value="1.237246" />
       <origin xyz="-0.001568 0.000046 0.292163" rpy="0 0 0" />
       <inertia ixx="0.033872" iyy="0.033868"

File: duatic_dynaarm_description/urdf/common/corydoras12/dynaarm_parameters.urdf.xacro (robot description, xacro)
@@ -169,6 +169,5 @@
   <xacro:property name="link04_inertial">
     <inertial>
-      <!-- The mass here is 100g more than the value in CAD, but through testing we found out that freedrive works better with the increased value (09.12.25 Antonis & Marc)-->
-      <mass value="1.337246" />
+      <mass value="1.237246" />
       <origin xyz="-0.001568 0.000046 0.292163" rpy="0 0 0" />
       <inertia ixx="0.033872" iyy="0.033868"

Commit message: feat(): removing the option to enable/disable covers (#16)

File: duatic_dynaarm_description/urdf/common/baracuda12/dynaarm_parameters.urdf.xacro (robot description, xacro)
@@ -40,29 +40,11 @@
   <xacro:property name="end_effector" value="${tf_prefix}flange" />
   <!-- Meshes -->
-  <xacro:if value="${covers}">
-    <xacro:property name="base_mesh" value="base_mesh.dae" />
-    <xacro:property name="link01_mesh" value="shoulder_mesh.dae" />
-    <xacro:property name="link02_mesh" value="upperarm_mesh.dae" />
-    <xacro:property name="link03_mesh" value="elbow_mesh.dae" />
-    <xacro:property name="link04_mesh" value="forearm_mesh.dae" />
-    <xacro:property name="link05_mesh" value="wrist1_mesh.dae" />
-    <xacro:property name="link06_mesh" value="wrist2_mesh.dae" />
-    <xacro:property name="base_cover_mesh" value="base_mesh.dae" />
-    <xacro:property name="link01_cover_mesh" value="shoulder_mesh.dae" />
-    <xacro:property name="link02_cover_mesh" value="upperarm_mesh.dae" />
-    <xacro:property name="link03_cover_mesh" value="elbow_mesh.dae" />
-    <xacro:property name="link04_cover_mesh" value="forearm_mesh.dae" />
-    <xacro:property name="link05_cover_mesh" value="wrist1_mesh.dae" />
-    <xacro:property name="link06_cover_mesh" value="wrist2_mesh.dae" />
-  </xacro:if>
-  <xacro:unless value="${covers}">
-    <xacro:property name="base_mesh" value="base_mesh.dae" />
-    <xacro:property name="link01_mesh" value="shoulder_mesh.dae" />
-    <xacro:property name="link02_mesh" value="upperarm_mesh.dae" />
-    <xacro:property name="link03_mesh" value="elbow_mesh.dae" />
-    <xacro:property name="link04_mesh" value="forearm_mesh.dae" />
-    <xacro:property name="link05_mesh" value="wrist1_mesh.dae" />
-    <xacro:property name="link06_mesh" value="wrist2_mesh.dae" />
-  </xacro:unless>
+  <xacro:property name="base_mesh" value="base_mesh.dae" />
+  <xacro:property name="link01_mesh" value="shoulder_mesh.dae" />
+  <xacro:property name="link02_mesh" value="upperarm_mesh.dae" />
+  <xacro:property name="link03_mesh" value="elbow_mesh.dae" />
+  <xacro:property name="link04_mesh" value="forearm_mesh.dae" />
+  <xacro:property name="link05_mesh" value="wrist1_mesh.dae" />
+  <xacro:property name="link06_mesh" value="wrist2_mesh.dae" />
   <!-- Joint properties -->
   <xacro:property name="joint_base_name" value="${tf_prefix}joint_base" />
@@ -187,6 +169,5 @@
   <xacro:property name="link04_inertial">
     <inertial>
-      <!-- The mass here is 100g more than the value in CAD, but through testing we found out that freedrive works better with the increased value (09.12.25 Antonis & Marc)-->
-      <mass value="1.337246" />
+      <mass value="1.237246" />
       <origin xyz="-0.001568 0.000046 0.292163" rpy="0 0 0" />
       <inertia ixx="0.033872" iyy="0.033868"
@@ -224,53 +205,4 @@
         izz="0.00002702" ixy="0"
         ixz="0.00000008" iyz="0" />
-    </inertial>
-  </xacro:property>
-  <!-- Covers -->
-  <xacro:property name="base_cover_inertial">
-    <inertial>
-      <mass value="0.098" />
-      <origin xyz="${0.0*mm_to_m} ${0.0*mm_to_m} ${-60.7*mm_to_m}" rpy="0 0 0" />
-      <inertia ixx="${0.000349}" iyy="${0.000338}" izz="${0.000649}" ixy="${0.000000018}"
-        ixz="${-0.000000001}" iyz="${-0.000000002}" />
-    </inertial>
-  </xacro:property>
-  <xacro:property name="link01_cover_inertial">
-    <inertial>
-      <mass value="0.135" />
-      <origin xyz="${-0.039*mm_to_m} ${-0.015*mm_to_m} ${-31.709*mm_to_m}" rpy="0 0 0" />
-      <inertia ixx="${0.00068}" iyy="${0.000517}" izz="${0.000646}" ixy="${-0.000000318}"
-        ixz="${-0.000000206}" iyz="${-0.000000074}" />
-    </inertial>
-  </xacro:property>
-  <xacro:property name="link02_cover_inertial">
-    <inertial>
-      <mass value="0.743" />
-      <origin xyz="${167.97*mm_to_m} ${0.081*mm_to_m} ${0.0*mm_to_m}" rpy="0 0 0" />
-      <inertia ixx="${0.0054}" iyy="${0.025}" izz="${0.0293}" ixy="${-0.000004814}"
-        ixz="${-0.000000101}" iyz="${0.000000134}" />
-    </inertial>
-  </xacro:property>
-  <xacro:property name="link03_cover_inertial">
-    <inertial>
-      <mass value="0.383" />
-      <origin xyz="${37.807*mm_to_m} ${-101.52*mm_to_m} ${0.184*mm_to_m}" rpy="0 0 0" />
-      <inertia ixx="${0.00139}" iyy="${0.00176}" izz="${0.00225}" ixy="${-0.000150269}"
-        ixz="${0.000002221}" iyz="${-0.000003993}" />
-    </inertial>
-  </xacro:property>
-  <xacro:property name="link04_cover_inertial">
-    <inertial>
-      <mass value="0.158" />
-      <origin xyz="${-9.28*mm_to_m} ${-0.008*mm_to_m} ${377.34*mm_to_m}" rpy="0 0 0" />
-      <inertia ixx="${0.000594}" iyy="${0.000846}" izz="${0.000485}" ixy="${-0.000000100}"
-        ixz="${-0.000057116}" iyz="${0.000000128}" />
-    </inertial>
-  </xacro:property>
-  <xacro:property name="link05_cover_inertial">
-    <inertial>
-      <mass value="0.121" />
-      <origin xyz="${54.24*mm_to_m} ${-0.0012*mm_to_m} ${-0.0069*mm_to_m}" rpy="0 0 0" />
-      <inertia ixx="${0.0003}" iyy="${0.00049}" izz="${0.00053}" ixy="${-0.000000004}"
-        ixz="${0.0}" iyz="${-0.000000043}" />
     </inertial>
   </xacro:property>

File: duatic_dynaarm_description/urdf/common/corydoras12/dynaarm_parameters.urdf.xacro (robot description, xacro)
@@ -40,29 +40,11 @@
   <xacro:property name="end_effector" value="${tf_prefix}flange" />
   <!-- Meshes -->
-  <xacro:if value="${covers}">
-    <xacro:property name="base_mesh" value="base_mesh.dae" />
-    <xacro:property name="link01_mesh" value="shoulder_mesh.dae" />
-    <xacro:property name="link02_mesh" value="upperarm_mesh.dae" />
-    <xacro:property name="link03_mesh" value="elbow_mesh.dae" />
-    <xacro:property name="link04_mesh" value="forearm_mesh.dae" />
-    <xacro:property name="link05_mesh" value="wrist1_mesh.dae" />
-    <xacro:property name="link06_mesh" value="wrist2_mesh.dae" />
-    <xacro:property name="base_cover_mesh" value="base_mesh.dae" />
-    <xacro:property name="link01_cover_mesh" value="shoulder_mesh.dae" />
-    <xacro:property name="link02_cover_mesh" value="upperarm_mesh.dae" />
-    <xacro:property name="link03_cover_mesh" value="elbow_mesh.dae" />
-    <xacro:property name="link04_cover_mesh" value="forearm_mesh.dae" />
-    <xacro:property name="link05_cover_mesh" value="wrist1_mesh.dae" />
-    <xacro:property name="link06_cover_mesh" value="wrist2_mesh.dae" />
-  </xacro:if>
-  <xacro:unless value="${covers}">
-    <xacro:property name="base_mesh" value="base_mesh.dae" />
-    <xacro:property name="link01_mesh" value="shoulder_mesh.dae" />
-    <xacro:property name="link02_mesh" value="upperarm_mesh.dae" />
-    <xacro:property name="link03_mesh" value="elbow_mesh.dae" />
-    <xacro:property name="link04_mesh" value="forearm_mesh.dae" />
-    <xacro:property name="link05_mesh" value="wrist1_mesh.dae" />
-    <xacro:property name="link06_mesh" value="wrist2_mesh.dae" />
-  </xacro:unless>
+  <xacro:property name="base_mesh" value="base_mesh.dae" />
+  <xacro:property name="link01_mesh" value="shoulder_mesh.dae" />
+  <xacro:property name="link02_mesh" value="upperarm_mesh.dae" />
+  <xacro:property name="link03_mesh" value="elbow_mesh.dae" />
+  <xacro:property name="link04_mesh" value="forearm_mesh.dae" />
+  <xacro:property name="link05_mesh" value="wrist1_mesh.dae" />
+  <xacro:property name="link06_mesh" value="wrist2_mesh.dae" />
   <!-- Joint properties -->
   <xacro:property name="joint_base_name" value="${tf_prefix}joint_base" />
@@ -187,6 +169,5 @@
   <xacro:property name="link04_inertial">
     <inertial>
-      <!-- The mass here is 100g more than the value in CAD, but through testing we found out that freedrive works better with the increased value (09.12.25 Antonis & Marc)-->
-      <mass value="1.337246" />
+      <mass value="1.237246" />
       <origin xyz="-0.001568 0.000046 0.292163" rpy="0 0 0" />
       <inertia ixx="0.033872" iyy="0.033868"
@@ -224,53 +205,4 @@
         izz="0.00002702" ixy="0"
         ixz="0.00000008" iyz="0" />
-    </inertial>
-  </xacro:property>
-  <!-- Covers -->
-  <xacro:property name="base_cover_inertial">
-    <inertial>
-      <mass value="0.098" />
-      <origin xyz="${0.0*mm_to_m} ${0.0*mm_to_m} ${-60.7*mm_to_m}" rpy="0 0 0" />
-      <inertia ixx="${0.000349}" iyy="${0.000338}" izz="${0.000649}" ixy="${0.000000018}"
-        ixz="${-0.000000001}" iyz="${-0.000000002}" />
-    </inertial>
-  </xacro:property>
-  <xacro:property name="link01_cover_inertial">
-    <inertial>
-      <mass value="0.135" />
-      <origin xyz="${-0.039*mm_to_m} ${-0.015*mm_to_m} ${-31.709*mm_to_m}" rpy="0 0 0" />
-      <inertia ixx="${0.00068}" iyy="${0.000517}" izz="${0.000646}" ixy="${-0.000000318}"
-        ixz="${-0.000000206}" iyz="${-0.000000074}" />
-    </inertial>
-  </xacro:property>
-  <xacro:property name="link02_cover_inertial">
-    <inertial>
-      <mass value="0.743" />
-      <origin xyz="${167.97*mm_to_m} ${0.081*mm_to_m} ${0.0*mm_to_m}" rpy="0 0 0" />
-      <inertia ixx="${0.0054}" iyy="${0.025}" izz="${0.0293}" ixy="${-0.000004814}"
-        ixz="${-0.000000101}" iyz="${0.000000134}" />
-    </inertial>
-  </xacro:property>
-  <xacro:property name="link03_cover_inertial">
-    <inertial>
-      <mass value="0.383" />
-      <origin xyz="${37.807*mm_to_m} ${-101.52*mm_to_m} ${0.184*mm_to_m}" rpy="0 0 0" />
-      <inertia ixx="${0.00139}" iyy="${0.00176}" izz="${0.00225}" ixy="${-0.000150269}"
-        ixz="${0.000002221}" iyz="${-0.000003993}" />
-    </inertial>
-  </xacro:property>
-  <xacro:property name="link04_cover_inertial">
-    <inertial>
-      <mass value="0.158" />
-      <origin xyz="${-9.28*mm_to_m} ${-0.008*mm_to_m} ${377.34*mm_to_m}" rpy="0 0 0" />
-      <inertia ixx="${0.000594}" iyy="${0.000846}" izz="${0.000485}" ixy="${-0.000000100}"
-        ixz="${-0.000057116}" iyz="${0.000000128}" />
-    </inertial>
-  </xacro:property>
-  <xacro:property name="link05_cover_inertial">
-    <inertial>
-      <mass value="0.121" />
-      <origin xyz="${54.24*mm_to_m} ${-0.0012*mm_to_m} ${-0.0069*mm_to_m}" rpy="0 0 0" />
-      <inertia ixx="${0.0003}" iyy="${0.00049}" izz="${0.00053}" ixy="${-0.000000004}"
-        ixz="${0.0}" iyz="${-0.000000043}" />
     </inertial>
   </xacro:property>

Commit message: Added new meshes

File: duatic_dynaarm_description/urdf/common/baracuda12/dynaarm_parameters.urdf.xacro (robot description, xacro)
@@ -40,11 +40,11 @@
   <xacro:property name="end_effector" value="${tf_prefix}flange" />
   <!-- Meshes -->
-  <xacro:property name="base_mesh" value="base_mesh.dae" />
-  <xacro:property name="link01_mesh" value="shoulder_mesh.dae" />
-  <xacro:property name="link02_mesh" value="upperarm_mesh.dae" />
-  <xacro:property name="link03_mesh" value="elbow_mesh.dae" />
-  <xacro:property name="link04_mesh" value="forearm_mesh.dae" />
-  <xacro:property name="link05_mesh" value="wrist1_mesh.dae" />
-  <xacro:property name="link06_mesh" value="wrist2_mesh.dae" />
+  <xacro:property name="base_mesh" value="base_mesh.glb" />
+  <xacro:property name="link01_mesh" value="shoulder_mesh.glb" />
+  <xacro:property name="link02_mesh" value="upperarm_mesh.glb" />
+  <xacro:property name="link03_mesh" value="elbow_mesh.glb" />
+  <xacro:property name="link04_mesh" value="forearm_mesh.glb" />
+  <xacro:property name="link05_mesh" value="wrist1_mesh.glb" />
+  <xacro:property name="link06_mesh" value="wrist2_mesh.glb" />
   <!-- Joint properties -->
   <xacro:property name="joint_base_name" value="${tf_prefix}joint_base" />

File: duatic_dynaarm_description/urdf/common/corydoras12/dynaarm_parameters.urdf.xacro (robot description, xacro)
@@ -40,11 +40,11 @@
   <xacro:property name="end_effector" value="${tf_prefix}flange" />
   <!-- Meshes -->
-  <xacro:property name="base_mesh" value="base_mesh.dae" />
-  <xacro:property name="link01_mesh" value="shoulder_mesh.dae" />
-  <xacro:property name="link02_mesh" value="upperarm_mesh.dae" />
-  <xacro:property name="link03_mesh" value="elbow_mesh.dae" />
-  <xacro:property name="link04_mesh" value="forearm_mesh.dae" />
-  <xacro:property name="link05_mesh" value="wrist1_mesh.dae" />
-  <xacro:property name="link06_mesh" value="wrist2_mesh.dae" />
+  <xacro:property name="base_mesh" value="base_mesh.glb" />
+  <xacro:property name="link01_mesh" value="shoulder_mesh.glb" />
+  <xacro:property name="link02_mesh" value="upperarm_mesh.glb" />
+  <xacro:property name="link03_mesh" value="elbow_mesh.glb" />
+  <xacro:property name="link04_mesh" value="forearm_mesh.glb" />
+  <xacro:property name="link05_mesh" value="wrist1_mesh.glb" />
+  <xacro:property name="link06_mesh" value="wrist2_mesh.glb" />
   <!-- Joint properties -->
   <xacro:property name="joint_base_name" value="${tf_prefix}joint_base" />
@@ -56,5 +56,5 @@
   <xacro:property name="joint_1_joint_type" value="revolute" />
   <xacro:property name="joint_1_axis_xyz" value="0 0 1" />
-  <xacro:property name="joint_1_origin_xyz" value="0 0 0.1105" />
+  <xacro:property name="joint_1_origin_xyz" value="0 0 0" />
   <xacro:property name="joint_1_origin_rpy" value="0 0 0" />
   <xacro:property name="joint_1_lower_limit" value="${-J_PI - J_PI/2 + 0.4}" />
@@ -63,5 +63,5 @@
   <xacro:property name="joint_2_joint_type" value="revolute" />
   <xacro:property name="joint_2_axis_xyz" value="0 0 1" />
-  <xacro:property name="joint_2_origin_xyz" value="0 0 0.047" />
+  <xacro:property name="joint_2_origin_xyz" value="0 0 0.1575" />
   <xacro:property name="joint_2_origin_rpy" value="${J_PI/2} ${-J_PI/2} 0" />
   <xacro:property name="joint_2_lower_limit" value="${-J_PI/2 - 0.15}" />

Commit message: we are defining joint-space limits not hardware-related limits, i.e. moving also the effort-limits definitions out into the common urdf

File: duatic_dynaarm_description/urdf/common/baracuda12/dynaarm_parameters.urdf.xacro (robot description, xacro)
@@ -54,5 +54,4 @@
   <xacro:property name="joint_1_lower_limit" value="${-J_PI - J_PI/2 + 0.4}" />
   <xacro:property name="joint_1_upper_limit" value="${J_PI + J_PI/2 - 0.4}" />
-  <xacro:property name="joint_1_limit_effort" value="${drive_T120_limit_effort}" />
   <xacro:property name="joint_2_name" value="${tf_prefix}shoulder_flexion" />
   <xacro:property name="joint_2_joint_type" value="revolute" />
@@ -62,5 +61,4 @@
   <xacro:property name="joint_2_lower_limit" value="${-J_PI/2 - 0.15}" />
   <xacro:property name="joint_2_upper_limit" value="${J_PI/2 + 0.15}" />
-  <xacro:property name="joint_2_limit_effort" value="${drive_T120_limit_effort}" />
   <xacro:property name="joint_3_name" value="${tf_prefix}elbow_flexion" />
   <xacro:property name="joint_3_joint_type" value="revolute" />
@@ -70,5 +68,4 @@
   <xacro:property name="joint_3_lower_limit" value="0.00" />
   <xacro:property name="joint_3_upper_limit" value="${J_PI - 0.05}" />
-  <xacro:property name="joint_3_limit_effort" value="${drive_T120_limit_effort}" />
   <xacro:property name="joint_3_cam_name" value="${tf_prefix}elbow_camera" />
   <xacro:property name="joint_3_cam_joint_type" value="fixed" />
@@ -83,5 +80,4 @@
   <xacro:property name="joint_4_lower_limit" value="${-J_PI - J_PI/2}" />
   <xacro:property name="joint_4_upper_limit" value="${J_PI + J_PI/2}" />
-  <xacro:property name="joint_4_limit_effort" value="${drive_T40_limit_effort}" />
   <xacro:property name="joint_5_name" value="${tf_prefix}wrist_flexion" />
   <xacro:property name="joint_5_joint_type" value="revolute" />
@@ -91,5 +87,4 @@
   <xacro:property name="joint_5_lower_limit" value="${-J_PI/2 -0.25}" />
   <xacro:property name="joint_5_upper_limit" value="${J_PI/2 + 0.25}" />
-  <xacro:property name="joint_5_limit_effort" value="${drive_T40_limit_effort}" />
   <xacro:property name="joint_5_cam_name" value="${tf_prefix}wrist_flexion_camera" />
   <xacro:property name="joint_5_cam_joint_type" value="fixed" />
@@ -104,5 +99,4 @@
   <xacro:property name="joint_6_lower_limit" value="${-J_PI/2}" />
   <xacro:property name="joint_6_upper_limit" value="${J_PI + J_PI/2}" />
-  <xacro:property name="joint_6_limit_effort" value="${drive_T40_limit_effort}" />
   <xacro:property name="joint_ee_name" value="${tf_prefix}flange_fix_joint" />
   <xacro:property name="joint_ee_xyz" value="0.0 0.0 0.009" />

File: duatic_dynaarm_description/urdf/common/corydoras12/dynaarm_parameters.urdf.xacro (robot description, xacro)
@@ -54,5 +54,4 @@
   <xacro:property name="joint_1_lower_limit" value="${-J_PI - J_PI/2 + 0.4}" />
   <xacro:property name="joint_1_upper_limit" value="${J_PI + J_PI/2 - 0.4}" />
-  <xacro:property name="joint_1_limit_effort" value="${drive_T120_limit_effort}" />
   <xacro:property name="joint_2_name" value="${tf_prefix}shoulder_flexion" />
   <xacro:property name="joint_2_joint_type" value="revolute" />
@@ -62,5 +61,4 @@
   <xacro:property name="joint_2_lower_limit" value="${-J_PI/2 - 0.15}" />
   <xacro:property name="joint_2_upper_limit" value="${J_PI/2 + 0.15}" />
-  <xacro:property name="joint_2_limit_effort" value="${drive_T120_limit_effort}" />
   <xacro:property name="joint_3_name" value="${tf_prefix}elbow_flexion" />
   <xacro:property name="joint_3_joint_type" value="revolute" />
@@ -70,5 +68,4 @@
   <xacro:property name="joint_3_lower_limit" value="0.00" />
   <xacro:property name="joint_3_upper_limit" value="${J_PI - 0.05}" />
-  <xacro:property name="joint_3_limit_effort" value="${drive_T120_limit_effort}" />
   <xacro:property name="joint_3_cam_name" value="${tf_prefix}elbow_camera" />
   <xacro:property name="joint_3_cam_joint_type" value="fixed" />
@@ -83,5 +80,4 @@
   <xacro:property name="joint_4_lower_limit" value="${-J_PI - J_PI/2}" />
   <xacro:property name="joint_4_upper_limit" value="${J_PI + J_PI/2}" />
-  <xacro:property name="joint_4_limit_effort" value="${drive_T40_limit_effort}" />
   <xacro:property name="joint_5_name" value="${tf_prefix}wrist_flexion" />
   <xacro:property name="joint_5_joint_type" value="revolute" />
@@ -91,5 +87,4 @@
   <xacro:property name="joint_5_lower_limit" value="${-J_PI/2 -0.25}" />
   <xacro:property name="joint_5_upper_limit" value="${J_PI/2 + 0.25}" />
-  <xacro:property name="joint_5_limit_effort" value="${drive_T40_limit_effort}" />
   <xacro:property name="joint_5_cam_name" value="${tf_prefix}wrist_flexion_camera" />
   <xacro:property name="joint_5_cam_joint_type" value="fixed" />
@@ -104,5 +99,4 @@
   <xacro:property name="joint_6_lower_limit" value="${-J_PI/2}" />
   <xacro:property name="joint_6_upper_limit" value="${J_PI + J_PI/2}" />
-  <xacro:property name="joint_6_limit_effort" value="${drive_T40_limit_effort}" />
   <xacro:property name="joint_ee_name" value="${tf_prefix}flange_fix_joint" />
   <xacro:property name="joint_ee_xyz" value="0.0 0.0 0.009" />

File: duatic_dynaarm_description/urdf/common/dynaarm_common.urdf.xacro (robot description, xacro)
@@ -29,9 +29,4 @@
   <xacro:property name="mm_to_m" value="0.001" />
   <!-- -->
-  <!-- Common Properties -->
-  <!-- -->
-  <xacro:property name="drive_T40_limit_effort" value="40.0" />
-  <xacro:property name="drive_T120_limit_effort" value="120.0" />
-  <!-- -->
   <!-- Common Definitions -->
   <!-- -->
@@ -42,4 +37,10 @@
   <xacro:property name="joint_5_limit_vel" value="13.647" />
   <xacro:property name="joint_6_limit_vel" value="13.647" />
+  <xacro:property name="joint_1_limit_effort" value="120.0" />
+  <xacro:property name="joint_2_limit_effort" value="120.0" />
+  <xacro:property name="joint_3_limit_effort" value="120.0" />
+  <xacro:property name="joint_4_limit_effort" value="40.0" />
+  <xacro:property name="joint_5_limit_effort" value="40.0" />
+  <xacro:property name="joint_6_limit_effort" value="40.0" />
   <!-- -->
   <!-- DynaArm Base Link Macro -->

Commit message: Added base mesh for standalone dynaarm

File: duatic_dynaarm_description/urdf/common/baracuda12/dynaarm_parameters.urdf.xacro (robot description, xacro)
@@ -40,5 +40,5 @@
   <xacro:property name="end_effector" value="${tf_prefix}flange" />
   <!-- Meshes -->
-  <xacro:property name="base_mesh" value="base_mesh.glb" />
+  <xacro:property name="base_mesh" value="${'base_mesh_standalone.glb' if standalone else 'base_mesh_attached.glb'}" />
   <xacro:property name="link01_mesh" value="shoulder_mesh.glb" />
   <xacro:property name="link02_mesh" value="upperarm_mesh.glb" />

File: duatic_dynaarm_description/urdf/common/corydoras12/dynaarm_parameters.urdf.xacro (robot description, xacro)
@@ -40,5 +40,5 @@
   <xacro:property name="end_effector" value="${tf_prefix}flange" />
   <!-- Meshes -->
-  <xacro:property name="base_mesh" value="base_mesh.glb" />
+  <xacro:property name="base_mesh" value="${'base_mesh_standalone.glb' if standalone else 'base_mesh_attached.glb'}" />
   <xacro:property name="link01_mesh" value="shoulder_mesh.glb" />
   <xacro:property name="link02_mesh" value="upperarm_mesh.glb" />

File: duatic_dynaarm_description/urdf/dynaarm.urdf.xacro (robot description, xacro)
@@ -26,5 +26,5 @@
   <!-- -->
   <xacro:macro name="dynaarm_description"
-    params="tf_prefix parent_link collision:='simple' version *origin">
+    params="tf_prefix parent_link collision:='simple' version standalone:=true *origin">
     <!-- Set ee_parent -->
     <xacro:property name="ee_parent" value="${base}" />

File: duatic_dynaarm_description/urdf/dynaarm_standalone.urdf.xacro (robot description, xacro)
@@ -37,5 +37,6 @@
                 parent_link="base_link"
                 collision="$(arg collision)"
-                version="$(arg version)">
+                version="$(arg version)"
+                standalone="true">
     <origin xyz="0 0 0" rpy="0.0 0.0 0.0" />
   </xacro:dynaarm_description>
