Commit message: feat: widen simple collision mesh of base

File: duatic_dynaarm_description/urdf/common/baracuda12/dynaarm_parameters.urdf.xacro (robot description, xacro)
@@ -212,5 +212,5 @@
         <collision>
             <geometry>
-                <cylinder length='0.1' radius='0.05'/>
+                <cylinder length='0.1' radius='0.075'/>
             </geometry>
             <origin xyz='0 0 0.05' rpy='0 0 0'/>

File: duatic_dynaarm_description/urdf/common/corydoras12/dynaarm_parameters.urdf.xacro (robot description, xacro)
@@ -212,5 +212,5 @@
         <collision>
             <geometry>
-                <cylinder length='0.1' radius='0.05'/>
+                <cylinder length='0.1' radius='0.075'/>
             </geometry>
             <origin xyz='0 0 0.05' rpy='0 0 0'/>

Commit message: as requested: default values directly inside the joint descriptions

File: duatic_dynaarm_description/urdf/common/baracuda12/dynaarm_parameters.urdf.xacro (robot description, xacro)
@@ -22,9 +22,4 @@
 -->
 <robot xmlns:xacro="http://www.ros.org/wiki/xacro">
-  <!-- DuaDrive Defaults -->
-  <xacro:property name="duadrive_T120_limit_vel" value="10.64" />
-  <xacro:property name="duadrive_T120_limit_effort" value="120.0" />
-  <xacro:property name="duadrive_T40_limit_vel" value="13.647" />
-  <xacro:property name="duadrive_T40_limit_effort" value="40.0" />
   <!-- Links -->
   <xacro:property name="base" value="${tf_prefix}base" />
@@ -60,6 +55,6 @@
   <xacro:property name="joint_1_lower_limit" value="${-J_PI - J_PI/2 + 0.4}" />
   <xacro:property name="joint_1_upper_limit" value="${J_PI + J_PI/2 - 0.4}" />
-  <xacro:property name="joint_1_limit_vel_default" value="${duadrive_T120_limit_vel}" />
-  <xacro:property name="joint_1_limit_effort_default" value="${duadrive_T120_limit_effort}" />
+  <xacro:property name="joint_1_limit_vel_default" value="10.64" />
+  <xacro:property name="joint_1_limit_effort_default" value="120.0" />
   <xacro:property name="joint_2_name" value="${tf_prefix}shoulder_flexion" />
   <xacro:property name="joint_2_joint_type" value="revolute" />
@@ -69,6 +64,6 @@
   <xacro:property name="joint_2_lower_limit" value="${-J_PI/2 - 0.15}" />
   <xacro:property name="joint_2_upper_limit" value="${J_PI/2 + 0.15}" />
-  <xacro:property name="joint_2_limit_vel_default" value="${duadrive_T120_limit_vel}" />
-  <xacro:property name="joint_2_limit_effort_default" value="${duadrive_T120_limit_effort}" />
+  <xacro:property name="joint_2_limit_vel_default" value="10.64" />
+  <xacro:property name="joint_2_limit_effort_default" value="120.0" />
   <xacro:property name="joint_3_name" value="${tf_prefix}elbow_flexion" />
   <xacro:property name="joint_3_joint_type" value="revolute" />
@@ -78,6 +73,6 @@
   <xacro:property name="joint_3_lower_limit" value="0.00" />
   <xacro:property name="joint_3_upper_limit" value="${J_PI - 0.05}" />
-  <xacro:property name="joint_3_limit_vel_default" value="${duadrive_T120_limit_vel}" />
-  <xacro:property name="joint_3_limit_effort_default" value="${duadrive_T120_limit_effort}" />
+  <xacro:property name="joint_3_limit_vel_default" value="10.64" />
+  <xacro:property name="joint_3_limit_effort_default" value="120.0" />
   <xacro:property name="joint_3_cam_name" value="${tf_prefix}elbow_camera" />
   <xacro:property name="joint_3_cam_joint_type" value="fixed" />
@@ -92,6 +87,6 @@
   <xacro:property name="joint_4_lower_limit" value="${-J_PI - J_PI/2}" />
   <xacro:property name="joint_4_upper_limit" value="${J_PI + J_PI/2}" />
-  <xacro:property name="joint_4_limit_vel_default" value="${duadrive_T40_limit_vel}" />
-  <xacro:property name="joint_4_limit_effort_default" value="${duadrive_T40_limit_effort}" />
+  <xacro:property name="joint_4_limit_vel_default" value="13.647" />
+  <xacro:property name="joint_4_limit_effort_default" value="40.0" />
   <xacro:property name="joint_5_name" value="${tf_prefix}wrist_flexion" />
   <xacro:property name="joint_5_joint_type" value="revolute" />
@@ -101,6 +96,6 @@
   <xacro:property name="joint_5_lower_limit" value="${-J_PI/2 -0.25}" />
   <xacro:property name="joint_5_upper_limit" value="${J_PI/2 + 0.25}" />
-  <xacro:property name="joint_5_limit_vel_default" value="${duadrive_T40_limit_vel}" />
-  <xacro:property name="joint_5_limit_effort_default" value="${duadrive_T40_limit_effort}" />
+  <xacro:property name="joint_5_limit_vel_default" value="13.647" />
+  <xacro:property name="joint_5_limit_effort_default" value="40.0" />
   <xacro:property name="joint_5_cam_name" value="${tf_prefix}wrist_flexion_camera" />
   <xacro:property name="joint_5_cam_joint_type" value="fixed" />
@@ -115,6 +110,6 @@
   <xacro:property name="joint_6_lower_limit" value="${-J_PI/2}" />
   <xacro:property name="joint_6_upper_limit" value="${J_PI + J_PI/2}" />
-  <xacro:property name="joint_6_limit_vel_default" value="${duadrive_T40_limit_vel}" />
-  <xacro:property name="joint_6_limit_effort_default" value="${duadrive_T40_limit_effort}" />
+  <xacro:property name="joint_6_limit_vel_default" value="13.647" />
+  <xacro:property name="joint_6_limit_effort_default" value="40.0" />
   <xacro:property name="joint_ee_name" value="${tf_prefix}flange_fix_joint" />
   <xacro:property name="joint_ee_xyz" value="0.0 0.0 0.009" />

Commit message: revert(description): revert indent change not part of this PR

File: duatic_dynaarm_description/urdf/common/baracuda12/dynaarm_parameters.urdf.xacro (robot description, xacro)
@@ -186,6 +186,5 @@
   <xacro:property name="link05_inertial">
     <inertial>
-      <!-- <mass value="0.75007482" />  original value but doesn't work well - Needs to include the
-      cables inside the forearm tube?-->
+      <!-- <mass value="0.75007482" />  original value but doesn't work well - Needs to include the cables inside the forearm tube?-->
       <mass value="1.15007482" />
       <origin xyz="0.07972553 -0.00005038 0.02334747" rpy="0 0 0" />
@@ -215,60 +214,60 @@
     </inertial>
   </xacro:property>
-  <xacro:if value="${collision == 'simple'}">
+ <xacro:if value="${collision == 'simple'}">
     <!-- Collision properties -->
     <xacro:property name="base_collision">
-      <collision>
-        <geometry>
-          <cylinder length='0.1' radius='0.075' />
-        </geometry>
-        <origin xyz='0 0 0.05' rpy='0 0 0' />
-      </collision>
+        <collision>
+            <geometry>
+                <cylinder length='0.1' radius='0.075'/>
+            </geometry>
+            <origin xyz='0 0 0.05' rpy='0 0 0'/>
+        </collision>
     </xacro:property>
     <xacro:property name="link01_collision">
-      <collision>
-        <geometry>
-          <cylinder length='0.25' radius='0.06' />
-        </geometry>
-        <origin xyz='0 0 0.05' rpy='${J_PI/2} 0 0' />
-      </collision>
+          <collision>
+              <geometry>
+                  <cylinder length='0.25' radius='0.06'/>
+              </geometry>
+              <origin xyz='0 0 0.05' rpy='${J_PI/2} 0 0'/>
+          </collision>
     </xacro:property>
     <xacro:property name="link02_collision">
-      <collision>
-        <geometry>
-          <cylinder length='0.4' radius='0.05' />
-        </geometry>
-        <origin xyz='0.15 0 0' rpy='0 ${J_PI/2} 0' />
-      </collision>
+          <collision>
+              <geometry>
+                  <cylinder length='0.4' radius='0.05'/>
+              </geometry>
+              <origin xyz='0.15 0 0' rpy='0 ${J_PI/2} 0'/>
+          </collision>
     </xacro:property>
     <xacro:property name="link03_collision">
       <collision>
-        <geometry>
-          <cylinder length='0.2' radius='0.065' />
-        </geometry>
-        <origin xyz='-0.01 -0.05 0' rpy='${J_PI/2} 0 0' />
+          <geometry>
+              <cylinder length='0.2' radius='0.065'/>
+          </geometry>
+          <origin xyz='-0.01 -0.05 0' rpy='${J_PI/2} 0 0'/>
       </collision>
     </xacro:property>
     <xacro:property name="link04_collision">
       <collision>
-        <geometry>
-          <cylinder length='0.4' radius='0.04' />
-        </geometry>
-        <origin xyz='0 0 0.2' rpy='0 0 0' />
+          <geometry>
+              <cylinder length='0.4' radius='0.04'/>
+          </geometry>
+          <origin xyz='0 0 0.2' rpy='0 0 0'/>
       </collision>
     </xacro:property>
     <xacro:property name="link05_collision">
       <collision>
-        <geometry>
-          <cylinder length='0.125' radius='0.05' />
-        </geometry>
-        <origin xyz='0 0 0.025' rpy='0 0 ${J_PI/2}' />
+          <geometry>
+              <cylinder length='0.125' radius='0.05'/>
+          </geometry>
+          <origin xyz='0 0 0.025' rpy='0 0 ${J_PI/2}'/>
       </collision>
     </xacro:property>
     <xacro:property name="link06_collision">
       <collision>
-        <geometry>
-          <cylinder length='0.09' radius='0.052' />
-        </geometry>
-        <origin xyz='0.005 0 -0.035' rpy='0 0 0' />
+          <geometry>
+              <cylinder length='0.09' radius='0.052'/>
+          </geometry>
+          <origin xyz='0.005 0 -0.035' rpy='0 0 0'/>
       </collision>
     </xacro:property>

Commit message: revert: formatting changes unrelated to topic of this PR

File: duatic_dynaarm_description/urdf/common/baracuda12/dynaarm_parameters.urdf.xacro (robot description, xacro)
@@ -34,6 +34,5 @@
   <xacro:property name="end_effector" value="${tf_prefix}flange" />
   <!-- Meshes -->
-  <xacro:property name="base_mesh"
-    value="${'base_mesh_standalone.glb' if standalone else 'base_mesh_attached.glb'}" />
+  <xacro:property name="base_mesh" value="${'base_mesh_standalone.glb' if standalone else 'base_mesh_attached.glb'}" />
   <xacro:property name="link01_mesh" value="shoulder_mesh.glb" />
   <xacro:property name="link02_mesh" value="upperarm_mesh.glb" />

File: duatic_dynaarm_description/urdf/common/corydoras12/dynaarm_parameters.urdf.xacro (robot description, xacro)
@@ -34,6 +34,5 @@
   <xacro:property name="end_effector" value="${tf_prefix}flange" />
   <!-- Meshes -->
-  <xacro:property name="base_mesh"
-    value="${'base_mesh_standalone.glb' if standalone else 'base_mesh_attached.glb'}" />
+  <xacro:property name="base_mesh" value="${'base_mesh_standalone.glb' if standalone else 'base_mesh_attached.glb'}" />
   <xacro:property name="link01_mesh" value="shoulder_mesh.glb" />
   <xacro:property name="link02_mesh" value="upperarm_mesh.glb" />

File: duatic_dynaarm_description/urdf/common/dynaarm_common.urdf.xacro (robot description, xacro)
@@ -22,104 +22,103 @@
 -->
 <robot xmlns:xacro="http://www.ros.org/wiki/xacro">
-  <!-- -->
-  <!-- Common Constants -->
-  <!-- -->
-  <xacro:property name="J_PI" value="3.14159265359" />
-  <xacro:property name="mm2_to_m2" value="0.000001" />
-  <xacro:property name="mm_to_m" value="0.001" />
-  <!-- -->
-  <!-- DynaArm Base Link Macro -->
-  <!-- -->
-  <xacro:macro name="dynaarm_baselink"
-    params="link_name file_name **base_inertia **base_collision">
-    <link name="${link_name}">
-      <visual>
-        <geometry>
-          <mesh
-            filename="package://duatic_dynaarm_description/meshes/${version}/${file_name}"
-            scale="1.0 1.0 1.0" />
-        </geometry>
-        <material name="carbon_fiber">
-          <color rgba="0.792156862745098 0.819607843137255 0.933333333333333 1" />
-        </material>
-      </visual>
-      <xacro:insert_block name="base_collision" />
-      <xacro:insert_block name="base_inertia" />
-    </link>
-  </xacro:macro>
-  <!-- -->
-  <!-- DynaArm Link Macro -->
-  <!-- -->
-  <xacro:macro name="dynaarm_link"
-    params="link_name file_name **link_inertia">
-    <link name="${link_name}">
-      <visual>
-        <geometry>
-          <mesh
-            filename="package://duatic_dynaarm_description/meshes/${version}/${file_name}"
-            scale="1.0 1.0 1.0" />
-        </geometry>
-      </visual>
-      <xacro:insert_block name="link_inertia" />
-    </link>
-  </xacro:macro>
-  <!-- -->
-  <!-- DynaArm Link With Collision Macro -->
-  <!-- -->
-  <xacro:macro name="dynaarm_link_w_collision"
-    params="link_name file_name **link_inertia **link_collision">
-    <link name="${link_name}">
-      <visual>
-        <geometry>
-          <mesh
-            filename="package://duatic_dynaarm_description/meshes/${version}/${file_name}"
-            scale="1.0 1.0 1.0" />
-        </geometry>
-      </visual>
-      <xacro:insert_block name="link_inertia" />
-      <xacro:insert_block name="link_collision" />
-    </link>
-  </xacro:macro>
-  <!-- -->
-  <!-- DynaArm Virtual Link Macro -->
-  <!-- -->
-  <xacro:macro name="virtual_link"
-    params="link_name mass:=0.001 ixx:=0.0000001 iyy:=0.0000001 izz:=0.0000001">
-    <link name="${link_name}">
-      <visual>
-        <origin xyz="0 0 0" rpy="0 0 0" />
-        <geometry>
-          <box size="0.01 0.01 0.01" />
-        </geometry>
-      </visual>
-      <inertial>
-        <origin xyz="0.0 0.0 0.0" rpy="0 0 0" />
-        <mass value="${mass}" />
-        <inertia ixx="${ixx}" ixy="0.0" iyy="${iyy}" ixz="0.0" iyz="0.0" izz="${izz}" />
-      </inertial>
-      <collision>
-        <origin xyz="0 0 0" rpy="0 0 0" />
-        <geometry>
-          <box size="0.01 0.01 0.01" />
-        </geometry>
-      </collision>
-    </link>
-    <!-- Gazebo customization -->
-    <!-- Contact model -->
-    <xacro:property name="kp" value="10000.0" />
-    <xacro:property name="kd" value="10.0" />
-    <xacro:property name="mu" value="0.8" />
-    <gazebo reference="${link_name}">
-      <kp>${kp}</kp>
-      <kd>${kd}</kd>
-      <mu1>${mu}</mu1>
-      <mu2>${mu}</mu2>
-    </gazebo>
-  </xacro:macro>
-  <!-- -->
-  <!-- DynaArm Revolute Joint Macro -->
-  <!-- -->
-  <xacro:macro name="dynaarm_revolute_joint"
-    params="joint_name
+    <!-- -->
+    <!-- Common Constants -->
+    <!-- -->
+    <xacro:property name="J_PI" value="3.14159265359" />
+    <xacro:property name="mm2_to_m2" value="0.000001" />
+    <xacro:property name="mm_to_m" value="0.001" />
+    <!-- -->
+    <!-- DynaArm Base Link Macro -->
+    <!-- -->
+    <xacro:macro name="dynaarm_baselink"
+        params="link_name file_name **base_inertia **base_collision">
+        <link name="${link_name}">
+            <visual>
+                <geometry>
+                    <mesh
+                        filename="package://duatic_dynaarm_description/meshes/${version}/${file_name}"
+                        scale="1.0 1.0 1.0" />
+                </geometry>
+                <material name="carbon_fiber">
+                    <color rgba="0.792156862745098 0.819607843137255 0.933333333333333 1" />
+                </material>
+            </visual>
+            <xacro:insert_block name="base_collision" />
+            <xacro:insert_block name="base_inertia" />
+        </link>
+    </xacro:macro>
+    <!-- -->
+    <!-- DynaArm Link Macro -->
+    <!-- -->
+    <xacro:macro name="dynaarm_link"
+        params="link_name file_name **link_inertia">
+        <link name="${link_name}">
+            <visual>
+                <geometry>
+                    <mesh
+                        filename="package://duatic_dynaarm_description/meshes/${version}/${file_name}"
+                        scale="1.0 1.0 1.0" />
+                </geometry>
+            </visual>
+            <xacro:insert_block name="link_inertia" />
+        </link>
+    </xacro:macro>
+    <!-- -->
+    <!-- DynaArm Link With Collision Macro -->
+    <!-- -->
+    <xacro:macro name="dynaarm_link_w_collision"
+        params="link_name file_name **link_inertia **link_collision">
+        <link name="${link_name}">
+            <visual>
+                <geometry>
+                    <mesh
+                        filename="package://duatic_dynaarm_description/meshes/${version}/${file_name}"
+                        scale="1.0 1.0 1.0" />
+                </geometry>
+            </visual>
+            <xacro:insert_block name="link_inertia" />
+            <xacro:insert_block name="link_collision" />
+        </link>
+    </xacro:macro>
+    <!-- -->
+    <!-- DynaArm Virtual Link Macro -->
+    <!-- -->
+    <xacro:macro name="virtual_link" params="link_name mass:=0.001 ixx:=0.0000001 iyy:=0.0000001 izz:=0.0000001">
+        <link name="${link_name}">
+            <visual>
+                <origin xyz="0 0 0" rpy="0 0 0" />
+                <geometry>
+                    <box size="0.01 0.01 0.01" />
+                </geometry>
+            </visual>
+            <inertial>
+                <origin xyz="0.0 0.0 0.0" rpy="0 0 0" />
+                <mass value="${mass}" />
+                <inertia ixx="${ixx}" ixy="0.0" iyy="${iyy}" ixz="0.0" iyz="0.0" izz="${izz}" />
+            </inertial>
+            <collision>
+                <origin xyz="0 0 0" rpy="0 0 0" />
+                <geometry>
+                    <box size="0.01 0.01 0.01" />
+                </geometry>
+            </collision>
+        </link>
+        <!-- Gazebo customization -->
+        <!-- Contact model -->
+        <xacro:property name="kp" value="10000.0" />
+        <xacro:property name="kd" value="10.0" />
+        <xacro:property name="mu" value="0.8" />
+        <gazebo reference="${link_name}">
+            <kp>${kp}</kp>
+            <kd>${kd}</kd>
+            <mu1>${mu}</mu1>
+            <mu2>${mu}</mu2>
+        </gazebo>
+    </xacro:macro>
+    <!-- -->
+    <!-- DynaArm Revolute Joint Macro -->
+    <!-- -->
+    <xacro:macro name="dynaarm_revolute_joint"
+        params="joint_name
                 parent
                 child
@@ -131,26 +130,26 @@
                 joint_type
                 *origin">
-    <joint name="${joint_name}" type="${joint_type}">
-      <parent link="${parent}" />
-      <child link="${child}" />
-      <axis xyz="${joint_axis_xyz}" />
-      <limit effort="${joint_limit_effort}" command_effort="${joint_limit_effort}"
-        current="10" gear_velocity="${joint_limit_vel}" velocity="${joint_limit_vel}"
-        lower="${joint_lower_limit}" upper="${joint_upper_limit}" />
-      <!-- limit effort also defines torque limit and freeze controller gains -->
-      <xacro:insert_block name="origin" />
-    </joint>
-  </xacro:macro>
-  <!-- -->
-  <!-- DynaArm Fixed Joint Macro -->
-  <!-- -->
-  <xacro:macro name="dynaarm_joint_fixed"
-    params="joint_name parent child *origin">
-    <joint name="${joint_name}" type="fixed">
-      <parent link="${parent}" />
-      <child link="${child}" />
-      <limit effort="2000" velocity="0" lower="0" upper="0" />
-      <xacro:insert_block name="origin" />
-    </joint>
-  </xacro:macro>
+        <joint name="${joint_name}" type="${joint_type}">
+            <parent link="${parent}" />
+            <child link="${child}" />
+            <axis xyz="${joint_axis_xyz}" />
+            <limit effort="${joint_limit_effort}" command_effort="${joint_limit_effort}"
+                current="10" gear_velocity="${joint_limit_vel}" velocity="${joint_limit_vel}"
+                lower="${joint_lower_limit}" upper="${joint_upper_limit}" />
+            <!-- limit effort also defines torque limit and freeze controller gains -->
+            <xacro:insert_block name="origin" />
+        </joint>
+    </xacro:macro>
+    <!-- -->
+    <!-- DynaArm Fixed Joint Macro -->
+    <!-- -->
+    <xacro:macro name="dynaarm_joint_fixed"
+        params="joint_name parent child *origin">
+        <joint name="${joint_name}" type="fixed">
+            <parent link="${parent}" />
+            <child link="${child}" />
+            <limit effort="2000" velocity="0" lower="0" upper="0" />
+            <xacro:insert_block name="origin" />
+        </joint>
+    </xacro:macro>
 </robot>

File: duatic_dynaarm_description/urdf/dynaarm.urdf.xacro (robot description, xacro)
@@ -26,18 +26,12 @@
   <!-- -->
   <xacro:macro name="dynaarm_description"
-    params="tf_prefix parent_link
-      collision:='simple'
-      version
-      standalone:='true'
+    params="tf_prefix parent_link collision:='simple' version standalone:=true
       joint_limits:=${xacro.load_yaml('$(find duatic_dynaarm_description)/config/limits/limits.yaml')}
       *origin">
     <!-- Set ee_parent -->
     <xacro:property name="ee_parent" value="${base}" />
-    <xacro:include
-      filename="$(find duatic_dynaarm_description)/urdf/common/dynaarm_common.urdf.xacro" />
-    <!-- Include the version specific information and also load the ethercat addresses from the
-    drive file -->
-    <xacro:include
-      filename="$(find duatic_dynaarm_description)/urdf/common/${version}/dynaarm_parameters.urdf.xacro" />
+    <xacro:include filename="$(find duatic_dynaarm_description)/urdf/common/dynaarm_common.urdf.xacro" />
+    <!-- Include the version specific information and also load the ethercat addresses from the drive file -->
+    <xacro:include filename="$(find duatic_dynaarm_description)/urdf/common/${version}/dynaarm_parameters.urdf.xacro" />
     <xacro:dynaarm_joint_fixed joint_name="${joint_base_name}"
       parent="${parent_link}"
@@ -206,10 +200,10 @@
   <!-- -->
   <xacro:macro name="dynaarm_tool">
-    <xacro:virtual_link link_name="${end_effector}" />
-    <xacro:dynaarm_joint_fixed joint_name="${joint_ee_name}"
-      parent="${ee_parent}"
-      child="${end_effector}">
-      <origin xyz="${joint_ee_origin_xyz}" rpy="${joint_ee_origin_rpy}" />
-    </xacro:dynaarm_joint_fixed>
+      <xacro:virtual_link link_name="${end_effector}" />
+      <xacro:dynaarm_joint_fixed joint_name="${joint_ee_name}"
+          parent="${ee_parent}"
+          child="${end_effector}">
+          <origin xyz="${joint_ee_origin_xyz}" rpy="${joint_ee_origin_rpy}" />
+      </xacro:dynaarm_joint_fixed>
   </xacro:macro>
 </robot>
