Commit message: refactor(description): define joint velocity and effort limits per version
Rename the baracuda12 joint_N_limit_vel_default and
joint_N_limit_effort_default properties to joint_N_limit_vel and
joint_N_limit_effort, and add the same properties to corydoras12, so
both versions define their default velocity and effort limits next to
the position limits.

File: duatic_dynaarm_description/urdf/common/baracuda12/dynaarm_parameters.urdf.xacro (robot description, xacro)
@@ -54,6 +54,6 @@
   <xacro:property name="joint_1_lower_limit" value="${-J_PI - J_PI/2 + 0.4}" />
   <xacro:property name="joint_1_upper_limit" value="${J_PI + J_PI/2 - 0.4}" />
-  <xacro:property name="joint_1_limit_vel_default" value="10.64" />
-  <xacro:property name="joint_1_limit_effort_default" value="120.0" />
+  <xacro:property name="joint_1_limit_vel" value="10.64" />
+  <xacro:property name="joint_1_limit_effort" value="120.0" />
   <xacro:property name="joint_2_name" value="${tf_prefix}shoulder_flexion" />
   <xacro:property name="joint_2_joint_type" value="revolute" />
@@ -63,6 +63,6 @@
   <xacro:property name="joint_2_lower_limit" value="${-J_PI/2 - 0.15}" />
   <xacro:property name="joint_2_upper_limit" value="${J_PI/2 + 0.15}" />
-  <xacro:property name="joint_2_limit_vel_default" value="10.64" />
-  <xacro:property name="joint_2_limit_effort_default" value="120.0" />
+  <xacro:property name="joint_2_limit_vel" value="10.64" />
+  <xacro:property name="joint_2_limit_effort" value="120.0" />
   <xacro:property name="joint_3_name" value="${tf_prefix}elbow_flexion" />
   <xacro:property name="joint_3_joint_type" value="revolute" />
@@ -72,6 +72,6 @@
   <xacro:property name="joint_3_lower_limit" value="0.00" />
   <xacro:property name="joint_3_upper_limit" value="${J_PI - 0.05}" />
-  <xacro:property name="joint_3_limit_vel_default" value="10.64" />
-  <xacro:property name="joint_3_limit_effort_default" value="120.0" />
+  <xacro:property name="joint_3_limit_vel" value="10.64" />
+  <xacro:property name="joint_3_limit_effort" value="120.0" />
   <xacro:property name="joint_3_cam_name" value="${tf_prefix}elbow_camera" />
   <xacro:property name="joint_3_cam_joint_type" value="fixed" />
@@ -86,6 +86,6 @@
   <xacro:property name="joint_4_lower_limit" value="${-J_PI - J_PI/2}" />
   <xacro:property name="joint_4_upper_limit" value="${J_PI + J_PI/2}" />
-  <xacro:property name="joint_4_limit_vel_default" value="13.647" />
-  <xacro:property name="joint_4_limit_effort_default" value="40.0" />
+  <xacro:property name="joint_4_limit_vel" value="13.647" />
+  <xacro:property name="joint_4_limit_effort" value="40.0" />
   <xacro:property name="joint_5_name" value="${tf_prefix}wrist_flexion" />
   <xacro:property name="joint_5_joint_type" value="revolute" />
@@ -95,6 +95,6 @@
   <xacro:property name="joint_5_lower_limit" value="${-J_PI/2 -0.25}" />
   <xacro:property name="joint_5_upper_limit" value="${J_PI/2 + 0.25}" />
-  <xacro:property name="joint_5_limit_vel_default" value="13.647" />
-  <xacro:property name="joint_5_limit_effort_default" value="40.0" />
+  <xacro:property name="joint_5_limit_vel" value="13.647" />
+  <xacro:property name="joint_5_limit_effort" value="40.0" />
   <xacro:property name="joint_5_cam_name" value="${tf_prefix}wrist_flexion_camera" />
   <xacro:property name="joint_5_cam_joint_type" value="fixed" />
@@ -109,6 +109,6 @@
   <xacro:property name="joint_6_lower_limit" value="${-J_PI/2}" />
   <xacro:property name="joint_6_upper_limit" value="${J_PI + J_PI/2}" />
-  <xacro:property name="joint_6_limit_vel_default" value="13.647" />
-  <xacro:property name="joint_6_limit_effort_default" value="40.0" />
+  <xacro:property name="joint_6_limit_vel" value="13.647" />
+  <xacro:property name="joint_6_limit_effort" value="40.0" />
   <xacro:property name="joint_ee_name" value="${tf_prefix}flange_fix_joint" />
   <xacro:property name="joint_ee_xyz" value="0.0 0.0 0.009" />

File: duatic_dynaarm_description/urdf/common/corydoras12/dynaarm_parameters.urdf.xacro (robot description, xacro)
@@ -54,4 +54,6 @@
   <xacro:property name="joint_1_lower_limit" value="${-J_PI - J_PI/2 + 0.4}" />
   <xacro:property name="joint_1_upper_limit" value="${J_PI + J_PI/2 - 0.4}" />
+  <xacro:property name="joint_1_limit_vel" value="10.64" />
+  <xacro:property name="joint_1_limit_effort" value="120.0" />
   <xacro:property name="joint_2_name" value="${tf_prefix}shoulder_flexion" />
   <xacro:property name="joint_2_joint_type" value="revolute" />
@@ -61,4 +63,6 @@
   <xacro:property name="joint_2_lower_limit" value="${-J_PI/2 - 0.15}" />
   <xacro:property name="joint_2_upper_limit" value="${J_PI/2 + 0.15}" />
+  <xacro:property name="joint_2_limit_vel" value="10.64" />
+  <xacro:property name="joint_2_limit_effort" value="120.0" />
   <xacro:property name="joint_3_name" value="${tf_prefix}elbow_flexion" />
   <xacro:property name="joint_3_joint_type" value="revolute" />
@@ -68,4 +72,6 @@
   <xacro:property name="joint_3_lower_limit" value="0.00" />
   <xacro:property name="joint_3_upper_limit" value="${J_PI - 0.05}" />
+  <xacro:property name="joint_3_limit_vel" value="10.64" />
+  <xacro:property name="joint_3_limit_effort" value="120.0" />
   <xacro:property name="joint_3_cam_name" value="${tf_prefix}elbow_camera" />
   <xacro:property name="joint_3_cam_joint_type" value="fixed" />
@@ -80,4 +86,6 @@
   <xacro:property name="joint_4_lower_limit" value="${-J_PI - J_PI/2}" />
   <xacro:property name="joint_4_upper_limit" value="${J_PI + J_PI/2}" />
+  <xacro:property name="joint_4_limit_vel" value="13.647" />
+  <xacro:property name="joint_4_limit_effort" value="40.0" />
   <xacro:property name="joint_5_name" value="${tf_prefix}wrist_flexion" />
   <xacro:property name="joint_5_joint_type" value="revolute" />
@@ -87,4 +95,6 @@
   <xacro:property name="joint_5_lower_limit" value="${-J_PI/2 -0.25}" />
   <xacro:property name="joint_5_upper_limit" value="${J_PI/2 + 0.25}" />
+  <xacro:property name="joint_5_limit_vel" value="13.647" />
+  <xacro:property name="joint_5_limit_effort" value="40.0" />
   <xacro:property name="joint_5_cam_name" value="${tf_prefix}wrist_flexion_camera" />
   <xacro:property name="joint_5_cam_joint_type" value="fixed" />
@@ -99,4 +109,6 @@
   <xacro:property name="joint_6_lower_limit" value="${-J_PI/2}" />
   <xacro:property name="joint_6_upper_limit" value="${J_PI + J_PI/2}" />
+  <xacro:property name="joint_6_limit_vel" value="13.647" />
+  <xacro:property name="joint_6_limit_effort" value="40.0" />
   <xacro:property name="joint_ee_name" value="${tf_prefix}flange_fix_joint" />
   <xacro:property name="joint_ee_xyz" value="0.0 0.0 0.009" />

Commit message: refactor(description): keep constants in the version parameter files
Move J_PI, mm2_to_m2 and mm_to_m from dynaarm_common.urdf.xacro back
into the baracuda12 and corydoras12 parameter files, where they are
defined on main. The generated URDF is unchanged.

File: duatic_dynaarm_description/urdf/common/baracuda12/dynaarm_parameters.urdf.xacro (robot description, xacro)
@@ -22,4 +22,7 @@
 -->
 <robot xmlns:xacro="http://www.ros.org/wiki/xacro">
+  <xacro:property name="J_PI" value="3.14159265359" />
+  <xacro:property name="mm2_to_m2" value="0.000001" />
+  <xacro:property name="mm_to_m" value="0.001" />
   <!-- Links -->
   <xacro:property name="base" value="${tf_prefix}base" />

File: duatic_dynaarm_description/urdf/common/dynaarm_common.urdf.xacro (robot description, xacro)
@@ -22,10 +22,4 @@
 -->
 <robot xmlns:xacro="http://www.ros.org/wiki/xacro">
-    <!-- -->
-    <!-- Common Constants -->
-    <!-- -->
-    <xacro:property name="J_PI" value="3.14159265359" />
-    <xacro:property name="mm2_to_m2" value="0.000001" />
-    <xacro:property name="mm_to_m" value="0.001" />
     <!-- -->
     <!-- DynaArm Base Link Macro -->

Commit message: refactor(description): remove unused URDF properties
Fourteen parameter properties and the camera mount inertials were
defined in both version files but never read. The ee_parent set in
dynaarm.urdf.xacro was always overwritten by the parameters file.
Properties defined inside dynaarm_description are scoped to that macro,
so no downstream description can depend on them. Rendered URDFs are
byte-identical.

File: duatic_dynaarm_description/urdf/common/baracuda12/dynaarm_parameters.urdf.xacro (robot description, xacro)
@@ -23,6 +23,4 @@
 <robot xmlns:xacro="http://www.ros.org/wiki/xacro">
   <xacro:property name="J_PI" value="3.14159265359" />
-  <xacro:property name="mm2_to_m2" value="0.000001" />
-  <xacro:property name="mm_to_m" value="0.001" />
   <!-- Links -->
   <xacro:property name="base" value="${tf_prefix}base" />
@@ -46,8 +44,4 @@
   <!-- Joint properties -->
   <xacro:property name="joint_base_name" value="${tf_prefix}joint_base" />
-  <xacro:property name="joint_base_joint_type" value="revolute" />
-  <xacro:property name="joint_base_axis_xyz" value="0 0 0" />
-  <xacro:property name="joint_base_origin_xyz" value="0 0 0" />
-  <xacro:property name="joint_base_origin_rpy" value="0 0 0" />
   <xacro:property name="joint_1_name" value="${tf_prefix}shoulder_rotation" />
   <xacro:property name="joint_1_joint_type" value="revolute" />
@@ -78,6 +72,4 @@
   <xacro:property name="joint_3_limit_effort" value="120.0" />
   <xacro:property name="joint_3_cam_name" value="${tf_prefix}elbow_camera" />
-  <xacro:property name="joint_3_cam_joint_type" value="fixed" />
-  <xacro:property name="joint_3_cam_axis_xyz" value="0 0 0" />
   <xacro:property name="joint_3_cam_origin_xyz" value="0.0345 -0.1235 0" />
   <xacro:property name="joint_3_cam_origin_rpy" value="0.0 0.0 0.0" />
@@ -101,6 +93,4 @@
   <xacro:property name="joint_5_limit_effort" value="40.0" />
   <xacro:property name="joint_5_cam_name" value="${tf_prefix}wrist_flexion_camera" />
-  <xacro:property name="joint_5_cam_joint_type" value="fixed" />
-  <xacro:property name="joint_5_cam_axis_xyz" value="0 0 0" />
   <xacro:property name="joint_5_cam_origin_xyz" value="0.032 0 -0.017" />
   <xacro:property name="joint_5_cam_origin_rpy" value="0.0 0.0 0.0" />
@@ -115,10 +105,6 @@
   <xacro:property name="joint_6_limit_effort" value="40.0" />
   <xacro:property name="joint_ee_name" value="${tf_prefix}flange_fix_joint" />
-  <xacro:property name="joint_ee_xyz" value="0.0 0.0 0.009" />
   <xacro:property name="joint_ee_origin_xyz" value="0.0 0.0 0.009" />
-  <xacro:property name="joint_ee_origin_4dof_xyz" value="0.0 0.0 0.009" />
   <xacro:property name="joint_ee_origin_rpy" value="0.0 0.0 ${J_PI/2}" />
-  <xacro:property name="joint_ee_origin_4dof_rpy" value="0.0 0.0 ${J_PI/2}" />
-  <xacro:property name="joint_ee_rpy" value="0 0 0" />
   <!-- Base Robot -->
   <xacro:property name="base_inertial">
@@ -165,14 +151,4 @@
     </inertial>
   </xacro:property>
-  <!-- Camera Mounting Point 1 -->
-  <xacro:property name="link03_cam_inertial">
-    <inertial>
-      <mass value="1e-6" />
-      <origin xyz="0.0 0.0 0.0" rpy="0 0 0" />
-      <inertia ixx="1e-6" iyy="1e-6"
-        izz="1e-6" ixy="1e-6"
-        ixz="1e-6" iyz="1e-6" />
-    </inertial>
-  </xacro:property>
   <!-- Forearm -->
   <xacro:property name="link04_inertial">
@@ -194,14 +170,4 @@
         izz="0.00078106" ixy="0.00000076"
         ixz="0.00011795" iyz="-0.00000079" />
-    </inertial>
-  </xacro:property>
-  <!-- Camera Mounting Point 2 -->
-  <xacro:property name="link05_cam_inertial">
-    <inertial>
-      <mass value="1e-6" />
-      <origin xyz="0.0 0.0 0.0" rpy="0 0 0" />
-      <inertia ixx="1e-6" iyy="1e-6"
-        izz="1e-6" ixy="1e-6"
-        ixz="1e-6" iyz="1e-6" />
     </inertial>
   </xacro:property>

File: duatic_dynaarm_description/urdf/dynaarm.urdf.xacro (robot description, xacro)
@@ -29,6 +29,4 @@
       joint_limits_yaml:=''
       *origin">
-    <!-- Set ee_parent -->
-    <xacro:property name="ee_parent" value="${base}" />
     <xacro:include filename="$(find duatic_dynaarm_description)/urdf/common/dynaarm_common.urdf.xacro" />
     <!-- Include the version specific information and also load the ethercat addresses from the drive file -->
