Commit message: refactor(description): let corydoras12 reuse the baracuda12 parameters
The corydoras12 and baracuda12 parameter files were identical, and the
versions will not diverge in kinematics or inertia. The corydoras12 file
now includes the baracuda12 one instead of duplicating it, so the
parameters stay per version and an unsupported version still fails at
the include. The ee_parent alias always resolved to link06, so the
flange joint uses link06 directly. Rendered URDFs are byte-identical,
with and without a joint limits file.

File: duatic_dynaarm_description/urdf/common/baracuda12/dynaarm_parameters.urdf.xacro (robot description, xacro)
@@ -315,5 +315,3 @@
     </xacro:property>
   </xacro:if>
-  <!-- Set the ee_parent -->
-  <xacro:property name="ee_parent" value="${link06}" />
 </robot>

File: duatic_dynaarm_description/urdf/common/corydoras12/dynaarm_parameters.urdf.xacro (robot description, xacro)
@@ -22,298 +22,5 @@
 -->
 <robot xmlns:xacro="http://www.ros.org/wiki/xacro">
-  <xacro:property name="J_PI" value="3.14159265359" />
-  <!-- Links -->
-  <xacro:property name="base" value="${tf_prefix}base" />
-  <xacro:property name="link01" value="${tf_prefix}shoulder" />
-  <xacro:property name="link02" value="${tf_prefix}upperarm" />
-  <xacro:property name="link03" value="${tf_prefix}elbow" />
-  <xacro:property name="link03_cam" value="${tf_prefix}elbow_camera_mount" />
-  <xacro:property name="link04" value="${tf_prefix}forearm" />
-  <xacro:property name="link05" value="${tf_prefix}wrist_1" />
-  <xacro:property name="link05_cam" value="${tf_prefix}wrist_1_camera_mount" />
-  <xacro:property name="link06" value="${tf_prefix}wrist_2" />
-  <xacro:property name="end_effector" value="${tf_prefix}flange" />
-  <!-- Meshes -->
-  <xacro:property name="base_mesh" value="${'base_mesh_standalone.glb' if standalone else 'base_mesh_attached.glb'}" />
-  <xacro:property name="link01_mesh" value="shoulder_mesh.glb" />
-  <xacro:property name="link02_mesh" value="upperarm_mesh.glb" />
-  <xacro:property name="link03_mesh" value="elbow_mesh.glb" />
-  <xacro:property name="link04_mesh" value="forearm_mesh.glb" />
-  <xacro:property name="link05_mesh" value="wrist1_mesh.glb" />
-  <xacro:property name="link06_mesh" value="wrist2_mesh.glb" />
-  <!-- Joint properties -->
-  <xacro:property name="joint_base_name" value="${tf_prefix}joint_base" />
-  <xacro:property name="joint_1_name" value="${tf_prefix}shoulder_rotation" />
-  <xacro:property name="joint_1_joint_type" value="revolute" />
-  <xacro:property name="joint_1_axis_xyz" value="0 0 1" />
-  <xacro:property name="joint_1_origin_xyz" value="0 0 0.1105" />
-  <xacro:property name="joint_1_origin_rpy" value="0 0 0" />
-  <xacro:property name="joint_1_lower_limit" value="${-J_PI - J_PI/2 + 0.4}" />
-  <xacro:property name="joint_1_upper_limit" value="${J_PI + J_PI/2 - 0.4}" />
-  <xacro:property name="joint_1_limit_vel" value="10.64" />
-  <xacro:property name="joint_1_limit_effort" value="120.0" />
-  <xacro:property name="joint_2_name" value="${tf_prefix}shoulder_flexion" />
-  <xacro:property name="joint_2_joint_type" value="revolute" />
-  <xacro:property name="joint_2_axis_xyz" value="0 0 1" />
-  <xacro:property name="joint_2_origin_xyz" value="0 0 0.047" />
-  <xacro:property name="joint_2_origin_rpy" value="${J_PI/2} ${-J_PI/2} 0" />
-  <xacro:property name="joint_2_lower_limit" value="${-J_PI/2 - 0.15}" />
-  <xacro:property name="joint_2_upper_limit" value="${J_PI/2 + 0.15}" />
-  <xacro:property name="joint_2_limit_vel" value="10.64" />
-  <xacro:property name="joint_2_limit_effort" value="120.0" />
-  <xacro:property name="joint_3_name" value="${tf_prefix}elbow_flexion" />
-  <xacro:property name="joint_3_joint_type" value="revolute" />
-  <xacro:property name="joint_3_axis_xyz" value="0 0 1" />
-  <xacro:property name="joint_3_origin_xyz" value="0.4127 0 0" />
-  <xacro:property name="joint_3_origin_rpy" value="0 0 0" />
-  <xacro:property name="joint_3_lower_limit" value="0.00" />
-  <xacro:property name="joint_3_upper_limit" value="${J_PI - 0.05}" />
-  <xacro:property name="joint_3_limit_vel" value="10.64" />
-  <xacro:property name="joint_3_limit_effort" value="120.0" />
-  <xacro:property name="joint_3_cam_name" value="${tf_prefix}elbow_camera" />
-  <xacro:property name="joint_3_cam_origin_xyz" value="0.0345 -0.1235 0" />
-  <xacro:property name="joint_3_cam_origin_rpy" value="0.0 0.0 0.0" />
-  <xacro:property name="joint_4_name" value="${tf_prefix}forearm_rotation" />
-  <xacro:property name="joint_4_joint_type" value="revolute" />
-  <xacro:property name="joint_4_axis_xyz" value="0 0 1" />
-  <xacro:property name="joint_4_origin_xyz" value="0.0262 -0.0855 0" />
-  <xacro:property name="joint_4_origin_rpy" value="${J_PI/2} ${J_PI/2} ${J_PI/2}" />
-  <xacro:property name="joint_4_lower_limit" value="${-J_PI - J_PI/2}" />
-  <xacro:property name="joint_4_upper_limit" value="${J_PI + J_PI/2}" />
-  <xacro:property name="joint_4_limit_vel" value="13.647" />
-  <xacro:property name="joint_4_limit_effort" value="40.0" />
-  <xacro:property name="joint_5_name" value="${tf_prefix}wrist_flexion" />
-  <xacro:property name="joint_5_joint_type" value="revolute" />
-  <xacro:property name="joint_5_axis_xyz" value="0 0 1" />
-  <xacro:property name="joint_5_origin_xyz" value="0.0295 0 0.4207" />
-  <xacro:property name="joint_5_origin_rpy" value="0 ${-J_PI/2} 0" />
-  <xacro:property name="joint_5_lower_limit" value="${-J_PI/2 -0.25}" />
-  <xacro:property name="joint_5_upper_limit" value="${J_PI/2 + 0.25}" />
-  <xacro:property name="joint_5_limit_vel" value="13.647" />
-  <xacro:property name="joint_5_limit_effort" value="40.0" />
-  <xacro:property name="joint_5_cam_name" value="${tf_prefix}wrist_flexion_camera" />
-  <xacro:property name="joint_5_cam_origin_xyz" value="0.032 0 -0.017" />
-  <xacro:property name="joint_5_cam_origin_rpy" value="0.0 0.0 0.0" />
-  <xacro:property name="joint_6_name" value="${tf_prefix}wrist_rotation" />
-  <xacro:property name="joint_6_joint_type" value="revolute" />
-  <xacro:property name="joint_6_axis_xyz" value="0 0 1" />
-  <xacro:property name="joint_6_origin_xyz" value="0.117 0.0 0.0295" />
-  <xacro:property name="joint_6_origin_rpy" value="${-J_PI/2} ${J_PI/2} ${-J_PI/2}" />
-  <xacro:property name="joint_6_lower_limit" value="${-J_PI/2}" />
-  <xacro:property name="joint_6_upper_limit" value="${J_PI + J_PI/2}" />
-  <xacro:property name="joint_6_limit_vel" value="13.647" />
-  <xacro:property name="joint_6_limit_effort" value="40.0" />
-  <xacro:property name="joint_ee_name" value="${tf_prefix}flange_fix_joint" />
-  <xacro:property name="joint_ee_origin_xyz" value="0.0 0.0 0.009" />
-  <xacro:property name="joint_ee_origin_rpy" value="0.0 0.0 ${J_PI/2}" />
-  <!-- Base Robot -->
-  <xacro:property name="base_inertial">
-    <inertial>
-      <mass value="1.94219788" />
-      <origin
-        xyz="0.00243205 0.00250861 0.05299306"
-        rpy="0 0 0" />
-      <inertia ixx="0.00434815" iyy="0.00446542"
-        izz="0.00446174" ixy="0.00028867"
-        ixz="-0.00015925" iyz="-0.00015771" />
-    </inertial>
-  </xacro:property>
-  <!-- Shoulder -->
-  <xacro:property name="link01_inertial">
-    <inertial>
-      <mass value="2.825469" />
-      <origin xyz="0.000012 0.000480 0.039513" rpy="0 0 0" />
-      <inertia ixx="0.013069" iyy="0.004793"
-        izz="0.012242" ixy="0.000033"
-        ixz="-0.000002" iyz="-0.000046" />
-    </inertial>
-  </xacro:property>
-  <!-- Upper Arm -->
-  <xacro:property name="link02_inertial">
-    <inertial>
-      <!-- Original - <mass value="1.72040464" /> -->
-      <mass value="2.12040464" />
-      <origin xyz="0.20391301 -0.00000528 -0.00015224"
-        rpy="0 0 0" />
-      <inertia ixx="0.00155499" iyy="0.05067934"
-        izz="0.0507131" ixy="0.00000098"
-        ixz="0.00004108" iyz="-0.00000143" />
-    </inertial>
-  </xacro:property>
-  <!-- Elbow -->
-  <xacro:property name="link03_inertial">
-    <inertial>
-      <mass value="0.82320237" />
-      <origin xyz="0.00383866 -0.07802638 -0.00026928" rpy="0 0 0" />
-      <inertia ixx="0.00107419" iyy="0.00087121"
-        izz="0.00113856" ixy="0.00004166"
-        ixz="-0.00000398" iyz="-0.0000119" />
-    </inertial>
-  </xacro:property>
-  <!-- Forearm -->
-  <xacro:property name="link04_inertial">
-    <inertial>
-      <mass value="1.237246" />
-      <origin xyz="-0.001568 0.000046 0.292163" rpy="0 0 0" />
-      <inertia ixx="0.033872" iyy="0.033868"
-        izz="0.001041" ixy="0.000002"
-        ixz="-0.000276" iyz="0.000018" />
-    </inertial>
-  </xacro:property>
-  <!-- wrist_1 -->
-  <xacro:property name="link05_inertial">
-    <inertial>
-      <!-- <mass value="0.75007482" />  original value but doesn't work well - Needs to include the cables inside the forearm tube?-->
-      <mass value="1.15007482" />
-      <origin xyz="0.07972553 -0.00005038 0.02334747" rpy="0 0 0" />
-      <inertia ixx="0.00065953" iyy="0.00088282"
-        izz="0.00078106" ixy="0.00000076"
-        ixz="0.00011795" iyz="-0.00000079" />
-    </inertial>
-  </xacro:property>
-  <!-- Wrist 2 -->
-  <xacro:property name="link06_inertial">
-    <inertial>
-      <mass value="0.0478406" />
-      <origin xyz="0.00045711 0.00000557 0.00344945" rpy="0 0 0" />
-      <inertia ixx="0.00001366" iyy="0.00001419"
-        izz="0.00002702" ixy="0"
-        ixz="0.00000008" iyz="0" />
-    </inertial>
-  </xacro:property>
- <xacro:if value="${collision == 'simple'}">
-    <!-- Collision properties -->
-    <xacro:property name="base_collision">
-        <collision>
-            <geometry>
-                <cylinder length='0.1' radius='0.075'/>
-            </geometry>
-            <origin xyz='0 0 0.05' rpy='0 0 0'/>
-        </collision>
-    </xacro:property>
-    <xacro:property name="link01_collision">
-          <collision>
-              <geometry>
-                  <cylinder length='0.25' radius='0.06'/>
-              </geometry>
-              <origin xyz='0 0 0.05' rpy='${J_PI/2} 0 0'/>
-          </collision>
-    </xacro:property>
-    <xacro:property name="link02_collision">
-          <collision>
-              <geometry>
-                  <cylinder length='0.4' radius='0.05'/>
-              </geometry>
-              <origin xyz='0.15 0 0' rpy='0 ${J_PI/2} 0'/>
-          </collision>
-    </xacro:property>
-    <xacro:property name="link03_collision">
-      <collision>
-          <geometry>
-              <cylinder length='0.2' radius='0.065'/>
-          </geometry>
-          <origin xyz='-0.01 -0.05 0' rpy='${J_PI/2} 0 0'/>
-      </collision>
-    </xacro:property>
-    <xacro:property name="link04_collision">
-      <collision>
-          <geometry>
-              <cylinder length='0.4' radius='0.04'/>
-          </geometry>
-          <origin xyz='0 0 0.2' rpy='0 0 0'/>
-      </collision>
-    </xacro:property>
-    <xacro:property name="link05_collision">
-      <collision>
-          <geometry>
-              <cylinder length='0.125' radius='0.05'/>
-          </geometry>
-          <origin xyz='0 0 0.025' rpy='0 0 ${J_PI/2}'/>
-      </collision>
-    </xacro:property>
-    <xacro:property name="link06_collision">
-      <collision>
-          <geometry>
-              <cylinder length='0.09' radius='0.052'/>
-          </geometry>
-          <origin xyz='0.005 0 -0.035' rpy='0 0 0'/>
-      </collision>
-    </xacro:property>
-  </xacro:if>
-  <xacro:if value="${collision == 'complex'}">
-    <!-- Collision properties: reuse the visual meshes (base_mesh already resolves to the
-         standalone/attached variant) instead of the separate collision_meshes/*.stl files -->
-    <xacro:property name="base_collision">
-      <collision>
-        <origin xyz="0 0 0" rpy="0 0 0" />
-        <geometry>
-          <mesh
-            filename="package://duatic_dynaarm_description/meshes/${version}/${base_mesh}"
-            scale="1 1 1" />
-        </geometry>
-      </collision>
-    </xacro:property>
-    <xacro:property name="link01_collision">
-      <collision>
-        <origin xyz="0 0 0" rpy="0 0 0" />
-        <geometry>
-          <mesh
-            filename="package://duatic_dynaarm_description/meshes/${version}/${link01_mesh}"
-            scale="1 1 1" />
-        </geometry>
-      </collision>
-    </xacro:property>
-    <xacro:property name="link02_collision">
-      <collision>
-        <origin xyz="0 0 0" rpy="0 0 0" />
-        <geometry>
-          <mesh
-            filename="package://duatic_dynaarm_description/meshes/${version}/${link02_mesh}"
-            scale="1 1 1" />
-        </geometry>
-      </collision>
-    </xacro:property>
-    <xacro:property name="link03_collision">
-      <collision>
-        <origin xyz="0 0 0" rpy="0 0 0" />
-        <geometry>
-          <mesh
-            filename="package://duatic_dynaarm_description/meshes/${version}/${link03_mesh}"
-            scale="1 1 1" />
-        </geometry>
-      </collision>
-    </xacro:property>
-    <xacro:property name="link04_collision">
-      <collision>
-        <origin xyz="0 0 0" rpy="0 0 0" />
-        <geometry>
-          <mesh
-            filename="package://duatic_dynaarm_description/meshes/${version}/${link04_mesh}"
-            scale="1 1 1" />
-        </geometry>
-      </collision>
-    </xacro:property>
-    <xacro:property name="link05_collision">
-      <collision>
-        <origin xyz="0 0 0" rpy="0 0 0" />
-        <geometry>
-          <mesh
-            filename="package://duatic_dynaarm_description/meshes/${version}/${link05_mesh}"
-            scale="1 1 1" />
-        </geometry>
-      </collision>
-    </xacro:property>
-    <xacro:property name="link06_collision">
-      <collision>
-        <origin xyz="0 0 0" rpy="0 0 0" />
-        <geometry>
-          <mesh
-            filename="package://duatic_dynaarm_description/meshes/${version}/${link06_mesh}"
-            scale="1 1 1" />
-        </geometry>
-      </collision>
-    </xacro:property>
-  </xacro:if>
-  <!-- Set the ee_parent -->
-  <xacro:property name="ee_parent" value="${link06}" />
+  <!-- corydoras12 uses the baracuda12 parameters; only the meshes differ -->
+  <xacro:include filename="$(find duatic_dynaarm_description)/urdf/common/baracuda12/dynaarm_parameters.urdf.xacro" />
 </robot>

File: duatic_dynaarm_description/urdf/dynaarm.urdf.xacro (robot description, xacro)
@@ -30,5 +30,4 @@
       *origin">
     <xacro:include filename="$(find duatic_dynaarm_description)/urdf/common/dynaarm_common.urdf.xacro" />
-    <!-- Include the version specific information and also load the ethercat addresses from the drive file -->
     <xacro:include filename="$(find duatic_dynaarm_description)/urdf/common/${version}/dynaarm_parameters.urdf.xacro" />
     <!-- Per joint velocity and effort limits that replace the defaults -->
@@ -190,5 +189,5 @@
     <xacro:virtual_link link_name="${end_effector}" />
     <xacro:dynaarm_joint_fixed joint_name="${joint_ee_name}"
-      parent="${ee_parent}"
+      parent="${link06}"
       child="${end_effector}">
       <origin xyz="${joint_ee_origin_xyz}" rpy="${joint_ee_origin_rpy}" />

Commit message: refactor(description): build mesh collisions in dynaarm_link
With collision:=complex every link reused its own visual mesh as
collision geometry, written out as seven near-identical properties.
dynaarm_link now emits that collision itself from the mesh it already
renders, and the parameters file only defines the simple shapes, which
are always available and indented like the rest of the file. Rendered
URDFs are byte-identical to the previous commit.

File: duatic_dynaarm_description/urdf/common/baracuda12/dynaarm_parameters.urdf.xacro (robot description, xacro)
@@ -182,136 +182,60 @@
     </inertial>
   </xacro:property>
- <xacro:if value="${collision == 'simple'}">
-    <!-- Collision properties -->
-    <xacro:property name="base_collision">
-        <collision>
-            <geometry>
-                <cylinder length='0.1' radius='0.075'/>
-            </geometry>
-            <origin xyz='0 0 0.05' rpy='0 0 0'/>
-        </collision>
-    </xacro:property>
-    <xacro:property name="link01_collision">
-          <collision>
-              <geometry>
-                  <cylinder length='0.25' radius='0.06'/>
-              </geometry>
-              <origin xyz='0 0 0.05' rpy='${J_PI/2} 0 0'/>
-          </collision>
-    </xacro:property>
-    <xacro:property name="link02_collision">
-          <collision>
-              <geometry>
-                  <cylinder length='0.4' radius='0.05'/>
-              </geometry>
-              <origin xyz='0.15 0 0' rpy='0 ${J_PI/2} 0'/>
-          </collision>
-    </xacro:property>
-    <xacro:property name="link03_collision">
-      <collision>
-          <geometry>
-              <cylinder length='0.2' radius='0.065'/>
-          </geometry>
-          <origin xyz='-0.01 -0.05 0' rpy='${J_PI/2} 0 0'/>
-      </collision>
-    </xacro:property>
-    <xacro:property name="link04_collision">
-      <collision>
-          <geometry>
-              <cylinder length='0.4' radius='0.04'/>
-          </geometry>
-          <origin xyz='0 0 0.2' rpy='0 0 0'/>
-      </collision>
-    </xacro:property>
-    <xacro:property name="link05_collision">
-      <collision>
-          <geometry>
-              <cylinder length='0.125' radius='0.05'/>
-          </geometry>
-          <origin xyz='0 0 0.025' rpy='0 0 ${J_PI/2}'/>
-      </collision>
-    </xacro:property>
-    <xacro:property name="link06_collision">
-      <collision>
-          <geometry>
-              <cylinder length='0.09' radius='0.052'/>
-          </geometry>
-          <origin xyz='0.005 0 -0.035' rpy='0 0 0'/>
-      </collision>
-    </xacro:property>
-  </xacro:if>
-  <xacro:if value="${collision == 'complex'}">
-    <!-- Collision properties: reuse the visual meshes (base_mesh already resolves to the
-         standalone/attached variant) instead of the separate collision_meshes/*.stl files -->
-    <xacro:property name="base_collision">
-      <collision>
-        <origin xyz="0 0 0" rpy="0 0 0" />
-        <geometry>
-          <mesh
-            filename="package://duatic_dynaarm_description/meshes/${version}/${base_mesh}"
-            scale="1 1 1" />
-        </geometry>
-      </collision>
-    </xacro:property>
-    <xacro:property name="link01_collision">
-      <collision>
-        <origin xyz="0 0 0" rpy="0 0 0" />
-        <geometry>
-          <mesh
-            filename="package://duatic_dynaarm_description/meshes/${version}/${link01_mesh}"
-            scale="1 1 1" />
-        </geometry>
-      </collision>
-    </xacro:property>
-    <xacro:property name="link02_collision">
-      <collision>
-        <origin xyz="0 0 0" rpy="0 0 0" />
-        <geometry>
-          <mesh
-            filename="package://duatic_dynaarm_description/meshes/${version}/${link02_mesh}"
-            scale="1 1 1" />
-        </geometry>
-      </collision>
-    </xacro:property>
-    <xacro:property name="link03_collision">
-      <collision>
-        <origin xyz="0 0 0" rpy="0 0 0" />
-        <geometry>
-          <mesh
-            filename="package://duatic_dynaarm_description/meshes/${version}/${link03_mesh}"
-            scale="1 1 1" />
-        </geometry>
-      </collision>
-    </xacro:property>
-    <xacro:property name="link04_collision">
-      <collision>
-        <origin xyz="0 0 0" rpy="0 0 0" />
-        <geometry>
-          <mesh
-            filename="package://duatic_dynaarm_description/meshes/${version}/${link04_mesh}"
-            scale="1 1 1" />
-        </geometry>
-      </collision>
-    </xacro:property>
-    <xacro:property name="link05_collision">
-      <collision>
-        <origin xyz="0 0 0" rpy="0 0 0" />
-        <geometry>
-          <mesh
-            filename="package://duatic_dynaarm_description/meshes/${version}/${link05_mesh}"
-            scale="1 1 1" />
-        </geometry>
-      </collision>
-    </xacro:property>
-    <xacro:property name="link06_collision">
-      <collision>
-        <origin xyz="0 0 0" rpy="0 0 0" />
-        <geometry>
-          <mesh
-            filename="package://duatic_dynaarm_description/meshes/${version}/${link06_mesh}"
-            scale="1 1 1" />
-        </geometry>
-      </collision>
-    </xacro:property>
-  </xacro:if>
+  <!-- Collision geometry for collision:=simple; collision:=complex reuses the visual meshes -->
+  <xacro:property name="base_collision">
+    <collision>
+      <geometry>
+        <cylinder length='0.1' radius='0.075'/>
+      </geometry>
+      <origin xyz='0 0 0.05' rpy='0 0 0'/>
+    </collision>
+  </xacro:property>
+  <xacro:property name="link01_collision">
+    <collision>
+      <geometry>
+        <cylinder length='0.25' radius='0.06'/>
+      </geometry>
+      <origin xyz='0 0 0.05' rpy='${J_PI/2} 0 0'/>
+    </collision>
+  </xacro:property>
+  <xacro:property name="link02_collision">
+    <collision>
+      <geometry>
+        <cylinder length='0.4' radius='0.05'/>
+      </geometry>
+      <origin xyz='0.15 0 0' rpy='0 ${J_PI/2} 0'/>
+    </collision>
+  </xacro:property>
+  <xacro:property name="link03_collision">
+    <collision>
+      <geometry>
+        <cylinder length='0.2' radius='0.065'/>
+      </geometry>
+      <origin xyz='-0.01 -0.05 0' rpy='${J_PI/2} 0 0'/>
+    </collision>
+  </xacro:property>
+  <xacro:property name="link04_collision">
+    <collision>
+      <geometry>
+        <cylinder length='0.4' radius='0.04'/>
+      </geometry>
+      <origin xyz='0 0 0.2' rpy='0 0 0'/>
+    </collision>
+  </xacro:property>
+  <xacro:property name="link05_collision">
+    <collision>
+      <geometry>
+        <cylinder length='0.125' radius='0.05'/>
+      </geometry>
+      <origin xyz='0 0 0.025' rpy='0 0 ${J_PI/2}'/>
+    </collision>
+  </xacro:property>
+  <xacro:property name="link06_collision">
+    <collision>
+      <geometry>
+        <cylinder length='0.09' radius='0.052'/>
+      </geometry>
+      <origin xyz='0.005 0 -0.035' rpy='0 0 0'/>
+    </collision>
+  </xacro:property>
 </robot>

File: duatic_dynaarm_description/urdf/common/dynaarm_common.urdf.xacro (robot description, xacro)
@@ -41,5 +41,17 @@
             </visual>
             <xacro:insert_block name="link_inertia" />
-            <xacro:insert_block name="link_collision" />
+            <xacro:if value="${collision == 'simple'}">
+                <xacro:insert_block name="link_collision" />
+            </xacro:if>
+            <xacro:if value="${collision == 'complex'}">
+                <collision>
+                    <origin xyz="0 0 0" rpy="0 0 0" />
+                    <geometry>
+                        <mesh
+                            filename="package://duatic_dynaarm_description/meshes/${version}/${file_name}"
+                            scale="1 1 1" />
+                    </geometry>
+                </collision>
+            </xacro:if>
         </link>
     </xacro:macro>
