Commit message: refactor(description): fix arm joint type to revolute
Every arm joint passed joint_type=revolute through a per-joint property.
dynaarm_revolute_joint now emits the type itself and the six
joint_N_joint_type properties are gone. Rendered URDFs are
byte-identical.

File: duatic_dynaarm_description/urdf/common/baracuda12/dynaarm_parameters.urdf.xacro (robot description, xacro)
@@ -44,5 +44,4 @@
   <xacro:property name="joint_base_name" value="${tf_prefix}joint_base" />
   <xacro:property name="joint_1_name" value="${tf_prefix}shoulder_rotation" />
-  <xacro:property name="joint_1_joint_type" value="revolute" />
   <xacro:property name="joint_1_axis_xyz" value="0 0 1" />
   <xacro:property name="joint_1_origin_xyz" value="0 0 0.1105" />
@@ -53,5 +52,4 @@
   <xacro:property name="joint_1_limit_effort" value="120.0" />
   <xacro:property name="joint_2_name" value="${tf_prefix}shoulder_flexion" />
-  <xacro:property name="joint_2_joint_type" value="revolute" />
   <xacro:property name="joint_2_axis_xyz" value="0 0 1" />
   <xacro:property name="joint_2_origin_xyz" value="0 0 0.047" />
@@ -62,5 +60,4 @@
   <xacro:property name="joint_2_limit_effort" value="120.0" />
   <xacro:property name="joint_3_name" value="${tf_prefix}elbow_flexion" />
-  <xacro:property name="joint_3_joint_type" value="revolute" />
   <xacro:property name="joint_3_axis_xyz" value="0 0 1" />
   <xacro:property name="joint_3_origin_xyz" value="0.4127 0 0" />
@@ -74,5 +71,4 @@
   <xacro:property name="joint_3_cam_origin_rpy" value="0.0 0.0 0.0" />
   <xacro:property name="joint_4_name" value="${tf_prefix}forearm_rotation" />
-  <xacro:property name="joint_4_joint_type" value="revolute" />
   <xacro:property name="joint_4_axis_xyz" value="0 0 1" />
   <xacro:property name="joint_4_origin_xyz" value="0.0262 -0.0855 0" />
@@ -83,5 +79,4 @@
   <xacro:property name="joint_4_limit_effort" value="40.0" />
   <xacro:property name="joint_5_name" value="${tf_prefix}wrist_flexion" />
-  <xacro:property name="joint_5_joint_type" value="revolute" />
   <xacro:property name="joint_5_axis_xyz" value="0 0 1" />
   <xacro:property name="joint_5_origin_xyz" value="0.0295 0 0.4207" />
@@ -95,5 +90,4 @@
   <xacro:property name="joint_5_cam_origin_rpy" value="0.0 0.0 0.0" />
   <xacro:property name="joint_6_name" value="${tf_prefix}wrist_rotation" />
-  <xacro:property name="joint_6_joint_type" value="revolute" />
   <xacro:property name="joint_6_axis_xyz" value="0 0 1" />
   <xacro:property name="joint_6_origin_xyz" value="0.117 0.0 0.0295" />

File: duatic_dynaarm_description/urdf/common/dynaarm_common.urdf.xacro (robot description, xacro)
@@ -94,5 +94,4 @@
                 joint_limit_vel
                 joint_limit_effort
-                joint_type
                 *origin">
         <!-- joint_limits overrides the default velocity and effort per joint -->
@@ -100,5 +99,5 @@
         <xacro:property name="effort" value="${limits.get('max_effort', joint_limit_effort)}" />
         <xacro:property name="velocity" value="${limits.get('max_velocity', joint_limit_vel)}" />
-        <joint name="${joint_name}" type="${joint_type}">
+        <joint name="${joint_name}" type="revolute">
             <parent link="${parent}" />
             <child link="${child}" />

File: duatic_dynaarm_description/urdf/dynaarm.urdf.xacro (robot description, xacro)
@@ -64,6 +64,5 @@
       joint_upper_limit="${joint_1_upper_limit}"
       joint_limit_vel="${joint_1_limit_vel}"
-      joint_limit_effort="${joint_1_limit_effort}"
-      joint_type="${joint_1_joint_type}">
+      joint_limit_effort="${joint_1_limit_effort}">
       <origin xyz="${joint_1_origin_xyz}" rpy="${joint_1_origin_rpy}" />
     </xacro:dynaarm_revolute_joint>
@@ -85,6 +84,5 @@
       joint_upper_limit="${joint_2_upper_limit}"
       joint_limit_vel="${joint_2_limit_vel}"
-      joint_limit_effort="${joint_2_limit_effort}"
-      joint_type="${joint_2_joint_type}">
+      joint_limit_effort="${joint_2_limit_effort}">
       <origin xyz="${joint_2_origin_xyz}" rpy="${joint_2_origin_rpy}" />
     </xacro:dynaarm_revolute_joint>
@@ -106,6 +104,5 @@
       joint_upper_limit="${joint_3_upper_limit}"
       joint_limit_vel="${joint_3_limit_vel}"
-      joint_limit_effort="${joint_3_limit_effort}"
-      joint_type="${joint_3_joint_type}">
+      joint_limit_effort="${joint_3_limit_effort}">
       <origin xyz="${joint_3_origin_xyz}" rpy="${joint_3_origin_rpy}" />
     </xacro:dynaarm_revolute_joint>
@@ -134,6 +131,5 @@
       joint_upper_limit="${joint_4_upper_limit}"
       joint_limit_vel="${joint_4_limit_vel}"
-      joint_limit_effort="${joint_4_limit_effort}"
-      joint_type="${joint_4_joint_type}">
+      joint_limit_effort="${joint_4_limit_effort}">
       <origin xyz="${joint_4_origin_xyz}" rpy="${joint_4_origin_rpy}" />
     </xacro:dynaarm_revolute_joint>
@@ -154,6 +150,5 @@
       joint_upper_limit="${joint_5_upper_limit}"
       joint_limit_vel="${joint_5_limit_vel}"
-      joint_limit_effort="${joint_5_limit_effort}"
-      joint_type="${joint_5_joint_type}">
+      joint_limit_effort="${joint_5_limit_effort}">
       <origin xyz="${joint_5_origin_xyz}" rpy="${joint_5_origin_rpy}" />
     </xacro:dynaarm_revolute_joint>
@@ -182,6 +177,5 @@
       joint_upper_limit="${joint_6_upper_limit}"
       joint_limit_vel="${joint_6_limit_vel}"
-      joint_limit_effort="${joint_6_limit_effort}"
-      joint_type="${joint_6_joint_type}">
+      joint_limit_effort="${joint_6_limit_effort}">
       <origin xyz="${joint_6_origin_xyz}" rpy="${joint_6_origin_rpy}" />
     </xacro:dynaarm_revolute_joint>

Commit message: refactor(description): use xacro's built-in pi constant
Replace the hand-written J_PI property (3.14159265359) with xacro's
${pi}, which is available in every xacro expression. Rendered URDFs are
unchanged apart from the extra digits of precision in the angles.

File: duatic_dynaarm_description/urdf/common/baracuda12/dynaarm_parameters.urdf.xacro (robot description, xacro)
@@ -22,5 +22,4 @@
 -->
 <robot xmlns:xacro="http://www.ros.org/wiki/xacro">
-  <xacro:property name="J_PI" value="3.14159265359" />
   <!-- Links -->
   <xacro:property name="base" value="${tf_prefix}base" />
@@ -49,6 +48,6 @@
   <xacro:property name="joint_1_origin_xyz" value="0 0 0.1105" />
   <xacro:property name="joint_1_origin_rpy" value="0 0 0" />
-  <xacro:property name="joint_1_lower_limit" value="${-J_PI - J_PI/2 + 0.4}" />
-  <xacro:property name="joint_1_upper_limit" value="${J_PI + J_PI/2 - 0.4}" />
+  <xacro:property name="joint_1_lower_limit" value="${-pi - pi/2 + 0.4}" />
+  <xacro:property name="joint_1_upper_limit" value="${pi + pi/2 - 0.4}" />
   <xacro:property name="joint_1_limit_vel" value="10.64" />
   <xacro:property name="joint_1_limit_effort" value="120.0" />
@@ -57,7 +56,7 @@
   <xacro:property name="joint_2_axis_xyz" value="0 0 1" />
   <xacro:property name="joint_2_origin_xyz" value="0 0 0.047" />
-  <xacro:property name="joint_2_origin_rpy" value="${J_PI/2} ${-J_PI/2} 0" />
-  <xacro:property name="joint_2_lower_limit" value="${-J_PI/2 - 0.15}" />
-  <xacro:property name="joint_2_upper_limit" value="${J_PI/2 + 0.15}" />
+  <xacro:property name="joint_2_origin_rpy" value="${pi/2} ${-pi/2} 0" />
+  <xacro:property name="joint_2_lower_limit" value="${-pi/2 - 0.15}" />
+  <xacro:property name="joint_2_upper_limit" value="${pi/2 + 0.15}" />
   <xacro:property name="joint_2_limit_vel" value="10.64" />
   <xacro:property name="joint_2_limit_effort" value="120.0" />
@@ -68,5 +67,5 @@
   <xacro:property name="joint_3_origin_rpy" value="0 0 0" />
   <xacro:property name="joint_3_lower_limit" value="0.00" />
-  <xacro:property name="joint_3_upper_limit" value="${J_PI - 0.05}" />
+  <xacro:property name="joint_3_upper_limit" value="${pi - 0.05}" />
   <xacro:property name="joint_3_limit_vel" value="10.64" />
   <xacro:property name="joint_3_limit_effort" value="120.0" />
@@ -78,7 +77,7 @@
   <xacro:property name="joint_4_axis_xyz" value="0 0 1" />
   <xacro:property name="joint_4_origin_xyz" value="0.0262 -0.0855 0" />
-  <xacro:property name="joint_4_origin_rpy" value="${J_PI/2} ${J_PI/2} ${J_PI/2}" />
-  <xacro:property name="joint_4_lower_limit" value="${-J_PI - J_PI/2}" />
-  <xacro:property name="joint_4_upper_limit" value="${J_PI + J_PI/2}" />
+  <xacro:property name="joint_4_origin_rpy" value="${pi/2} ${pi/2} ${pi/2}" />
+  <xacro:property name="joint_4_lower_limit" value="${-pi - pi/2}" />
+  <xacro:property name="joint_4_upper_limit" value="${pi + pi/2}" />
   <xacro:property name="joint_4_limit_vel" value="13.647" />
   <xacro:property name="joint_4_limit_effort" value="40.0" />
@@ -87,7 +86,7 @@
   <xacro:property name="joint_5_axis_xyz" value="0 0 1" />
   <xacro:property name="joint_5_origin_xyz" value="0.0295 0 0.4207" />
-  <xacro:property name="joint_5_origin_rpy" value="0 ${-J_PI/2} 0" />
-  <xacro:property name="joint_5_lower_limit" value="${-J_PI/2 -0.25}" />
-  <xacro:property name="joint_5_upper_limit" value="${J_PI/2 + 0.25}" />
+  <xacro:property name="joint_5_origin_rpy" value="0 ${-pi/2} 0" />
+  <xacro:property name="joint_5_lower_limit" value="${-pi/2 -0.25}" />
+  <xacro:property name="joint_5_upper_limit" value="${pi/2 + 0.25}" />
   <xacro:property name="joint_5_limit_vel" value="13.647" />
   <xacro:property name="joint_5_limit_effort" value="40.0" />
@@ -99,12 +98,12 @@
   <xacro:property name="joint_6_axis_xyz" value="0 0 1" />
   <xacro:property name="joint_6_origin_xyz" value="0.117 0.0 0.0295" />
-  <xacro:property name="joint_6_origin_rpy" value="${-J_PI/2} ${J_PI/2} ${-J_PI/2}" />
-  <xacro:property name="joint_6_lower_limit" value="${-J_PI/2}" />
-  <xacro:property name="joint_6_upper_limit" value="${J_PI + J_PI/2}" />
+  <xacro:property name="joint_6_origin_rpy" value="${-pi/2} ${pi/2} ${-pi/2}" />
+  <xacro:property name="joint_6_lower_limit" value="${-pi/2}" />
+  <xacro:property name="joint_6_upper_limit" value="${pi + pi/2}" />
   <xacro:property name="joint_6_limit_vel" value="13.647" />
   <xacro:property name="joint_6_limit_effort" value="40.0" />
   <xacro:property name="joint_ee_name" value="${tf_prefix}flange_fix_joint" />
   <xacro:property name="joint_ee_origin_xyz" value="0.0 0.0 0.009" />
-  <xacro:property name="joint_ee_origin_rpy" value="0.0 0.0 ${J_PI/2}" />
+  <xacro:property name="joint_ee_origin_rpy" value="0.0 0.0 ${pi/2}" />
   <!-- Base Robot -->
   <xacro:property name="base_inertial">
@@ -196,5 +195,5 @@
         <cylinder length='0.25' radius='0.06'/>
       </geometry>
-      <origin xyz='0 0 0.05' rpy='${J_PI/2} 0 0'/>
+      <origin xyz='0 0 0.05' rpy='${pi/2} 0 0'/>
     </collision>
   </xacro:property>
@@ -204,5 +203,5 @@
         <cylinder length='0.4' radius='0.05'/>
       </geometry>
-      <origin xyz='0.15 0 0' rpy='0 ${J_PI/2} 0'/>
+      <origin xyz='0.15 0 0' rpy='0 ${pi/2} 0'/>
     </collision>
   </xacro:property>
@@ -212,5 +211,5 @@
         <cylinder length='0.2' radius='0.065'/>
       </geometry>
-      <origin xyz='-0.01 -0.05 0' rpy='${J_PI/2} 0 0'/>
+      <origin xyz='-0.01 -0.05 0' rpy='${pi/2} 0 0'/>
     </collision>
   </xacro:property>
@@ -228,5 +227,5 @@
         <cylinder length='0.125' radius='0.05'/>
       </geometry>
-      <origin xyz='0 0 0.025' rpy='0 0 ${J_PI/2}'/>
+      <origin xyz='0 0 0.025' rpy='0 0 ${pi/2}'/>
     </collision>
   </xacro:property>

Commit message: refactor(description): rename simple collision blocks to *_simplified
link_collision is only inserted for collision:=simple, since the complex
variant builds its collision from the visual mesh. Rename the macro block
parameter to link_collision_simplified and the per-link blocks to
<link>_collision_simplified so the names say which variant they serve.

File: duatic_dynaarm_description/urdf/common/baracuda12/dynaarm_parameters.urdf.xacro (robot description, xacro)
@@ -182,5 +182,5 @@
   </xacro:property>
   <!-- Collision geometry for collision:=simple; collision:=complex reuses the visual meshes -->
-  <xacro:property name="base_collision">
+  <xacro:property name="base_collision_simplified">
     <collision>
       <geometry>
@@ -190,5 +190,5 @@
     </collision>
   </xacro:property>
-  <xacro:property name="link01_collision">
+  <xacro:property name="link01_collision_simplified">
     <collision>
       <geometry>
@@ -198,5 +198,5 @@
     </collision>
   </xacro:property>
-  <xacro:property name="link02_collision">
+  <xacro:property name="link02_collision_simplified">
     <collision>
       <geometry>
@@ -206,5 +206,5 @@
     </collision>
   </xacro:property>
-  <xacro:property name="link03_collision">
+  <xacro:property name="link03_collision_simplified">
     <collision>
       <geometry>
@@ -214,5 +214,5 @@
     </collision>
   </xacro:property>
-  <xacro:property name="link04_collision">
+  <xacro:property name="link04_collision_simplified">
     <collision>
       <geometry>
@@ -222,5 +222,5 @@
     </collision>
   </xacro:property>
-  <xacro:property name="link05_collision">
+  <xacro:property name="link05_collision_simplified">
     <collision>
       <geometry>
@@ -230,5 +230,5 @@
     </collision>
   </xacro:property>
-  <xacro:property name="link06_collision">
+  <xacro:property name="link06_collision_simplified">
     <collision>
       <geometry>

File: duatic_dynaarm_description/urdf/common/dynaarm_common.urdf.xacro (robot description, xacro)
@@ -26,5 +26,5 @@
     <!-- -->
     <xacro:macro name="dynaarm_link"
-        params="link_name file_name **link_inertia **link_collision">
+        params="link_name file_name **link_inertia **link_collision_simplified">
         <link name="${link_name}">
             <visual>
@@ -35,5 +35,5 @@
             <xacro:insert_block name="link_inertia" />
             <xacro:if value="${collision == 'simple'}">
-                <xacro:insert_block name="link_collision" />
+                <xacro:insert_block name="link_collision_simplified" />
             </xacro:if>
             <xacro:if value="${collision == 'complex'}">

File: duatic_dynaarm_description/urdf/dynaarm.urdf.xacro (robot description, xacro)
@@ -43,7 +43,7 @@
         <xacro:insert_block name="base_inertial" />
       </link_inertia>
-      <link_collision>
-        <xacro:insert_block name="base_collision" />
-      </link_collision>
+      <link_collision_simplified>
+        <xacro:insert_block name="base_collision_simplified" />
+      </link_collision_simplified>
     </xacro:dynaarm_link>
     <!-- Link: Shoulder -->
@@ -52,7 +52,7 @@
         <xacro:insert_block name="link01_inertial" />
       </link_inertia>
-      <link_collision>
-        <xacro:insert_block name="link01_collision" />
-      </link_collision>
+      <link_collision_simplified>
+        <xacro:insert_block name="link01_collision_simplified" />
+      </link_collision_simplified>
     </xacro:dynaarm_link>
     <!-- Joint: Shoulder Rotation -->
@@ -73,7 +73,7 @@
         <xacro:insert_block name="link02_inertial" />
       </link_inertia>
-      <link_collision>
-        <xacro:insert_block name="link02_collision" />
-      </link_collision>
+      <link_collision_simplified>
+        <xacro:insert_block name="link02_collision_simplified" />
+      </link_collision_simplified>
     </xacro:dynaarm_link>
     <!-- Joint: Shoulder Flexion -->
@@ -94,7 +94,7 @@
         <xacro:insert_block name="link03_inertial" />
       </link_inertia>
-      <link_collision>
-        <xacro:insert_block name="link03_collision" />
-      </link_collision>
+      <link_collision_simplified>
+        <xacro:insert_block name="link03_collision_simplified" />
+      </link_collision_simplified>
     </xacro:dynaarm_link>
     <!-- Joint: Elbow Flexion -->
@@ -123,7 +123,7 @@
         <xacro:insert_block name="link04_inertial" />
       </link_inertia>
-      <link_collision>
-        <xacro:insert_block name="link04_collision" />
-      </link_collision>
+      <link_collision_simplified>
+        <xacro:insert_block name="link04_collision_simplified" />
+      </link_collision_simplified>
     </xacro:dynaarm_link>
     <!-- Joint: Forearm Rotation -->
@@ -143,7 +143,7 @@
         <xacro:insert_block name="link05_inertial" />
       </link_inertia>
-      <link_collision>
-        <xacro:insert_block name="link05_collision" />
-      </link_collision>
+      <link_collision_simplified>
+        <xacro:insert_block name="link05_collision_simplified" />
+      </link_collision_simplified>
     </xacro:dynaarm_link>
     <!-- Joint: Wrist Flexion -->
@@ -171,7 +171,7 @@
         <xacro:insert_block name="link06_inertial" />
       </link_inertia>
-      <link_collision>
-        <xacro:insert_block name="link06_collision" />
-      </link_collision>
+      <link_collision_simplified>
+        <xacro:insert_block name="link06_collision_simplified" />
+      </link_collision_simplified>
     </xacro:dynaarm_link>
     <!-- Joint: Wrist Rotation -->
