Commit message: feat(urdf): adapt limits for new wrist rotation cover (#10)

File: duatic_dynaarm_description/urdf/common/arowana4/dynaarm_parameters.urdf.xacro (robot description, xacro)
@@ -109,5 +109,5 @@
   <xacro:property name="joint_6_origin_xyz" value="0.12 0.0 0.03" />
   <xacro:property name="joint_6_origin_rpy" value="${-J_PI/2} 0 ${-J_PI/2}" />
-  <xacro:property name="joint_6_lower_limit" value="${-J_PI - J_PI/2}" />
+  <xacro:property name="joint_6_lower_limit" value="${-J_PI/2}" />
   <xacro:property name="joint_6_upper_limit" value="${J_PI + J_PI/2}" />
   <xacro:property name="joint_ee_name" value="${tf_prefix}flange_fix_joint" />

File: duatic_dynaarm_description/urdf/common/baracuda12/dynaarm_parameters.urdf.xacro (robot description, xacro)
@@ -121,5 +121,5 @@
   <xacro:property name="joint_6_origin_xyz" value="0.117 0.0 0.0295" />
   <xacro:property name="joint_6_origin_rpy" value="${-J_PI/2} ${J_PI/2} ${-J_PI/2}" />
-  <xacro:property name="joint_6_lower_limit" value="${-J_PI - J_PI/2}" />
+  <xacro:property name="joint_6_lower_limit" value="${-J_PI/2}" />
   <xacro:property name="joint_6_upper_limit" value="${J_PI + J_PI/2}" />
   <xacro:property name="joint_ee_name" value="${tf_prefix}flange_fix_joint" />
