Commit message: Include information if a specific arm version has brakes or not

File: duatic_dynaarm_driver/urdf/dynaarm.ros2control.xacro (robot description, xacro)
@@ -33,5 +33,6 @@
         dof
         ethercat_addresses
-        drive_parameter_folder:=''">
+        drive_parameter_folder:=''
+        has_brakes:=true">
       <!--Allow the user to pass a custom folder for drive parameters-->
       <xacro:property name="default_drive_parameter_folder" value="$(find duatic_dynaarm_driver)/config/${version}" />
@@ -48,5 +49,6 @@
           mode="${mode}"
           parent_unit="${parent_unit}"
-          drive_parameter_file_path="${drive_parameter_folder_internal}/shoulder_rotation.yaml" />
+          drive_parameter_file_path="${drive_parameter_folder_internal}/shoulder_rotation.yaml"
+          has_brake="${has_brakes}" />
       </xacro:if>
       <xacro:if value="${dof >= 2}">
@@ -56,5 +58,6 @@
           mode="${mode}"
           parent_unit="${parent_unit}"
-          drive_parameter_file_path="${drive_parameter_folder_internal}/shoulder_flexion.yaml" />
+          drive_parameter_file_path="${drive_parameter_folder_internal}/shoulder_flexion.yaml"
+          has_brake="${has_brakes}" />
       </xacro:if>
       <xacro:if value="${dof >= 3}">
@@ -64,5 +67,6 @@
           mode="${mode}"
           parent_unit="${parent_unit}"
-          drive_parameter_file_path="${drive_parameter_folder_internal}/elbow_flexion.yaml" />
+          drive_parameter_file_path="${drive_parameter_folder_internal}/elbow_flexion.yaml"
+          has_brake="${has_brakes}" />
       </xacro:if>
       <xacro:if value="${dof >= 4}">
@@ -72,5 +76,6 @@
           mode="${mode}"
           parent_unit="${parent_unit}"
-          drive_parameter_file_path="${drive_parameter_folder_internal}/forearm_rotation.yaml" />
+          drive_parameter_file_path="${drive_parameter_folder_internal}/forearm_rotation.yaml"
+          has_brake="${has_brakes}" />
       </xacro:if>
       <xacro:if value="${dof >= 5}">
@@ -80,5 +85,6 @@
           mode="${mode}"
           parent_unit="${parent_unit}"
-          drive_parameter_file_path="${drive_parameter_folder_internal}/wrist_flexion.yaml" />
+          drive_parameter_file_path="${drive_parameter_folder_internal}/wrist_flexion.yaml"
+          has_brake="${has_brakes}" />
       </xacro:if>
       <xacro:if value="${dof >= 6}">
@@ -88,5 +94,6 @@
           mode="${mode}"
           parent_unit="${parent_unit}"
-          drive_parameter_file_path="${drive_parameter_folder_internal}/wrist_rotation.yaml" />
+          drive_parameter_file_path="${drive_parameter_folder_internal}/wrist_rotation.yaml"
+          has_brake="${has_brakes}" />
       </xacro:if>
       <!--
@@ -135,4 +142,11 @@
         </xacro:if>
       </hardware>
+      <!--Make the assumption that all newer arms will have brakes (very likely)-->
+      <xacro:if value="${version in ['arowana4', 'baracuda12']}">
+        <xacro:property name="has_brakes" value="false"/>
+      </xacro:if>
+      <xacro:unless value="${version in ['arowana4', 'baracuda12']}">
+        <xacro:property name="has_brakes" value="true"/>
+      </xacro:unless>
       <xacro:dynaarm_ros2_control_joints
         tf_prefix="${tf_prefix}"
@@ -142,5 +156,6 @@
         parent_unit="${tf_prefix}DynaarmSystem"
         ethercat_addresses="${ethercat_addresses}"
-        dof="${dof}"/>
+        dof="${dof}"
+        has_brakes="${has_brakes}"/>
     </ros2_control>
   </xacro:macro>

Commit message: fix mistake made in last commit

File: duatic_dynaarm_driver/urdf/dynaarm.ros2control.xacro (robot description, xacro)
@@ -33,6 +33,12 @@
         dof
         ethercat_addresses
-        drive_parameter_folder:=''
-        has_brakes:=true">
+        drive_parameter_folder:=''">
+      <!--Make the assumption that all newer arms will have brakes (very likely)-->
+      <xacro:if value="${version in ['arowana4', 'baracuda12']}">
+        <xacro:property name="has_brakes" value="false"/>
+      </xacro:if>
+      <xacro:unless value="${version in ['arowana4', 'baracuda12']}">
+        <xacro:property name="has_brakes" value="true"/>
+      </xacro:unless>
       <!--Allow the user to pass a custom folder for drive parameters-->
       <xacro:property name="default_drive_parameter_folder" value="$(find duatic_dynaarm_driver)/config/${version}" />
@@ -142,11 +148,4 @@
         </xacro:if>
       </hardware>
-      <!--Make the assumption that all newer arms will have brakes (very likely)-->
-      <xacro:if value="${version in ['arowana4', 'baracuda12']}">
-        <xacro:property name="has_brakes" value="false"/>
-      </xacro:if>
-      <xacro:unless value="${version in ['arowana4', 'baracuda12']}">
-        <xacro:property name="has_brakes" value="true"/>
-      </xacro:unless>
       <xacro:dynaarm_ros2_control_joints
         tf_prefix="${tf_prefix}"
@@ -156,6 +155,5 @@
         parent_unit="${tf_prefix}DynaarmSystem"
         ethercat_addresses="${ethercat_addresses}"
-        dof="${dof}"
-        has_brakes="${has_brakes}"/>
+        dof="${dof}"/>
     </ros2_control>
   </xacro:macro>

Commit message: Include information if a specific arm version has brakes or not (#18)
* Include information if a specific arm version has brakes or not

* fix mistake made in last commit

* apply the same gains to corydoras as baracuda

File: duatic_dynaarm_driver/urdf/dynaarm.ros2control.xacro (robot description, xacro)
@@ -34,4 +34,11 @@
         ethercat_addresses
         drive_parameter_folder:=''">
+      <!--Make the assumption that all newer arms will have brakes (very likely)-->
+      <xacro:if value="${version in ['arowana4', 'baracuda12']}">
+        <xacro:property name="has_brakes" value="false"/>
+      </xacro:if>
+      <xacro:unless value="${version in ['arowana4', 'baracuda12']}">
+        <xacro:property name="has_brakes" value="true"/>
+      </xacro:unless>
       <!--Allow the user to pass a custom folder for drive parameters-->
       <xacro:property name="default_drive_parameter_folder" value="$(find duatic_dynaarm_driver)/config/${version}" />
@@ -48,5 +55,6 @@
           mode="${mode}"
           parent_unit="${parent_unit}"
-          drive_parameter_file_path="${drive_parameter_folder_internal}/shoulder_rotation.yaml" />
+          drive_parameter_file_path="${drive_parameter_folder_internal}/shoulder_rotation.yaml"
+          has_brake="${has_brakes}" />
       </xacro:if>
       <xacro:if value="${dof >= 2}">
@@ -56,5 +64,6 @@
           mode="${mode}"
           parent_unit="${parent_unit}"
-          drive_parameter_file_path="${drive_parameter_folder_internal}/shoulder_flexion.yaml" />
+          drive_parameter_file_path="${drive_parameter_folder_internal}/shoulder_flexion.yaml"
+          has_brake="${has_brakes}" />
       </xacro:if>
       <xacro:if value="${dof >= 3}">
@@ -64,5 +73,6 @@
           mode="${mode}"
           parent_unit="${parent_unit}"
-          drive_parameter_file_path="${drive_parameter_folder_internal}/elbow_flexion.yaml" />
+          drive_parameter_file_path="${drive_parameter_folder_internal}/elbow_flexion.yaml"
+          has_brake="${has_brakes}" />
       </xacro:if>
       <xacro:if value="${dof >= 4}">
@@ -72,5 +82,6 @@
           mode="${mode}"
           parent_unit="${parent_unit}"
-          drive_parameter_file_path="${drive_parameter_folder_internal}/forearm_rotation.yaml" />
+          drive_parameter_file_path="${drive_parameter_folder_internal}/forearm_rotation.yaml"
+          has_brake="${has_brakes}" />
       </xacro:if>
       <xacro:if value="${dof >= 5}">
@@ -80,5 +91,6 @@
           mode="${mode}"
           parent_unit="${parent_unit}"
-          drive_parameter_file_path="${drive_parameter_folder_internal}/wrist_flexion.yaml" />
+          drive_parameter_file_path="${drive_parameter_folder_internal}/wrist_flexion.yaml"
+          has_brake="${has_brakes}" />
       </xacro:if>
       <xacro:if value="${dof >= 6}">
@@ -88,5 +100,6 @@
           mode="${mode}"
           parent_unit="${parent_unit}"
-          drive_parameter_file_path="${drive_parameter_folder_internal}/wrist_rotation.yaml" />
+          drive_parameter_file_path="${drive_parameter_folder_internal}/wrist_rotation.yaml"
+          has_brake="${has_brakes}" />
       </xacro:if>
       <!--
