Commit message: feat: deprecate arowana4

File: duatic_dynaarm_description/urdf/dynaarm.urdf.xacro (robot description, xacro)
@@ -139,23 +139,13 @@
     <!-- 4 DoF -->
     <xacro:if value="${dof >= 4}">
-      <xacro:if value="${version == 'arowana4'}">
-        <!-- dynaarm_FOREARM -->
-        <xacro:dynaarm_link link_name="${link04}" file_name="${link04_mesh}">
-          <link_inertia>
-            <xacro:insert_block name="link04_inertial" />
-          </link_inertia>
-        </xacro:dynaarm_link>
-      </xacro:if>
-      <xacro:if value="${version == 'baracuda12' or version == 'corydoras12'}">
-        <!-- dynaarm_FOREARM -->
-        <xacro:dynaarm_link_w_collision link_name="${link04}" file_name="${link04_mesh}">
-          <link_inertia>
-            <xacro:insert_block name="link04_inertial" />
-          </link_inertia>
-          <link_collision>
-            <xacro:insert_block name="link04_collision" />
-          </link_collision>
-        </xacro:dynaarm_link_w_collision>
-      </xacro:if>
+      <!-- dynaarm_FOREARM -->
+      <xacro:dynaarm_link_w_collision link_name="${link04}" file_name="${link04_mesh}">
+        <link_inertia>
+          <xacro:insert_block name="link04_inertial" />
+        </link_inertia>
+        <link_collision>
+          <xacro:insert_block name="link04_collision" />
+        </link_collision>
+      </xacro:dynaarm_link_w_collision>
       <!-- forearm_rotation -->
       <xacro:dynaarm_revolute_joint joint_name="${joint_4_name}" parent="${link03}"
@@ -205,23 +195,13 @@
     <!-- 6 DoF -->
     <xacro:if value="${dof >= 6}">
-      <xacro:if value="${version == 'arowana4'}">
-        <!-- WRIST_2 -->
-        <xacro:dynaarm_link link_name="${link06}" file_name="${link06_mesh}">
-          <link_inertia>
-            <xacro:insert_block name="link06_inertial" />
-          </link_inertia>
-        </xacro:dynaarm_link>
-      </xacro:if>
-      <xacro:if value="${version == 'baracuda12' or version == 'corydoras12'}">
-        <!-- WRIST_2 -->
-        <xacro:dynaarm_link_w_collision link_name="${link06}" file_name="${link06_mesh}">
-          <link_inertia>
-            <xacro:insert_block name="link06_inertial" />
-          </link_inertia>
-          <link_collision>
-            <xacro:insert_block name="link06_collision" />
-          </link_collision>
-        </xacro:dynaarm_link_w_collision>
-      </xacro:if>
+      <!-- WRIST_2 -->
+      <xacro:dynaarm_link_w_collision link_name="${link06}" file_name="${link06_mesh}">
+        <link_inertia>
+          <xacro:insert_block name="link06_inertial" />
+        </link_inertia>
+        <link_collision>
+          <xacro:insert_block name="link06_collision" />
+        </link_collision>
+      </xacro:dynaarm_link_w_collision>
       <!-- wrist_rotation -->
       <xacro:dynaarm_revolute_joint joint_name="${joint_6_name}" parent="${link05}"

File: duatic_dynaarm_driver/urdf/dynaarm.ros2control.xacro (robot description, xacro)
@@ -35,10 +35,5 @@
         drive_parameter_folder:=''">
       <!--Make the assumption that all newer arms will have brakes (very likely)-->
-      <xacro:if value="${version in ['arowana4', 'baracuda12']}">
-        <xacro:property name="has_brakes" value="false"/>
-      </xacro:if>
-      <xacro:unless value="${version in ['arowana4', 'baracuda12']}">
-        <xacro:property name="has_brakes" value="true"/>
-      </xacro:unless>
+      <xacro:property name="has_brakes" value="${version not in ['baracuda12']}"/>
       <!--Allow the user to pass a custom folder for drive parameters-->
       <xacro:property name="default_drive_parameter_folder" value="$(find duatic_dynaarm_driver)/config/${version}" />

Commit message: fix(urdf): remove if clause that always results in true

File: duatic_dynaarm_description/urdf/dynaarm.urdf.xacro (robot description, xacro)
@@ -125,15 +125,12 @@
         <origin xyz="${joint_3_origin_xyz}" rpy="${joint_3_origin_rpy}" />
       </xacro:dynaarm_revolute_joint>
-      <!--dynaarm_ELBOW_CAMERA_BASE-->
-      <xacro:if value="${version == 'baracuda12' or version == 'corydoras12'}">
-        <!-- Virtual elbow camera link -->
-        <xacro:virtual_link link_name="${link03_cam}" />
-        <!-- Camera fixed on elbow -->
-        <xacro:dynaarm_joint_fixed joint_name="${joint_3_cam_name}"
-          parent="${link03}"
-          child="${link03_cam}">
-          <origin xyz="${joint_3_cam_origin_xyz}" rpy="${joint_3_cam_origin_rpy}" />
-        </xacro:dynaarm_joint_fixed>
-      </xacro:if>
+      <!-- Virtual elbow camera link -->
+      <xacro:virtual_link link_name="${link03_cam}" />
+      <!-- Camera fixed on elbow -->
+      <xacro:dynaarm_joint_fixed joint_name="${joint_3_cam_name}"
+        parent="${link03}"
+        child="${link03_cam}">
+        <origin xyz="${joint_3_cam_origin_xyz}" rpy="${joint_3_cam_origin_rpy}" />
+      </xacro:dynaarm_joint_fixed>
     </xacro:if>
     <!-- 4 DoF -->
@@ -182,14 +179,12 @@
         <origin xyz="${joint_5_origin_xyz}" rpy="${joint_5_origin_rpy}" />
       </xacro:dynaarm_revolute_joint>
-      <xacro:if value="${version == 'baracuda12' or version == 'corydoras12'}">
-        <!-- Virtual wrist camera link -->
-        <xacro:virtual_link link_name="${link05_cam}" />
-        <!-- Camera fixed on wrist1 -->
-        <xacro:dynaarm_joint_fixed joint_name="${joint_5_cam_name}"
-          parent="${link05}"
-          child="${link05_cam}">
-          <origin xyz="${joint_5_cam_origin_xyz}" rpy="${joint_5_cam_origin_rpy}" />
-        </xacro:dynaarm_joint_fixed>
-      </xacro:if>
+      <!-- Virtual wrist camera link -->
+      <xacro:virtual_link link_name="${link05_cam}" />
+      <!-- Camera fixed on wrist1 -->
+      <xacro:dynaarm_joint_fixed joint_name="${joint_5_cam_name}"
+        parent="${link05}"
+        child="${link05_cam}">
+        <origin xyz="${joint_5_cam_origin_xyz}" rpy="${joint_5_cam_origin_rpy}" />
+      </xacro:dynaarm_joint_fixed>
     </xacro:if>
     <!-- 6 DoF -->

Commit message: feat: deprecate arowana4 (#22)

File: duatic_dynaarm_description/urdf/dynaarm.urdf.xacro (robot description, xacro)
@@ -125,37 +125,24 @@
         <origin xyz="${joint_3_origin_xyz}" rpy="${joint_3_origin_rpy}" />
       </xacro:dynaarm_revolute_joint>
-      <!--dynaarm_ELBOW_CAMERA_BASE-->
-      <xacro:if value="${version == 'baracuda12' or version == 'corydoras12'}">
-        <!-- Virtual elbow camera link -->
-        <xacro:virtual_link link_name="${link03_cam}" />
-        <!-- Camera fixed on elbow -->
-        <xacro:dynaarm_joint_fixed joint_name="${joint_3_cam_name}"
-          parent="${link03}"
-          child="${link03_cam}">
-          <origin xyz="${joint_3_cam_origin_xyz}" rpy="${joint_3_cam_origin_rpy}" />
-        </xacro:dynaarm_joint_fixed>
-      </xacro:if>
+      <!-- Virtual elbow camera link -->
+      <xacro:virtual_link link_name="${link03_cam}" />
+      <!-- Camera fixed on elbow -->
+      <xacro:dynaarm_joint_fixed joint_name="${joint_3_cam_name}"
+        parent="${link03}"
+        child="${link03_cam}">
+        <origin xyz="${joint_3_cam_origin_xyz}" rpy="${joint_3_cam_origin_rpy}" />
+      </xacro:dynaarm_joint_fixed>
     </xacro:if>
     <!-- 4 DoF -->
     <xacro:if value="${dof >= 4}">
-      <xacro:if value="${version == 'arowana4'}">
-        <!-- dynaarm_FOREARM -->
-        <xacro:dynaarm_link link_name="${link04}" file_name="${link04_mesh}">
-          <link_inertia>
-            <xacro:insert_block name="link04_inertial" />
-          </link_inertia>
-        </xacro:dynaarm_link>
-      </xacro:if>
-      <xacro:if value="${version == 'baracuda12' or version == 'corydoras12'}">
-        <!-- dynaarm_FOREARM -->
-        <xacro:dynaarm_link_w_collision link_name="${link04}" file_name="${link04_mesh}">
-          <link_inertia>
-            <xacro:insert_block name="link04_inertial" />
-          </link_inertia>
-          <link_collision>
-            <xacro:insert_block name="link04_collision" />
-          </link_collision>
-        </xacro:dynaarm_link_w_collision>
-      </xacro:if>
+      <!-- dynaarm_FOREARM -->
+      <xacro:dynaarm_link_w_collision link_name="${link04}" file_name="${link04_mesh}">
+        <link_inertia>
+          <xacro:insert_block name="link04_inertial" />
+        </link_inertia>
+        <link_collision>
+          <xacro:insert_block name="link04_collision" />
+        </link_collision>
+      </xacro:dynaarm_link_w_collision>
       <!-- forearm_rotation -->
       <xacro:dynaarm_revolute_joint joint_name="${joint_4_name}" parent="${link03}"
@@ -192,36 +179,24 @@
         <origin xyz="${joint_5_origin_xyz}" rpy="${joint_5_origin_rpy}" />
       </xacro:dynaarm_revolute_joint>
-      <xacro:if value="${version == 'baracuda12' or version == 'corydoras12'}">
-        <!-- Virtual wrist camera link -->
-        <xacro:virtual_link link_name="${link05_cam}" />
-        <!-- Camera fixed on wrist1 -->
-        <xacro:dynaarm_joint_fixed joint_name="${joint_5_cam_name}"
-          parent="${link05}"
-          child="${link05_cam}">
-          <origin xyz="${joint_5_cam_origin_xyz}" rpy="${joint_5_cam_origin_rpy}" />
-        </xacro:dynaarm_joint_fixed>
-      </xacro:if>
+      <!-- Virtual wrist camera link -->
+      <xacro:virtual_link link_name="${link05_cam}" />
+      <!-- Camera fixed on wrist1 -->
+      <xacro:dynaarm_joint_fixed joint_name="${joint_5_cam_name}"
+        parent="${link05}"
+        child="${link05_cam}">
+        <origin xyz="${joint_5_cam_origin_xyz}" rpy="${joint_5_cam_origin_rpy}" />
+      </xacro:dynaarm_joint_fixed>
     </xacro:if>
     <!-- 6 DoF -->
     <xacro:if value="${dof >= 6}">
-      <xacro:if value="${version == 'arowana4'}">
-        <!-- WRIST_2 -->
-        <xacro:dynaarm_link link_name="${link06}" file_name="${link06_mesh}">
-          <link_inertia>
-            <xacro:insert_block name="link06_inertial" />
-          </link_inertia>
-        </xacro:dynaarm_link>
-      </xacro:if>
-      <xacro:if value="${version == 'baracuda12' or version == 'corydoras12'}">
-        <!-- WRIST_2 -->
-        <xacro:dynaarm_link_w_collision link_name="${link06}" file_name="${link06_mesh}">
-          <link_inertia>
-            <xacro:insert_block name="link06_inertial" />
-          </link_inertia>
-          <link_collision>
-            <xacro:insert_block name="link06_collision" />
-          </link_collision>
-        </xacro:dynaarm_link_w_collision>
-      </xacro:if>
+      <!-- WRIST_2 -->
+      <xacro:dynaarm_link_w_collision link_name="${link06}" file_name="${link06_mesh}">
+        <link_inertia>
+          <xacro:insert_block name="link06_inertial" />
+        </link_inertia>
+        <link_collision>
+          <xacro:insert_block name="link06_collision" />
+        </link_collision>
+      </xacro:dynaarm_link_w_collision>
       <!-- wrist_rotation -->
       <xacro:dynaarm_revolute_joint joint_name="${joint_6_name}" parent="${link05}"
