Commit message: fix(urdf): reduce forearm mass by 100g

File: duatic_dynaarm_description/urdf/common/corydoras12/dynaarm_parameters.urdf.xacro (robot description, xacro)
@@ -187,6 +187,5 @@
   <xacro:property name="link04_inertial">
     <inertial>
-      <!-- The mass here is 100g more than the value in CAD, but through testing we found out that freedrive works better with the increased value (09.12.25 Antonis & Marc)-->
-      <mass value="1.337246" />
+      <mass value="1.237246" />
       <origin xyz="-0.001568 0.000046 0.292163" rpy="0 0 0" />
       <inertia ixx="0.033872" iyy="0.033868"

Commit message: fixed shoulder

File: duatic_dynaarm_description/urdf/common/corydoras12/dynaarm_parameters.urdf.xacro (robot description, xacro)
@@ -56,5 +56,5 @@
   <xacro:property name="joint_1_joint_type" value="revolute" />
   <xacro:property name="joint_1_axis_xyz" value="0 0 1" />
-  <xacro:property name="joint_1_origin_xyz" value="0 0 0" />
+  <xacro:property name="joint_1_origin_xyz" value="0 0 0.1105" />
   <xacro:property name="joint_1_origin_rpy" value="0 0 0" />
   <xacro:property name="joint_1_lower_limit" value="${-J_PI - J_PI/2 + 0.4}" />
@@ -63,5 +63,5 @@
   <xacro:property name="joint_2_joint_type" value="revolute" />
   <xacro:property name="joint_2_axis_xyz" value="0 0 1" />
-  <xacro:property name="joint_2_origin_xyz" value="0 0 0.1575" />
+  <xacro:property name="joint_2_origin_xyz" value="0 0 0.047" />
   <xacro:property name="joint_2_origin_rpy" value="${J_PI/2} ${-J_PI/2} 0" />
   <xacro:property name="joint_2_lower_limit" value="${-J_PI/2 - 0.15}" />

Commit message: revert(description): revert indent change not part of this PR

File: duatic_dynaarm_description/urdf/common/corydoras12/dynaarm_parameters.urdf.xacro (robot description, xacro)
@@ -174,6 +174,5 @@
   <xacro:property name="link05_inertial">
     <inertial>
-      <!-- <mass value="0.75007482" />  original value but doesn't work well - Needs to include the
-      cables inside the forearm tube?-->
+      <!-- <mass value="0.75007482" />  original value but doesn't work well - Needs to include the cables inside the forearm tube?-->
       <mass value="1.15007482" />
       <origin xyz="0.07972553 -0.00005038 0.02334747" rpy="0 0 0" />
@@ -203,60 +202,60 @@
     </inertial>
   </xacro:property>
-  <xacro:if value="${collision == 'simple'}">
+ <xacro:if value="${collision == 'simple'}">
     <!-- Collision properties -->
     <xacro:property name="base_collision">
-      <collision>
-        <geometry>
-          <cylinder length='0.1' radius='0.075' />
-        </geometry>
-        <origin xyz='0 0 0.05' rpy='0 0 0' />
-      </collision>
+        <collision>
+            <geometry>
+                <cylinder length='0.1' radius='0.075'/>
+            </geometry>
+            <origin xyz='0 0 0.05' rpy='0 0 0'/>
+        </collision>
     </xacro:property>
     <xacro:property name="link01_collision">
-      <collision>
-        <geometry>
-          <cylinder length='0.25' radius='0.06' />
-        </geometry>
-        <origin xyz='0 0 0.05' rpy='${J_PI/2} 0 0' />
-      </collision>
+          <collision>
+              <geometry>
+                  <cylinder length='0.25' radius='0.06'/>
+              </geometry>
+              <origin xyz='0 0 0.05' rpy='${J_PI/2} 0 0'/>
+          </collision>
     </xacro:property>
     <xacro:property name="link02_collision">
-      <collision>
-        <geometry>
-          <cylinder length='0.4' radius='0.05' />
-        </geometry>
-        <origin xyz='0.15 0 0' rpy='0 ${J_PI/2} 0' />
-      </collision>
+          <collision>
+              <geometry>
+                  <cylinder length='0.4' radius='0.05'/>
+              </geometry>
+              <origin xyz='0.15 0 0' rpy='0 ${J_PI/2} 0'/>
+          </collision>
     </xacro:property>
     <xacro:property name="link03_collision">
       <collision>
-        <geometry>
-          <cylinder length='0.2' radius='0.065' />
-        </geometry>
-        <origin xyz='-0.01 -0.05 0' rpy='${J_PI/2} 0 0' />
+          <geometry>
+              <cylinder length='0.2' radius='0.065'/>
+          </geometry>
+          <origin xyz='-0.01 -0.05 0' rpy='${J_PI/2} 0 0'/>
       </collision>
     </xacro:property>
     <xacro:property name="link04_collision">
       <collision>
-        <geometry>
-          <cylinder length='0.4' radius='0.04' />
-        </geometry>
-        <origin xyz='0 0 0.2' rpy='0 0 0' />
+          <geometry>
+              <cylinder length='0.4' radius='0.04'/>
+          </geometry>
+          <origin xyz='0 0 0.2' rpy='0 0 0'/>
       </collision>
     </xacro:property>
     <xacro:property name="link05_collision">
       <collision>
-        <geometry>
-          <cylinder length='0.125' radius='0.05' />
-        </geometry>
-        <origin xyz='0 0 0.025' rpy='0 0 ${J_PI/2}' />
+          <geometry>
+              <cylinder length='0.125' radius='0.05'/>
+          </geometry>
+          <origin xyz='0 0 0.025' rpy='0 0 ${J_PI/2}'/>
       </collision>
     </xacro:property>
     <xacro:property name="link06_collision">
       <collision>
-        <geometry>
-          <cylinder length='0.09' radius='0.052' />
-        </geometry>
-        <origin xyz='0.005 0 -0.035' rpy='0 0 0' />
+          <geometry>
+              <cylinder length='0.09' radius='0.052'/>
+          </geometry>
+          <origin xyz='0.005 0 -0.035' rpy='0 0 0'/>
       </collision>
     </xacro:property>
