Commit message: feat(): deleted the option to enable/disable covers

File: duatic_dynaarm_demo/duatic_dynaarm_single_example/duatic_dynaarm_single_example_description/urdf/dynaarm_single_example.urdf.xacro (robot description, xacro)
@@ -18,6 +18,4 @@
   <!-- physical ethercat bus, only used for real -->
   <xacro:arg name="ethercat_bus" default="eth0" />
-  <!-- Change to add covers to the arm -->
-  <xacro:arg name="covers" default="false" />
   <!-- v1, v2, ... -->
   <xacro:arg name="version" default="baracuda12" />
@@ -59,5 +57,4 @@
                 mode="$(arg mode)"
                 ethercat_bus="$(arg ethercat_bus)"
-                covers="$(arg covers)"
                 version="$(arg version)">
     <origin xyz="0 0 0" rpy="0.0 0.0 0.0" />

File: duatic_dynaarm_description/urdf/common/arowana4/dynaarm_parameters.urdf.xacro (robot description, xacro)
@@ -38,29 +38,11 @@
   <xacro:property name="end_effector" value="${tf_prefix}flange" />
   <!-- Meshes -->
-  <xacro:if value="${covers}">
-    <xacro:property name="base_mesh" value="base_mesh.dae" />
-    <xacro:property name="link01_mesh" value="shoulder_mesh.dae" />
-    <xacro:property name="link02_mesh" value="upperarm_mesh.dae" />
-    <xacro:property name="link03_mesh" value="elbow_mesh.dae" />
-    <xacro:property name="link04_mesh" value="forearm_mesh.dae" />
-    <xacro:property name="link05_mesh" value="wrist1_mesh.dae" />
-    <xacro:property name="link06_mesh" value="wrist2_mesh.dae" />
-    <xacro:property name="base_cover_mesh" value="base_cover_mesh.dae" />
-    <xacro:property name="link01_cover_mesh" value="shoulder_cover_mesh.dae" />
-    <xacro:property name="link02_cover_mesh" value="upperarm_cover_mesh.dae" />
-    <xacro:property name="link03_cover_mesh" value="elbow_cover_mesh.dae" />
-    <xacro:property name="link04_cover_mesh" value="forearm_cover_mesh.dae" />
-    <xacro:property name="link05_cover_mesh" value="wrist_1_cover_mesh.dae" />
-    <xacro:property name="link06_cover_mesh" value="wrist_2_cover_mesh.dae" />
-  </xacro:if>
-  <xacro:unless value="${covers}">
-    <xacro:property name="base_mesh" value="base_detailed_mesh.dae" />
-    <xacro:property name="link01_mesh" value="shoulder_detailed_mesh.dae" />
-    <xacro:property name="link02_mesh" value="upperarm_detailed_mesh.dae" />
-    <xacro:property name="link03_mesh" value="elbow_detailed_mesh.dae" />
-    <xacro:property name="link04_mesh" value="forearm_detailed_mesh.dae" />
-    <xacro:property name="link05_mesh" value="wrist1_detailed_mesh.dae" />
-    <xacro:property name="link06_mesh" value="wrist2_detailed_mesh.dae" />
-  </xacro:unless>
+  <xacro:property name="base_mesh" value="base_detailed_mesh.dae" />
+  <xacro:property name="link01_mesh" value="shoulder_detailed_mesh.dae" />
+  <xacro:property name="link02_mesh" value="upperarm_detailed_mesh.dae" />
+  <xacro:property name="link03_mesh" value="elbow_detailed_mesh.dae" />
+  <xacro:property name="link04_mesh" value="forearm_detailed_mesh.dae" />
+  <xacro:property name="link05_mesh" value="wrist1_detailed_mesh.dae" />
+  <xacro:property name="link06_mesh" value="wrist2_detailed_mesh.dae" />
   <!-- Joint properties -->
   <xacro:property name="joint_base_name" value="${tf_prefix}joint_base" />
@@ -185,53 +167,4 @@
     </inertial>
   </xacro:property>
-  <!-- Covers -->
-  <xacro:property name="base_cover_inertial">
-    <inertial>
-      <mass value="0.098" />
-      <origin xyz="${0.0*mm_to_m} ${0.0*mm_to_m} ${-60.7*mm_to_m}" rpy="0 0 0" />
-      <inertia ixx="${0.000349}" iyy="${0.000338}" izz="${0.000649}" ixy="${0.000000018}"
-        ixz="${-0.000000001}" iyz="${-0.000000002}" />
-    </inertial>
-  </xacro:property>
-  <xacro:property name="link01_cover_inertial">
-    <inertial>
-      <mass value="0.135" />
-      <origin xyz="${-0.039*mm_to_m} ${-0.015*mm_to_m} ${-31.709*mm_to_m}" rpy="0 0 0" />
-      <inertia ixx="${0.00068}" iyy="${0.000517}" izz="${0.000646}" ixy="${-0.000000318}"
-        ixz="${-0.000000206}" iyz="${-0.000000074}" />
-    </inertial>
-  </xacro:property>
-  <xacro:property name="link02_cover_inertial">
-    <inertial>
-      <mass value="0.743" />
-      <origin xyz="${167.97*mm_to_m} ${0.081*mm_to_m} ${0.0*mm_to_m}" rpy="0 0 0" />
-      <inertia ixx="${0.0054}" iyy="${0.025}" izz="${0.0293}" ixy="${-0.000004814}"
-        ixz="${-0.000000101}" iyz="${0.000000134}" />
-    </inertial>
-  </xacro:property>
-  <xacro:property name="link03_cover_inertial">
-    <inertial>
-      <mass value="0.383" />
-      <origin xyz="${37.807*mm_to_m} ${-101.52*mm_to_m} ${0.184*mm_to_m}" rpy="0 0 0" />
-      <inertia ixx="${0.00139}" iyy="${0.00176}" izz="${0.00225}" ixy="${-0.000150269}"
-        ixz="${0.000002221}" iyz="${-0.000003993}" />
-    </inertial>
-  </xacro:property>
-  <xacro:property name="link04_cover_inertial">
-    <inertial>
-      <mass value="0.158" />
-      <origin xyz="${-9.28*mm_to_m} ${-0.008*mm_to_m} ${377.34*mm_to_m}" rpy="0 0 0" />
-      <inertia ixx="${0.000594}" iyy="${0.000846}" izz="${0.000485}" ixy="${-0.000000100}"
-        ixz="${-0.000057116}" iyz="${0.000000128}" />
-    </inertial>
-  </xacro:property>
-  <xacro:property name="link05_cover_inertial">
-    <inertial>
-      <mass value="0.121" />
-      <origin xyz="${54.24*mm_to_m} ${-0.0012*mm_to_m} ${-0.0069*mm_to_m}" rpy="0 0 0" />
-      <inertia ixx="${0.0003}" iyy="${0.00049}" izz="${0.00053}" ixy="${-0.000000004}"
-        ixz="${0.0}" iyz="${-0.000000043}" />
-    </inertial>
-  </xacro:property>
   <!-- Collision properties -->
   <xacro:property name="base_collision">

File: duatic_dynaarm_description/urdf/common/baracuda12/dynaarm_parameters.urdf.xacro (robot description, xacro)
@@ -40,29 +40,11 @@
   <xacro:property name="end_effector" value="${tf_prefix}flange" />
   <!-- Meshes -->
-  <xacro:if value="${covers}">
-    <xacro:property name="base_mesh" value="base_mesh.dae" />
-    <xacro:property name="link01_mesh" value="shoulder_mesh.dae" />
-    <xacro:property name="link02_mesh" value="upperarm_mesh.dae" />
-    <xacro:property name="link03_mesh" value="elbow_mesh.dae" />
-    <xacro:property name="link04_mesh" value="forearm_mesh.dae" />
-    <xacro:property name="link05_mesh" value="wrist1_mesh.dae" />
-    <xacro:property name="link06_mesh" value="wrist2_mesh.dae" />
-    <xacro:property name="base_cover_mesh" value="base_mesh.dae" />
-    <xacro:property name="link01_cover_mesh" value="shoulder_mesh.dae" />
-    <xacro:property name="link02_cover_mesh" value="upperarm_mesh.dae" />
-    <xacro:property name="link03_cover_mesh" value="elbow_mesh.dae" />
-    <xacro:property name="link04_cover_mesh" value="forearm_mesh.dae" />
-    <xacro:property name="link05_cover_mesh" value="wrist1_mesh.dae" />
-    <xacro:property name="link06_cover_mesh" value="wrist2_mesh.dae" />
-  </xacro:if>
-  <xacro:unless value="${covers}">
-    <xacro:property name="base_mesh" value="base_mesh.dae" />
-    <xacro:property name="link01_mesh" value="shoulder_mesh.dae" />
-    <xacro:property name="link02_mesh" value="upperarm_mesh.dae" />
-    <xacro:property name="link03_mesh" value="elbow_mesh.dae" />
-    <xacro:property name="link04_mesh" value="forearm_mesh.dae" />
-    <xacro:property name="link05_mesh" value="wrist1_mesh.dae" />
-    <xacro:property name="link06_mesh" value="wrist2_mesh.dae" />
-  </xacro:unless>
+  <xacro:property name="base_mesh" value="base_mesh.dae" />
+  <xacro:property name="link01_mesh" value="shoulder_mesh.dae" />
+  <xacro:property name="link02_mesh" value="upperarm_mesh.dae" />
+  <xacro:property name="link03_mesh" value="elbow_mesh.dae" />
+  <xacro:property name="link04_mesh" value="forearm_mesh.dae" />
+  <xacro:property name="link05_mesh" value="wrist1_mesh.dae" />
+  <xacro:property name="link06_mesh" value="wrist2_mesh.dae" />
   <!-- Joint properties -->
   <xacro:property name="joint_base_name" value="${tf_prefix}joint_base" />
@@ -226,53 +208,4 @@
     </inertial>
   </xacro:property>
-  <!-- Covers -->
-  <xacro:property name="base_cover_inertial">
-    <inertial>
-      <mass value="0.098" />
-      <origin xyz="${0.0*mm_to_m} ${0.0*mm_to_m} ${-60.7*mm_to_m}" rpy="0 0 0" />
-      <inertia ixx="${0.000349}" iyy="${0.000338}" izz="${0.000649}" ixy="${0.000000018}"
-        ixz="${-0.000000001}" iyz="${-0.000000002}" />
-    </inertial>
-  </xacro:property>
-  <xacro:property name="link01_cover_inertial">
-    <inertial>
-      <mass value="0.135" />
-      <origin xyz="${-0.039*mm_to_m} ${-0.015*mm_to_m} ${-31.709*mm_to_m}" rpy="0 0 0" />
-      <inertia ixx="${0.00068}" iyy="${0.000517}" izz="${0.000646}" ixy="${-0.000000318}"
-        ixz="${-0.000000206}" iyz="${-0.000000074}" />
-    </inertial>
-  </xacro:property>
-  <xacro:property name="link02_cover_inertial">
-    <inertial>
-      <mass value="0.743" />
-      <origin xyz="${167.97*mm_to_m} ${0.081*mm_to_m} ${0.0*mm_to_m}" rpy="0 0 0" />
-      <inertia ixx="${0.0054}" iyy="${0.025}" izz="${0.0293}" ixy="${-0.000004814}"
-        ixz="${-0.000000101}" iyz="${0.000000134}" />
-    </inertial>
-  </xacro:property>
-  <xacro:property name="link03_cover_inertial">
-    <inertial>
-      <mass value="0.383" />
-      <origin xyz="${37.807*mm_to_m} ${-101.52*mm_to_m} ${0.184*mm_to_m}" rpy="0 0 0" />
-      <inertia ixx="${0.00139}" iyy="${0.00176}" izz="${0.00225}" ixy="${-0.000150269}"
-        ixz="${0.000002221}" iyz="${-0.000003993}" />
-    </inertial>
-  </xacro:property>
-  <xacro:property name="link04_cover_inertial">
-    <inertial>
-      <mass value="0.158" />
-      <origin xyz="${-9.28*mm_to_m} ${-0.008*mm_to_m} ${377.34*mm_to_m}" rpy="0 0 0" />
-      <inertia ixx="${0.000594}" iyy="${0.000846}" izz="${0.000485}" ixy="${-0.000000100}"
-        ixz="${-0.000057116}" iyz="${0.000000128}" />
-    </inertial>
-  </xacro:property>
-  <xacro:property name="link05_cover_inertial">
-    <inertial>
-      <mass value="0.121" />
-      <origin xyz="${54.24*mm_to_m} ${-0.0012*mm_to_m} ${-0.0069*mm_to_m}" rpy="0 0 0" />
-      <inertia ixx="${0.0003}" iyy="${0.00049}" izz="${0.00053}" ixy="${-0.000000004}"
-        ixz="${0.0}" iyz="${-0.000000043}" />
-    </inertial>
-  </xacro:property>
  <xacro:if value="${collision == 'simple'}">
     <!-- Collision properties -->

File: duatic_dynaarm_description/urdf/common/corydoras12/dynaarm_parameters.urdf.xacro (robot description, xacro)
@@ -40,29 +40,11 @@
   <xacro:property name="end_effector" value="${tf_prefix}flange" />
   <!-- Meshes -->
-  <xacro:if value="${covers}">
-    <xacro:property name="base_mesh" value="base_mesh.dae" />
-    <xacro:property name="link01_mesh" value="shoulder_mesh.dae" />
-    <xacro:property name="link02_mesh" value="upperarm_mesh.dae" />
-    <xacro:property name="link03_mesh" value="elbow_mesh.dae" />
-    <xacro:property name="link04_mesh" value="forearm_mesh.dae" />
-    <xacro:property name="link05_mesh" value="wrist1_mesh.dae" />
-    <xacro:property name="link06_mesh" value="wrist2_mesh.dae" />
-    <xacro:property name="base_cover_mesh" value="base_mesh.dae" />
-    <xacro:property name="link01_cover_mesh" value="shoulder_mesh.dae" />
-    <xacro:property name="link02_cover_mesh" value="upperarm_mesh.dae" />
-    <xacro:property name="link03_cover_mesh" value="elbow_mesh.dae" />
-    <xacro:property name="link04_cover_mesh" value="forearm_mesh.dae" />
-    <xacro:property name="link05_cover_mesh" value="wrist1_mesh.dae" />
-    <xacro:property name="link06_cover_mesh" value="wrist2_mesh.dae" />
-  </xacro:if>
-  <xacro:unless value="${covers}">
-    <xacro:property name="base_mesh" value="base_mesh.dae" />
-    <xacro:property name="link01_mesh" value="shoulder_mesh.dae" />
-    <xacro:property name="link02_mesh" value="upperarm_mesh.dae" />
-    <xacro:property name="link03_mesh" value="elbow_mesh.dae" />
-    <xacro:property name="link04_mesh" value="forearm_mesh.dae" />
-    <xacro:property name="link05_mesh" value="wrist1_mesh.dae" />
-    <xacro:property name="link06_mesh" value="wrist2_mesh.dae" />
-  </xacro:unless>
+  <xacro:property name="base_mesh" value="base_mesh.dae" />
+  <xacro:property name="link01_mesh" value="shoulder_mesh.dae" />
+  <xacro:property name="link02_mesh" value="upperarm_mesh.dae" />
+  <xacro:property name="link03_mesh" value="elbow_mesh.dae" />
+  <xacro:property name="link04_mesh" value="forearm_mesh.dae" />
+  <xacro:property name="link05_mesh" value="wrist1_mesh.dae" />
+  <xacro:property name="link06_mesh" value="wrist2_mesh.dae" />
   <!-- Joint properties -->
   <xacro:property name="joint_base_name" value="${tf_prefix}joint_base" />
@@ -226,53 +208,4 @@
     </inertial>
   </xacro:property>
-  <!-- Covers -->
-  <xacro:property name="base_cover_inertial">
-    <inertial>
-      <mass value="0.098" />
-      <origin xyz="${0.0*mm_to_m} ${0.0*mm_to_m} ${-60.7*mm_to_m}" rpy="0 0 0" />
-      <inertia ixx="${0.000349}" iyy="${0.000338}" izz="${0.000649}" ixy="${0.000000018}"
-        ixz="${-0.000000001}" iyz="${-0.000000002}" />
-    </inertial>
-  </xacro:property>
-  <xacro:property name="link01_cover_inertial">
-    <inertial>
-      <mass value="0.135" />
-      <origin xyz="${-0.039*mm_to_m} ${-0.015*mm_to_m} ${-31.709*mm_to_m}" rpy="0 0 0" />
-      <inertia ixx="${0.00068}" iyy="${0.000517}" izz="${0.000646}" ixy="${-0.000000318}"
-        ixz="${-0.000000206}" iyz="${-0.000000074}" />
-    </inertial>
-  </xacro:property>
-  <xacro:property name="link02_cover_inertial">
-    <inertial>
-      <mass value="0.743" />
-      <origin xyz="${167.97*mm_to_m} ${0.081*mm_to_m} ${0.0*mm_to_m}" rpy="0 0 0" />
-      <inertia ixx="${0.0054}" iyy="${0.025}" izz="${0.0293}" ixy="${-0.000004814}"
-        ixz="${-0.000000101}" iyz="${0.000000134}" />
-    </inertial>
-  </xacro:property>
-  <xacro:property name="link03_cover_inertial">
-    <inertial>
-      <mass value="0.383" />
-      <origin xyz="${37.807*mm_to_m} ${-101.52*mm_to_m} ${0.184*mm_to_m}" rpy="0 0 0" />
-      <inertia ixx="${0.00139}" iyy="${0.00176}" izz="${0.00225}" ixy="${-0.000150269}"
-        ixz="${0.000002221}" iyz="${-0.000003993}" />
-    </inertial>
-  </xacro:property>
-  <xacro:property name="link04_cover_inertial">
-    <inertial>
-      <mass value="0.158" />
-      <origin xyz="${-9.28*mm_to_m} ${-0.008*mm_to_m} ${377.34*mm_to_m}" rpy="0 0 0" />
-      <inertia ixx="${0.000594}" iyy="${0.000846}" izz="${0.000485}" ixy="${-0.000000100}"
-        ixz="${-0.000057116}" iyz="${0.000000128}" />
-    </inertial>
-  </xacro:property>
-  <xacro:property name="link05_cover_inertial">
-    <inertial>
-      <mass value="0.121" />
-      <origin xyz="${54.24*mm_to_m} ${-0.0012*mm_to_m} ${-0.0069*mm_to_m}" rpy="0 0 0" />
-      <inertia ixx="${0.0003}" iyy="${0.00049}" izz="${0.00053}" ixy="${-0.000000004}"
-        ixz="${0.0}" iyz="${-0.000000043}" />
-    </inertial>
-  </xacro:property>
  <xacro:if value="${collision == 'simple'}">
     <!-- Collision properties -->

File: duatic_dynaarm_description/urdf/dynaarm.urdf.xacro (robot description, xacro)
@@ -26,5 +26,5 @@
   <!-- -->
   <xacro:macro name="dynaarm_description"
-    params="tf_prefix parent_link collision:='simple' dof  covers version *origin">
+    params="tf_prefix parent_link collision:='simple' dof version *origin">
     <!-- Set ee_parent based on the specified DoF -->
     <xacro:property name="ee_parent" value="${base}" />
@@ -54,17 +54,4 @@
       </base_collision>
     </xacro:dynaarm_baselink>
-    <!-- Base Covers-->
-    <xacro:if value="${covers}">
-      <xacro:dynaarm_link link_name="${base}_cover" file_name="${base_cover_mesh}">
-        <link_inertia>
-          <xacro:insert_block name="base_cover_inertial" />
-        </link_inertia>
-      </xacro:dynaarm_link>
-      <xacro:dynaarm_joint_fixed joint_name="${base}_cover"
-        parent="${base}"
-        child="${base}_cover">
-        <origin xyz="0.0 0.0 0.0" rpy="0.0 0.0 0.0" />
-      </xacro:dynaarm_joint_fixed>
-    </xacro:if>
     <!-- 1 DoF -->
     <xacro:if value="${dof >= 1}">
@@ -90,16 +77,4 @@
         <origin xyz="${joint_1_origin_xyz}" rpy="${joint_1_origin_rpy}" />
       </xacro:dynaarm_revolute_joint>
-      <!-- 1 Dof & Covers-->
-      <xacro:if value="${covers}">
-        <xacro:dynaarm_link link_name="${link01}_cover" file_name="${link01_cover_mesh}">
-          <link_inertia>
-            <xacro:insert_block name="link01_cover_inertial" />
-          </link_inertia>
-        </xacro:dynaarm_link>
-        <xacro:dynaarm_joint_fixed joint_name="${link01}_cover" parent="${link01}"
-          child="${link01}_cover">
-          <origin xyz="0.0 0.0 0.0" rpy="0.0 0.0 0.0" />
-        </xacro:dynaarm_joint_fixed>
-      </xacro:if>
     </xacro:if>
     <!-- 2 DoF -->
@@ -126,16 +101,4 @@
         <origin xyz="${joint_2_origin_xyz}" rpy="${joint_2_origin_rpy}" />
       </xacro:dynaarm_revolute_joint>
-      <!-- 2 Dof & Covers-->
-      <xacro:if value="${covers}">
-        <xacro:dynaarm_link link_name="${link02}_cover" file_name="${link02_cover_mesh}">
-          <link_inertia>
-            <xacro:insert_block name="link02_cover_inertial" />
-          </link_inertia>
-        </xacro:dynaarm_link>
-        <xacro:dynaarm_joint_fixed joint_name="${link02}_cover" parent="${link02}"
-          child="${link02}_cover">
-          <origin xyz="0.0 0.0 0.0" rpy="0.0 0.0 0.0" />
-        </xacro:dynaarm_joint_fixed>
-      </xacro:if>
     </xacro:if>
     <!-- 3 DoF -->
@@ -173,16 +136,4 @@
         </xacro:dynaarm_joint_fixed>
       </xacro:if>
-      <!-- 3 Dof & Covers-->
-      <xacro:if value="${covers}">
-        <xacro:dynaarm_link link_name="${link03}_cover" file_name="${link03_cover_mesh}">
-          <link_inertia>
-            <xacro:insert_block name="link03_cover_inertial" />
-          </link_inertia>
-        </xacro:dynaarm_link>
-        <xacro:dynaarm_joint_fixed joint_name="${link03}_cover" parent="${link03}"
-          child="${link03}_cover">
-          <origin xyz="0.0 0.0 0.0" rpy="0.0 0.0 0.0" />
-        </xacro:dynaarm_joint_fixed>
-      </xacro:if>
     </xacro:if>
     <!-- 4 DoF -->
@@ -218,16 +169,4 @@
         <origin xyz="${joint_4_origin_xyz}" rpy="${joint_4_origin_rpy}" />
       </xacro:dynaarm_revolute_joint>
-      <!-- 4 Dof & Covers-->
-      <xacro:if value="${covers}">
-        <xacro:dynaarm_link link_name="${link04}_cover" file_name="${link04_cover_mesh}">
-          <link_inertia>
-            <xacro:insert_block name="link04_cover_inertial" />
-          </link_inertia>
-        </xacro:dynaarm_link>
-        <xacro:dynaarm_joint_fixed joint_name="${link04}_cover" parent="${link04}"
-          child="${link04}_cover">
-          <origin xyz="0.0 0.0 0.0" rpy="0.0 0.0 0.0" />
-        </xacro:dynaarm_joint_fixed>
-      </xacro:if>
     </xacro:if>
     <!-- 5 DoF -->
@@ -261,16 +200,4 @@
           child="${link05_cam}">
           <origin xyz="${joint_5_cam_origin_xyz}" rpy="${joint_5_cam_origin_rpy}" />
-        </xacro:dynaarm_joint_fixed>
-      </xacro:if>
-      <!-- 5 Dof & Covers-->
-      <xacro:if value="${covers}">
-        <xacro:dynaarm_link link_name="${link05}_cover" file_name="${link05_cover_mesh}">
-          <link_inertia>
-            <xacro:insert_block name="link05_cover_inertial" />
-          </link_inertia>
-        </xacro:dynaarm_link>
-        <xacro:dynaarm_joint_fixed joint_name="${link05}_cover" parent="${link05}"
-          child="${link05}_cover">
-          <origin xyz="0.0 0.0 0.0" rpy="0.0 0.0 0.0" />
         </xacro:dynaarm_joint_fixed>
       </xacro:if>

File: duatic_dynaarm_description/urdf/dynaarm_standalone.urdf.xacro (robot description, xacro)
@@ -28,6 +28,4 @@
   <!-- collision: simple, complex -->
   <xacro:arg name="collision" default="simple" />
-  <!-- Change to add covers to the arm -->
-  <xacro:arg name="covers" default="false" />
   <!-- v1, v2, ... -->
   <xacro:arg name="version" default="baracuda12" />
@@ -42,5 +40,4 @@
                 dof="$(arg dof)"
                 collision="$(arg collision)"
-                covers="$(arg covers)"
                 version="$(arg version)">
     <origin xyz="0 0 0" rpy="0.0 0.0 0.0" />

File: duatic_dynaarm_description/urdf/dynaarm_standalone_dual.urdf.xacro (robot description, xacro)
@@ -28,6 +28,4 @@
   <!-- collision: simple, complex-->
   <xacro:arg name="collision" default="complex" />
-  <!-- Change to add covers to the arm -->
-  <xacro:arg name="covers" default="false" />
   <!-- v1, v2, ... -->
   <xacro:arg name="version" default="baracuda12" />
@@ -38,5 +36,4 @@
                 parent_link="base_link"
                 dof="$(arg dof)"
-                covers="$(arg covers)"
                 collision="$(arg collision)"
                 version="$(arg version)">
@@ -47,5 +44,4 @@
                 parent_link="base_link"
                 dof="$(arg dof)"
-                covers="$(arg covers)"
                 collision="$(arg collision)"
                 version="$(arg version)">

File: duatic_dynaarm_driver/urdf/dynaarm.urdf.xacro (robot description, xacro)
@@ -33,5 +33,4 @@
                          start_in_freeze_mode:=false
                          drive_parameter_folder:=''
-                         covers
                          version
                          *origin">
@@ -49,5 +48,4 @@
                 collision="${collision}"
                 dof="${dof}"
-                covers="${covers}"
                 version="${version}">
             <xacro:insert_block name="origin" />
