Commit message: fix: remove obsolete dof parameter

File: duatic_dynaarm_driver/urdf/dynaarm.ros2control.xacro (robot description, xacro)
@@ -31,5 +31,4 @@
         version
         tf_prefix
-        dof
         ethercat_addresses
         drive_parameter_folder:=''">
@@ -44,64 +43,52 @@
         <xacro:property name="drive_parameter_folder_internal" value="${drive_parameter_folder}" />
       </xacro:unless>
-      <xacro:if value="${dof >= 1}">
-        <xacro:duadrive_interface_joint name="${tf_prefix}shoulder_rotation"
-          ethercat_address="${ethercat_addresses['shoulder_rotation']}"
-          ethercat_bus="${ethercat_bus}"
-          mode="${mode}"
-          parent_unit="${parent_unit}"
-          drive_parameter_file_path="${drive_parameter_folder_internal}/shoulder_rotation.yaml"
-          has_brake="${has_brakes}" />
-      </xacro:if>
-      <xacro:if value="${dof >= 2}">
-        <xacro:duadrive_interface_joint name="${tf_prefix}shoulder_flexion"
-          ethercat_address="${ethercat_addresses['shoulder_flexion']}"
-          ethercat_bus="${ethercat_bus}"
-          mode="${mode}"
-          parent_unit="${parent_unit}"
-          drive_parameter_file_path="${drive_parameter_folder_internal}/shoulder_flexion.yaml"
-          has_brake="${has_brakes}" />
-      </xacro:if>
-      <xacro:if value="${dof >= 3}">
-        <xacro:duadrive_interface_joint name="${tf_prefix}elbow_flexion"
-          ethercat_address="${ethercat_addresses['elbow_flexion']}"
-          ethercat_bus="${ethercat_bus}"
-          mode="${mode}"
-          parent_unit="${parent_unit}"
-          drive_parameter_file_path="${drive_parameter_folder_internal}/elbow_flexion.yaml"
-          has_brake="${has_brakes}" />
-      </xacro:if>
-      <xacro:if value="${dof >= 4}">
-        <xacro:duadrive_interface_joint name="${tf_prefix}forearm_rotation"
-          ethercat_address="${ethercat_addresses['forearm_rotation']}"
-          ethercat_bus="${ethercat_bus}"
-          mode="${mode}"
-          parent_unit="${parent_unit}"
-          drive_parameter_file_path="${drive_parameter_folder_internal}/forearm_rotation.yaml"
-          has_brake="${has_brakes}" />
-      </xacro:if>
-      <xacro:if value="${dof >= 5}">
-        <xacro:duadrive_interface_joint name="${tf_prefix}wrist_flexion"
-          ethercat_address="${ethercat_addresses['wrist_flexion']}"
-          ethercat_bus="${ethercat_bus}"
-          mode="${mode}"
-          parent_unit="${parent_unit}"
-          drive_parameter_file_path="${drive_parameter_folder_internal}/wrist_flexion.yaml"
-          has_brake="${has_brakes}" />
-      </xacro:if>
-      <xacro:if value="${dof >= 6}">
-        <xacro:duadrive_interface_joint name="${tf_prefix}wrist_rotation"
-          ethercat_address="${ethercat_addresses['wrist_rotation']}"
-          ethercat_bus="${ethercat_bus}"
-          mode="${mode}"
-          parent_unit="${parent_unit}"
-          drive_parameter_file_path="${drive_parameter_folder_internal}/wrist_rotation.yaml"
-          has_brake="${has_brakes}" />
-      </xacro:if>
-      <!--
-      <xacro:if value="${mode != 'isaac'}">
-        <gpio name="${parent_unit}">
-          <command_interface name="freeze_mode" />
-        </gpio>
-      </xacro:if>-->
+      <!-- Shoulder Rotation -->
+      <xacro:duadrive_interface_joint name="${tf_prefix}shoulder_rotation"
+        ethercat_address="${ethercat_addresses['shoulder_rotation']}"
+        ethercat_bus="${ethercat_bus}"
+        mode="${mode}"
+        parent_unit="${parent_unit}"
+        drive_parameter_file_path="${drive_parameter_folder_internal}/shoulder_rotation.yaml"
+        has_brake="${has_brakes}" />
+      <!-- Shoulder Flexion -->
+      <xacro:duadrive_interface_joint name="${tf_prefix}shoulder_flexion"
+        ethercat_address="${ethercat_addresses['shoulder_flexion']}"
+        ethercat_bus="${ethercat_bus}"
+        mode="${mode}"
+        parent_unit="${parent_unit}"
+        drive_parameter_file_path="${drive_parameter_folder_internal}/shoulder_flexion.yaml"
+        has_brake="${has_brakes}" />
+      <!-- Elbow Flexion -->
+      <xacro:duadrive_interface_joint name="${tf_prefix}elbow_flexion"
+        ethercat_address="${ethercat_addresses['elbow_flexion']}"
+        ethercat_bus="${ethercat_bus}"
+        mode="${mode}"
+        parent_unit="${parent_unit}"
+        drive_parameter_file_path="${drive_parameter_folder_internal}/elbow_flexion.yaml"
+        has_brake="${has_brakes}" />
+      <!-- Forearm Rotation -->
+      <xacro:duadrive_interface_joint name="${tf_prefix}forearm_rotation"
+        ethercat_address="${ethercat_addresses['forearm_rotation']}"
+        ethercat_bus="${ethercat_bus}"
+        mode="${mode}"
+        parent_unit="${parent_unit}"
+        drive_parameter_file_path="${drive_parameter_folder_internal}/forearm_rotation.yaml"
+        has_brake="${has_brakes}" />
+      <!-- Wrist Flexion -->
+      <xacro:duadrive_interface_joint name="${tf_prefix}wrist_flexion"
+        ethercat_address="${ethercat_addresses['wrist_flexion']}"
+        ethercat_bus="${ethercat_bus}"
+        mode="${mode}"
+        parent_unit="${parent_unit}"
+        drive_parameter_file_path="${drive_parameter_folder_internal}/wrist_flexion.yaml"
+        has_brake="${has_brakes}" />
+      <!-- Wrist Rotation -->
+      <xacro:duadrive_interface_joint name="${tf_prefix}wrist_rotation"
+        ethercat_address="${ethercat_addresses['wrist_rotation']}"
+        ethercat_bus="${ethercat_bus}"
+        mode="${mode}"
+        parent_unit="${parent_unit}"
+        drive_parameter_file_path="${drive_parameter_folder_internal}/wrist_rotation.yaml"
+        has_brake="${has_brakes}" />
   </xacro:macro>
   <xacro:macro name="dynaarm_ros2_control"
@@ -113,6 +100,5 @@
                        version
                        ethercat_addresses
-                       mode
-                       dof">
+                       mode">
     <ros2_control name="${tf_prefix}DynaarmSystem" type="system">
       <hardware>
@@ -149,6 +135,5 @@
         ethercat_bus="${ethercat_bus}"
         parent_unit="${tf_prefix}DynaarmSystem"
-        ethercat_addresses="${ethercat_addresses}"
-        dof="${dof}"/>
+        ethercat_addresses="${ethercat_addresses}"/>
     </ros2_control>
   </xacro:macro>

File: duatic_dynaarm_driver/urdf/dynaarm.urdf.xacro (robot description, xacro)
@@ -27,5 +27,4 @@
                          parent_link
                          collision:='simple'
-                         dof:='6'
                          mode
                          ethercat_bus
@@ -47,5 +46,4 @@
                 parent_link="${parent_link}"
                 collision="${collision}"
-                dof="${dof}"
                 version="${version}">
             <xacro:insert_block name="origin" />
@@ -58,6 +56,5 @@
                                     ethercat_addresses="${ethercat_addresses}"
                                     version="${version}"
-                                    mode="${mode}"
-                                    dof="${dof}"/>
+                                    mode="${mode}"/>
     </xacro:macro>
 </robot>

Commit message: Removed unused meshes

File: duatic_dynaarm_demo/duatic_dynaarm_single_example/duatic_dynaarm_single_example_description/urdf/dynaarm_single_example.urdf.xacro (robot description, xacro)
@@ -56,5 +56,5 @@
                 ethercat_bus="$(arg ethercat_bus)"
                 version="$(arg version)">
-    <origin xyz="0 0 0" rpy="0.0 0.0 0.0" />
+    <origin xyz="0 0 0.025" rpy="0.0 0.0 0.0" />
   </xacro:dynaarm>
   <!-- Include the control plugin -->
