Commit message: new proposal of limit positioning

File: duatic_dynaarm_demo/duatic_dynaarm_single_example/duatic_dynaarm_single_example_description/urdf/dynaarm_single_example.urdf.xacro (robot description, xacro)
@@ -2,12 +2,25 @@
 <!--
 Copyright 2025 Duatic AG
-Redistribution and use in source and binary forms, with or without modification, are permitted provided that the following conditions are met:
-1. Redistributions of source code must retain the above copyright notice, this list of conditions and the following disclaimer.
-2. Redistributions in binary form must reproduce the above copyright notice, this list of conditions and the following disclaimer in the documentation and/or other materials provided with the distribution.
-3. Neither the name of the copyright holder nor the names of its contributors may be used to endorse or promote products derived from this software without specific prior written permission.
-THIS SOFTWARE IS PROVIDED BY THE COPYRIGHT HOLDERS AND CONTRIBUTORS “AS IS” AND ANY EXPRESS OR IMPLIED WARRANTIES, INCLUDING, BUT NOT LIMITED TO, THE IMPLIED WARRANTIES OF MERCHANTABILITY AND FITNESS FOR A PARTICULAR PURPOSE ARE DISCLAIMED. IN NO EVENT SHALL THE COPYRIGHT HOLDER OR CONTRIBUTORS BE LIABLE FOR ANY DIRECT, INDIRECT, INCIDENTAL, SPECIAL, EXEMPLARY, OR CONSEQUENTIAL DAMAGES (INCLUDING, BUT NOT LIMITED TO, PROCUREMENT OF SUBSTITUTE GOODS OR SERVICES; LOSS OF USE, DATA, OR PROFITS; OR BUSINESS INTERRUPTION) HOWEVER CAUSED AND ON ANY THEORY OF LIABILITY, WHETHER IN CONTRACT, STRICT LIABILITY, OR TORT (INCLUDING NEGLIGENCE OR OTHERWISE) ARISING IN ANY WAY OUT OF THE USE OF THIS SOFTWARE, EVEN IF ADVISED OF THE POSSIBILITY OF SUCH DAMAGE.
+Redistribution and use in source and binary forms, with or without modification, are permitted
+provided that the following conditions are met:
+1. Redistributions of source code must retain the above copyright notice, this list of conditions
+and the following disclaimer.
+2. Redistributions in binary form must reproduce the above copyright notice, this list of
+conditions and the following disclaimer in the documentation and/or other materials provided with
+the distribution.
+3. Neither the name of the copyright holder nor the names of its contributors may be used to
+endorse or promote products derived from this software without specific prior written permission.
+THIS SOFTWARE IS PROVIDED BY THE COPYRIGHT HOLDERS AND CONTRIBUTORS “AS IS” AND ANY EXPRESS OR
+IMPLIED WARRANTIES, INCLUDING, BUT NOT LIMITED TO, THE IMPLIED WARRANTIES OF MERCHANTABILITY AND
+FITNESS FOR A PARTICULAR PURPOSE ARE DISCLAIMED. IN NO EVENT SHALL THE COPYRIGHT HOLDER OR
+CONTRIBUTORS BE LIABLE FOR ANY DIRECT, INDIRECT, INCIDENTAL, SPECIAL, EXEMPLARY, OR CONSEQUENTIAL
+DAMAGES (INCLUDING, BUT NOT LIMITED TO, PROCUREMENT OF SUBSTITUTE GOODS OR SERVICES; LOSS OF USE,
+DATA, OR PROFITS; OR BUSINESS INTERRUPTION) HOWEVER CAUSED AND ON ANY THEORY OF LIABILITY, WHETHER
+IN CONTRACT, STRICT LIABILITY, OR TORT (INCLUDING NEGLIGENCE OR OTHERWISE) ARISING IN ANY WAY OUT
+OF
+THE USE OF THIS SOFTWARE, EVEN IF ADVISED OF THE POSSIBILITY OF SUCH DAMAGE.
 -->
 <robot name="dynaarm" xmlns:xacro="http://www.ros.org/wiki/xacro">
-  <!--Example single arm setup-->
+  <!-- Example single arm setup -->
   <xacro:arg name="tf_prefix" default="" />
   <!-- simple, complex -->
@@ -20,40 +33,54 @@
   <xacro:arg name="version" default="baracuda12" />
   <xacro:arg name="namespace" default="" />
+  <!-- robot control limits -->
+  <xacro:arg name="shoulder_rotation_limit_vel" default="10.64" />
+  <xacro:arg name="shoulder_flexion_limit_vel" default="10.64" />
+  <xacro:arg name="elbow_flexion_limit_vel" default="10.64" />
+  <xacro:arg name="forearm_rotation_limit_vel" default="13.647" />
+  <xacro:arg name="wrist_flexion_limit_vel" default="13.647" />
+  <xacro:arg name="wrist_rotation_limit_vel" default="13.647" />
+  <xacro:arg name="shoulder_rotation_limit_effort" default="120.0" />
+  <xacro:arg name="shoulder_flexion_limit_effort" default="120.0" />
+  <xacro:arg name="elbow_flexion_limit_effort" default="120.0" />
+  <xacro:arg name="forearm_rotation_limit_effort" default="40.0" />
+  <xacro:arg name="wrist_flexion_limit_effort" default="40.0" />
+  <xacro:arg name="wrist_rotation_limit_effort" default="40.0" />
+  <!-- load robot description -->
   <xacro:include filename="$(find duatic_dynaarm_driver)/urdf/dynaarm.urdf.xacro" />
-<link name="base_link" />
+  <link name="base_link" />
   <link name="table">
     <visual>
       <origin xyz="0 0 0" rpy="0 0 0" />
       <geometry>
-          <box size="1.0 1.0 0.05"/>
+        <box size="1.0 1.0 0.05" />
       </geometry>
       <material name="Wood">
-        <color rgba="0.9 0.83 0.733 1.0"/>
+        <color rgba="0.9 0.83 0.733 1.0" />
       </material>
     </visual>
     <collision>
-      <origin xyz="0 0 0" rpy="0 0 0"/>
+      <origin xyz="0 0 0" rpy="0 0 0" />
       <geometry>
-          <box size="1.0 1.0 0.05"/>
+        <box size="1.0 1.0 0.05" />
       </geometry>
     </collision>
     <inertial>
-      <mass value="10.0"/>
-      <origin xyz="0 0 0"/>
-      <inertia ixx="1.0" ixy="0.0" ixz="0.0" iyy="1.0" iyz="0.0" izz="1.0"/>
+      <mass value="10.0" />
+      <origin xyz="0 0 0" />
+      <inertia ixx="1.0" ixy="0.0" ixz="0.0" iyy="1.0" iyz="0.0" izz="1.0" />
     </inertial>
   </link>
   <joint name="table_joint" type="fixed">
-    <parent link="base_link"/>
-    <child link="table"/>
-    <origin xyz="0 0 -0.025" rpy="0 0 0"/>
+    <parent link="base_link" />
+    <child link="table" />
+    <origin xyz="0 0 -0.025" rpy="0 0 0" />
   </joint>
   <!-- create an instance of the dynaarm and fix its base-->
   <xacro:dynaarm tf_prefix="$(arg tf_prefix)"
-                parent_link="table"
-                collision="$(arg collision)"
-                mode="$(arg mode)"
-                ethercat_bus="$(arg ethercat_bus)"
-                version="$(arg version)">
+    parent_link="table"
+    collision="$(arg collision)"
+    mode="$(arg mode)"
+    ethercat_bus="$(arg ethercat_bus)"
+    version="$(arg version)">
     <origin xyz="0 0 0" rpy="0.0 0.0 0.0" />
   </xacro:dynaarm>

File: duatic_dynaarm_description/urdf/common/baracuda12/dynaarm_parameters.urdf.xacro (robot description, xacro)
@@ -22,4 +22,22 @@
 -->
 <robot xmlns:xacro="http://www.ros.org/wiki/xacro">
+  <!-- DuaDrive Defaults -->
+  <xacro:property name="duadrive_T120_limit_vel" value="10.64" />
+  <xacro:property name="duadrive_T120_limit_effort" value="120.0" />
+  <xacro:property name="duadrive_T40_limit_vel" value="13.647" />
+  <xacro:property name="duadrive_T40_limit_effort" value="40.0" />
+  <!-- Joint limit overrides (fall back to the drive defaults above if not declared by the caller) -->
+  <xacro:arg name="shoulder_rotation_limit_vel" default="${duadrive_T120_limit_vel}" />
+  <xacro:arg name="shoulder_rotation_limit_effort" default="${duadrive_T120_limit_effort}" />
+  <xacro:arg name="shoulder_flexion_limit_vel" default="${duadrive_T120_limit_vel}" />
+  <xacro:arg name="shoulder_flexion_limit_effort" default="${duadrive_T120_limit_effort}" />
+  <xacro:arg name="elbow_flexion_limit_vel" default="${duadrive_T120_limit_vel}" />
+  <xacro:arg name="elbow_flexion_limit_effort" default="${duadrive_T120_limit_effort}" />
+  <xacro:arg name="forearm_rotation_limit_vel" default="${duadrive_T40_limit_vel}" />
+  <xacro:arg name="forearm_rotation_limit_effort" default="${duadrive_T40_limit_effort}" />
+  <xacro:arg name="wrist_flexion_limit_vel" default="${duadrive_T40_limit_vel}" />
+  <xacro:arg name="wrist_flexion_limit_effort" default="${duadrive_T40_limit_effort}" />
+  <xacro:arg name="wrist_rotation_limit_vel" default="${duadrive_T40_limit_vel}" />
+  <xacro:arg name="wrist_rotation_limit_effort" default="${duadrive_T40_limit_effort}" />
   <!-- Links -->
   <xacro:property name="base" value="${tf_prefix}base" />
@@ -54,4 +72,6 @@
   <xacro:property name="joint_1_lower_limit" value="${-J_PI - J_PI/2 + 0.4}" />
   <xacro:property name="joint_1_upper_limit" value="${J_PI + J_PI/2 - 0.4}" />
+  <xacro:property name="joint_1_limit_vel" value="${xacro.arg('shoulder_rotation_limit_vel')}" />
+  <xacro:property name="joint_1_limit_effort" value="${xacro.arg('shoulder_rotation_limit_effort')}" />
   <xacro:property name="joint_2_name" value="${tf_prefix}shoulder_flexion" />
   <xacro:property name="joint_2_joint_type" value="revolute" />
@@ -61,4 +81,6 @@
   <xacro:property name="joint_2_lower_limit" value="${-J_PI/2 - 0.15}" />
   <xacro:property name="joint_2_upper_limit" value="${J_PI/2 + 0.15}" />
+  <xacro:property name="joint_2_limit_vel" value="${xacro.arg('shoulder_flexion_limit_vel')}" />
+  <xacro:property name="joint_2_limit_effort" value="${xacro.arg('shoulder_flexion_limit_effort')}" />
   <xacro:property name="joint_3_name" value="${tf_prefix}elbow_flexion" />
   <xacro:property name="joint_3_joint_type" value="revolute" />
@@ -68,4 +90,6 @@
   <xacro:property name="joint_3_lower_limit" value="0.00" />
   <xacro:property name="joint_3_upper_limit" value="${J_PI - 0.05}" />
+  <xacro:property name="joint_3_limit_vel" value="${xacro.arg('elbow_flexion_limit_vel')}" />
+  <xacro:property name="joint_3_limit_effort" value="${xacro.arg('elbow_flexion_limit_effort')}" />
   <xacro:property name="joint_3_cam_name" value="${tf_prefix}elbow_camera" />
   <xacro:property name="joint_3_cam_joint_type" value="fixed" />
@@ -80,4 +104,6 @@
   <xacro:property name="joint_4_lower_limit" value="${-J_PI - J_PI/2}" />
   <xacro:property name="joint_4_upper_limit" value="${J_PI + J_PI/2}" />
+  <xacro:property name="joint_4_limit_vel" value="${xacro.arg('forearm_rotation_limit_vel')}" />
+  <xacro:property name="joint_4_limit_effort" value="${xacro.arg('forearm_rotation_limit_effort')}" />
   <xacro:property name="joint_5_name" value="${tf_prefix}wrist_flexion" />
   <xacro:property name="joint_5_joint_type" value="revolute" />
@@ -87,4 +113,6 @@
   <xacro:property name="joint_5_lower_limit" value="${-J_PI/2 -0.25}" />
   <xacro:property name="joint_5_upper_limit" value="${J_PI/2 + 0.25}" />
+  <xacro:property name="joint_5_limit_vel" value="${xacro.arg('wrist_flexion_limit_vel')}" />
+  <xacro:property name="joint_5_limit_effort" value="${xacro.arg('wrist_flexion_limit_effort')}" />
   <xacro:property name="joint_5_cam_name" value="${tf_prefix}wrist_flexion_camera" />
   <xacro:property name="joint_5_cam_joint_type" value="fixed" />
@@ -99,4 +127,6 @@
   <xacro:property name="joint_6_lower_limit" value="${-J_PI/2}" />
   <xacro:property name="joint_6_upper_limit" value="${J_PI + J_PI/2}" />
+  <xacro:property name="joint_6_limit_vel" value="${xacro.arg('wrist_rotation_limit_vel')}" />
+  <xacro:property name="joint_6_limit_effort" value="${xacro.arg('wrist_rotation_limit_effort')}" />
   <xacro:property name="joint_ee_name" value="${tf_prefix}flange_fix_joint" />
   <xacro:property name="joint_ee_xyz" value="0.0 0.0 0.009" />

File: duatic_dynaarm_description/urdf/common/corydoras12/dynaarm_parameters.urdf.xacro (robot description, xacro)
@@ -22,4 +22,22 @@
 -->
 <robot xmlns:xacro="http://www.ros.org/wiki/xacro">
+  <!-- DuaDrive Defaults -->
+  <xacro:property name="duadrive_T120_limit_vel" value="10.64" />
+  <xacro:property name="duadrive_T120_limit_effort" value="120.0" />
+  <xacro:property name="duadrive_T40_limit_vel" value="13.647" />
+  <xacro:property name="duadrive_T40_limit_effort" value="40.0" />
+  <!-- Joint limit overrides (fall back to the drive defaults above if not declared by the caller) -->
+  <xacro:arg name="shoulder_rotation_limit_vel" default="${duadrive_T120_limit_vel}" />
+  <xacro:arg name="shoulder_rotation_limit_effort" default="${duadrive_T120_limit_effort}" />
+  <xacro:arg name="shoulder_flexion_limit_vel" default="${duadrive_T120_limit_vel}" />
+  <xacro:arg name="shoulder_flexion_limit_effort" default="${duadrive_T120_limit_effort}" />
+  <xacro:arg name="elbow_flexion_limit_vel" default="${duadrive_T120_limit_vel}" />
+  <xacro:arg name="elbow_flexion_limit_effort" default="${duadrive_T120_limit_effort}" />
+  <xacro:arg name="forearm_rotation_limit_vel" default="${duadrive_T40_limit_vel}" />
+  <xacro:arg name="forearm_rotation_limit_effort" default="${duadrive_T40_limit_effort}" />
+  <xacro:arg name="wrist_flexion_limit_vel" default="${duadrive_T40_limit_vel}" />
+  <xacro:arg name="wrist_flexion_limit_effort" default="${duadrive_T40_limit_effort}" />
+  <xacro:arg name="wrist_rotation_limit_vel" default="${duadrive_T40_limit_vel}" />
+  <xacro:arg name="wrist_rotation_limit_effort" default="${duadrive_T40_limit_effort}" />
   <!-- Links -->
   <xacro:property name="base" value="${tf_prefix}base" />
@@ -54,4 +72,6 @@
   <xacro:property name="joint_1_lower_limit" value="${-J_PI - J_PI/2 + 0.4}" />
   <xacro:property name="joint_1_upper_limit" value="${J_PI + J_PI/2 - 0.4}" />
+  <xacro:property name="joint_1_limit_vel" value="${xacro.arg('shoulder_rotation_limit_vel')}" />
+  <xacro:property name="joint_1_limit_effort" value="${xacro.arg('shoulder_rotation_limit_effort')}" />
   <xacro:property name="joint_2_name" value="${tf_prefix}shoulder_flexion" />
   <xacro:property name="joint_2_joint_type" value="revolute" />
@@ -61,4 +81,6 @@
   <xacro:property name="joint_2_lower_limit" value="${-J_PI/2 - 0.15}" />
   <xacro:property name="joint_2_upper_limit" value="${J_PI/2 + 0.15}" />
+  <xacro:property name="joint_2_limit_vel" value="${xacro.arg('shoulder_flexion_limit_vel')}" />
+  <xacro:property name="joint_2_limit_effort" value="${xacro.arg('shoulder_flexion_limit_effort')}" />
   <xacro:property name="joint_3_name" value="${tf_prefix}elbow_flexion" />
   <xacro:property name="joint_3_joint_type" value="revolute" />
@@ -68,4 +90,6 @@
   <xacro:property name="joint_3_lower_limit" value="0.00" />
   <xacro:property name="joint_3_upper_limit" value="${J_PI - 0.05}" />
+  <xacro:property name="joint_3_limit_vel" value="${xacro.arg('elbow_flexion_limit_vel')}" />
+  <xacro:property name="joint_3_limit_effort" value="${xacro.arg('elbow_flexion_limit_effort')}" />
   <xacro:property name="joint_3_cam_name" value="${tf_prefix}elbow_camera" />
   <xacro:property name="joint_3_cam_joint_type" value="fixed" />
@@ -80,4 +104,6 @@
   <xacro:property name="joint_4_lower_limit" value="${-J_PI - J_PI/2}" />
   <xacro:property name="joint_4_upper_limit" value="${J_PI + J_PI/2}" />
+  <xacro:property name="joint_4_limit_vel" value="${xacro.arg('forearm_rotation_limit_vel')}" />
+  <xacro:property name="joint_4_limit_effort" value="${xacro.arg('forearm_rotation_limit_effort')}" />
   <xacro:property name="joint_5_name" value="${tf_prefix}wrist_flexion" />
   <xacro:property name="joint_5_joint_type" value="revolute" />
@@ -87,4 +113,6 @@
   <xacro:property name="joint_5_lower_limit" value="${-J_PI/2 -0.25}" />
   <xacro:property name="joint_5_upper_limit" value="${J_PI/2 + 0.25}" />
+  <xacro:property name="joint_5_limit_vel" value="${xacro.arg('wrist_flexion_limit_vel')}" />
+  <xacro:property name="joint_5_limit_effort" value="${xacro.arg('wrist_flexion_limit_effort')}" />
   <xacro:property name="joint_5_cam_name" value="${tf_prefix}wrist_flexion_camera" />
   <xacro:property name="joint_5_cam_joint_type" value="fixed" />
@@ -99,4 +127,6 @@
   <xacro:property name="joint_6_lower_limit" value="${-J_PI/2}" />
   <xacro:property name="joint_6_upper_limit" value="${J_PI + J_PI/2}" />
+  <xacro:property name="joint_6_limit_vel" value="${xacro.arg('wrist_rotation_limit_vel')}" />
+  <xacro:property name="joint_6_limit_effort" value="${xacro.arg('wrist_rotation_limit_effort')}" />
   <xacro:property name="joint_ee_name" value="${tf_prefix}flange_fix_joint" />
   <xacro:property name="joint_ee_xyz" value="0.0 0.0 0.009" />

File: duatic_dynaarm_description/urdf/common/dynaarm_common.urdf.xacro (robot description, xacro)
@@ -28,19 +28,4 @@
   <xacro:property name="mm2_to_m2" value="0.000001" />
   <xacro:property name="mm_to_m" value="0.001" />
-  <!-- -->
-  <!-- Common Definitions -->
-  <!-- -->
-  <xacro:property name="joint_1_limit_vel" value="10.64" />
-  <xacro:property name="joint_2_limit_vel" value="10.64" />
-  <xacro:property name="joint_3_limit_vel" value="10.64" />
-  <xacro:property name="joint_4_limit_vel" value="13.647" />
-  <xacro:property name="joint_5_limit_vel" value="13.647" />
-  <xacro:property name="joint_6_limit_vel" value="13.647" />
-  <xacro:property name="joint_1_limit_effort" value="120.0" />
-  <xacro:property name="joint_2_limit_effort" value="120.0" />
-  <xacro:property name="joint_3_limit_effort" value="120.0" />
-  <xacro:property name="joint_4_limit_effort" value="40.0" />
-  <xacro:property name="joint_5_limit_effort" value="40.0" />
-  <xacro:property name="joint_6_limit_effort" value="40.0" />
   <!-- -->
   <!-- DynaArm Base Link Macro -->
