Commit message: limits as macro parameters

File: duatic_dynaarm_demo/duatic_dynaarm_single_example/duatic_dynaarm_single_example_description/urdf/dynaarm_single_example.urdf.xacro (robot description, xacro)
@@ -33,17 +33,17 @@
   <xacro:arg name="version" default="baracuda12" />
   <xacro:arg name="namespace" default="" />
-  <!-- robot control limits -->
-  <xacro:arg name="shoulder_rotation_limit_vel" default="10.64" />
-  <xacro:arg name="shoulder_flexion_limit_vel" default="10.64" />
-  <xacro:arg name="elbow_flexion_limit_vel" default="10.64" />
-  <xacro:arg name="forearm_rotation_limit_vel" default="13.647" />
-  <xacro:arg name="wrist_flexion_limit_vel" default="13.647" />
-  <xacro:arg name="wrist_rotation_limit_vel" default="13.647" />
-  <xacro:arg name="shoulder_rotation_limit_effort" default="120.0" />
-  <xacro:arg name="shoulder_flexion_limit_effort" default="120.0" />
-  <xacro:arg name="elbow_flexion_limit_effort" default="120.0" />
-  <xacro:arg name="forearm_rotation_limit_effort" default="40.0" />
-  <xacro:arg name="wrist_flexion_limit_effort" default="40.0" />
-  <xacro:arg name="wrist_rotation_limit_effort" default="40.0" />
+  <!-- example definition of custom control limits; remove if not needed -->
+  <xacro:arg name="shoulder_rotation_limit_vel" default="" />
+  <xacro:arg name="shoulder_flexion_limit_vel" default="" />
+  <xacro:arg name="elbow_flexion_limit_vel" default="" />
+  <xacro:arg name="forearm_rotation_limit_vel" default="" />
+  <xacro:arg name="wrist_flexion_limit_vel" default="" />
+  <xacro:arg name="wrist_rotation_limit_vel" default="" />
+  <xacro:arg name="shoulder_rotation_limit_effort" default="" />
+  <xacro:arg name="shoulder_flexion_limit_effort" default="" />
+  <xacro:arg name="elbow_flexion_limit_effort" default="" />
+  <xacro:arg name="forearm_rotation_limit_effort" default="" />
+  <xacro:arg name="wrist_flexion_limit_effort" default="" />
+  <xacro:arg name="wrist_rotation_limit_effort" default="" />
   <!-- load robot description -->
   <xacro:include filename="$(find duatic_dynaarm_driver)/urdf/dynaarm.urdf.xacro" />
@@ -82,5 +82,17 @@
     mode="$(arg mode)"
     ethercat_bus="$(arg ethercat_bus)"
-    version="$(arg version)">
+    version="$(arg version)"
+    joint_1_limit_vel="$(arg shoulder_rotation_limit_vel)"
+    joint_2_limit_vel="$(arg shoulder_flexion_limit_vel)"
+    joint_3_limit_vel="$(arg elbow_flexion_limit_vel)"
+    joint_4_limit_vel="$(arg forearm_rotation_limit_vel)"
+    joint_5_limit_vel="$(arg wrist_flexion_limit_vel)"
+    joint_6_limit_vel="$(arg wrist_rotation_limit_vel)"
+    joint_1_limit_effort="$(arg shoulder_rotation_limit_effort)"
+    joint_2_limit_effort="$(arg shoulder_flexion_limit_effort)"
+    joint_3_limit_effort="$(arg elbow_flexion_limit_effort)"
+    joint_4_limit_effort="$(arg forearm_rotation_limit_effort)"
+    joint_5_limit_effort="$(arg wrist_flexion_limit_effort)"
+    joint_6_limit_effort="$(arg wrist_rotation_limit_effort)">
     <origin xyz="0 0 0" rpy="0.0 0.0 0.0" />
   </xacro:dynaarm>

File: duatic_dynaarm_description/urdf/common/baracuda12/dynaarm_parameters.urdf.xacro (robot description, xacro)
@@ -27,17 +27,4 @@
   <xacro:property name="duadrive_T40_limit_vel" value="13.647" />
   <xacro:property name="duadrive_T40_limit_effort" value="40.0" />
-  <!-- Joint limit overrides (fall back to the drive defaults above if not declared by the caller) -->
-  <xacro:arg name="shoulder_rotation_limit_vel" default="${duadrive_T120_limit_vel}" />
-  <xacro:arg name="shoulder_rotation_limit_effort" default="${duadrive_T120_limit_effort}" />
-  <xacro:arg name="shoulder_flexion_limit_vel" default="${duadrive_T120_limit_vel}" />
-  <xacro:arg name="shoulder_flexion_limit_effort" default="${duadrive_T120_limit_effort}" />
-  <xacro:arg name="elbow_flexion_limit_vel" default="${duadrive_T120_limit_vel}" />
-  <xacro:arg name="elbow_flexion_limit_effort" default="${duadrive_T120_limit_effort}" />
-  <xacro:arg name="forearm_rotation_limit_vel" default="${duadrive_T40_limit_vel}" />
-  <xacro:arg name="forearm_rotation_limit_effort" default="${duadrive_T40_limit_effort}" />
-  <xacro:arg name="wrist_flexion_limit_vel" default="${duadrive_T40_limit_vel}" />
-  <xacro:arg name="wrist_flexion_limit_effort" default="${duadrive_T40_limit_effort}" />
-  <xacro:arg name="wrist_rotation_limit_vel" default="${duadrive_T40_limit_vel}" />
-  <xacro:arg name="wrist_rotation_limit_effort" default="${duadrive_T40_limit_effort}" />
   <!-- Links -->
   <xacro:property name="base" value="${tf_prefix}base" />
@@ -72,6 +59,6 @@
   <xacro:property name="joint_1_lower_limit" value="${-J_PI - J_PI/2 + 0.4}" />
   <xacro:property name="joint_1_upper_limit" value="${J_PI + J_PI/2 - 0.4}" />
-  <xacro:property name="joint_1_limit_vel" value="${xacro.arg('shoulder_rotation_limit_vel')}" />
-  <xacro:property name="joint_1_limit_effort" value="${xacro.arg('shoulder_rotation_limit_effort')}" />
+  <xacro:property name="joint_1_limit_vel_default" value="${duadrive_T120_limit_vel}" />
+  <xacro:property name="joint_1_limit_effort_default" value="${duadrive_T120_limit_effort}" />
   <xacro:property name="joint_2_name" value="${tf_prefix}shoulder_flexion" />
   <xacro:property name="joint_2_joint_type" value="revolute" />
@@ -81,6 +68,6 @@
   <xacro:property name="joint_2_lower_limit" value="${-J_PI/2 - 0.15}" />
   <xacro:property name="joint_2_upper_limit" value="${J_PI/2 + 0.15}" />
-  <xacro:property name="joint_2_limit_vel" value="${xacro.arg('shoulder_flexion_limit_vel')}" />
-  <xacro:property name="joint_2_limit_effort" value="${xacro.arg('shoulder_flexion_limit_effort')}" />
+  <xacro:property name="joint_2_limit_vel_default" value="${duadrive_T120_limit_vel}" />
+  <xacro:property name="joint_2_limit_effort_default" value="${duadrive_T120_limit_effort}" />
   <xacro:property name="joint_3_name" value="${tf_prefix}elbow_flexion" />
   <xacro:property name="joint_3_joint_type" value="revolute" />
@@ -90,6 +77,6 @@
   <xacro:property name="joint_3_lower_limit" value="0.00" />
   <xacro:property name="joint_3_upper_limit" value="${J_PI - 0.05}" />
-  <xacro:property name="joint_3_limit_vel" value="${xacro.arg('elbow_flexion_limit_vel')}" />
-  <xacro:property name="joint_3_limit_effort" value="${xacro.arg('elbow_flexion_limit_effort')}" />
+  <xacro:property name="joint_3_limit_vel_default" value="${duadrive_T120_limit_vel}" />
+  <xacro:property name="joint_3_limit_effort_default" value="${duadrive_T120_limit_effort}" />
   <xacro:property name="joint_3_cam_name" value="${tf_prefix}elbow_camera" />
   <xacro:property name="joint_3_cam_joint_type" value="fixed" />
@@ -104,6 +91,6 @@
   <xacro:property name="joint_4_lower_limit" value="${-J_PI - J_PI/2}" />
   <xacro:property name="joint_4_upper_limit" value="${J_PI + J_PI/2}" />
-  <xacro:property name="joint_4_limit_vel" value="${xacro.arg('forearm_rotation_limit_vel')}" />
-  <xacro:property name="joint_4_limit_effort" value="${xacro.arg('forearm_rotation_limit_effort')}" />
+  <xacro:property name="joint_4_limit_vel_default" value="${duadrive_T40_limit_vel}" />
+  <xacro:property name="joint_4_limit_effort_default" value="${duadrive_T40_limit_effort}" />
   <xacro:property name="joint_5_name" value="${tf_prefix}wrist_flexion" />
   <xacro:property name="joint_5_joint_type" value="revolute" />
@@ -113,6 +100,6 @@
   <xacro:property name="joint_5_lower_limit" value="${-J_PI/2 -0.25}" />
   <xacro:property name="joint_5_upper_limit" value="${J_PI/2 + 0.25}" />
-  <xacro:property name="joint_5_limit_vel" value="${xacro.arg('wrist_flexion_limit_vel')}" />
-  <xacro:property name="joint_5_limit_effort" value="${xacro.arg('wrist_flexion_limit_effort')}" />
+  <xacro:property name="joint_5_limit_vel_default" value="${duadrive_T40_limit_vel}" />
+  <xacro:property name="joint_5_limit_effort_default" value="${duadrive_T40_limit_effort}" />
   <xacro:property name="joint_5_cam_name" value="${tf_prefix}wrist_flexion_camera" />
   <xacro:property name="joint_5_cam_joint_type" value="fixed" />
@@ -127,6 +114,6 @@
   <xacro:property name="joint_6_lower_limit" value="${-J_PI/2}" />
   <xacro:property name="joint_6_upper_limit" value="${J_PI + J_PI/2}" />
-  <xacro:property name="joint_6_limit_vel" value="${xacro.arg('wrist_rotation_limit_vel')}" />
-  <xacro:property name="joint_6_limit_effort" value="${xacro.arg('wrist_rotation_limit_effort')}" />
+  <xacro:property name="joint_6_limit_vel_default" value="${duadrive_T40_limit_vel}" />
+  <xacro:property name="joint_6_limit_effort_default" value="${duadrive_T40_limit_effort}" />
   <xacro:property name="joint_ee_name" value="${tf_prefix}flange_fix_joint" />
   <xacro:property name="joint_ee_xyz" value="0.0 0.0 0.009" />

File: duatic_dynaarm_description/urdf/common/corydoras12/dynaarm_parameters.urdf.xacro (robot description, xacro)
@@ -27,17 +27,4 @@
   <xacro:property name="duadrive_T40_limit_vel" value="13.647" />
   <xacro:property name="duadrive_T40_limit_effort" value="40.0" />
-  <!-- Joint limit overrides (fall back to the drive defaults above if not declared by the caller) -->
-  <xacro:arg name="shoulder_rotation_limit_vel" default="${duadrive_T120_limit_vel}" />
-  <xacro:arg name="shoulder_rotation_limit_effort" default="${duadrive_T120_limit_effort}" />
-  <xacro:arg name="shoulder_flexion_limit_vel" default="${duadrive_T120_limit_vel}" />
-  <xacro:arg name="shoulder_flexion_limit_effort" default="${duadrive_T120_limit_effort}" />
-  <xacro:arg name="elbow_flexion_limit_vel" default="${duadrive_T120_limit_vel}" />
-  <xacro:arg name="elbow_flexion_limit_effort" default="${duadrive_T120_limit_effort}" />
-  <xacro:arg name="forearm_rotation_limit_vel" default="${duadrive_T40_limit_vel}" />
-  <xacro:arg name="forearm_rotation_limit_effort" default="${duadrive_T40_limit_effort}" />
-  <xacro:arg name="wrist_flexion_limit_vel" default="${duadrive_T40_limit_vel}" />
-  <xacro:arg name="wrist_flexion_limit_effort" default="${duadrive_T40_limit_effort}" />
-  <xacro:arg name="wrist_rotation_limit_vel" default="${duadrive_T40_limit_vel}" />
-  <xacro:arg name="wrist_rotation_limit_effort" default="${duadrive_T40_limit_effort}" />
   <!-- Links -->
   <xacro:property name="base" value="${tf_prefix}base" />
@@ -72,6 +59,6 @@
   <xacro:property name="joint_1_lower_limit" value="${-J_PI - J_PI/2 + 0.4}" />
   <xacro:property name="joint_1_upper_limit" value="${J_PI + J_PI/2 - 0.4}" />
-  <xacro:property name="joint_1_limit_vel" value="${xacro.arg('shoulder_rotation_limit_vel')}" />
-  <xacro:property name="joint_1_limit_effort" value="${xacro.arg('shoulder_rotation_limit_effort')}" />
+  <xacro:property name="joint_1_limit_vel_default" value="${duadrive_T120_limit_vel}" />
+  <xacro:property name="joint_1_limit_effort_default" value="${duadrive_T120_limit_effort}" />
   <xacro:property name="joint_2_name" value="${tf_prefix}shoulder_flexion" />
   <xacro:property name="joint_2_joint_type" value="revolute" />
@@ -81,6 +68,6 @@
   <xacro:property name="joint_2_lower_limit" value="${-J_PI/2 - 0.15}" />
   <xacro:property name="joint_2_upper_limit" value="${J_PI/2 + 0.15}" />
-  <xacro:property name="joint_2_limit_vel" value="${xacro.arg('shoulder_flexion_limit_vel')}" />
-  <xacro:property name="joint_2_limit_effort" value="${xacro.arg('shoulder_flexion_limit_effort')}" />
+  <xacro:property name="joint_2_limit_vel_default" value="${duadrive_T120_limit_vel}" />
+  <xacro:property name="joint_2_limit_effort_default" value="${duadrive_T120_limit_effort}" />
   <xacro:property name="joint_3_name" value="${tf_prefix}elbow_flexion" />
   <xacro:property name="joint_3_joint_type" value="revolute" />
@@ -90,6 +77,6 @@
   <xacro:property name="joint_3_lower_limit" value="0.00" />
   <xacro:property name="joint_3_upper_limit" value="${J_PI - 0.05}" />
-  <xacro:property name="joint_3_limit_vel" value="${xacro.arg('elbow_flexion_limit_vel')}" />
-  <xacro:property name="joint_3_limit_effort" value="${xacro.arg('elbow_flexion_limit_effort')}" />
+  <xacro:property name="joint_3_limit_vel_default" value="${duadrive_T120_limit_vel}" />
+  <xacro:property name="joint_3_limit_effort_default" value="${duadrive_T120_limit_effort}" />
   <xacro:property name="joint_3_cam_name" value="${tf_prefix}elbow_camera" />
   <xacro:property name="joint_3_cam_joint_type" value="fixed" />
@@ -104,6 +91,6 @@
   <xacro:property name="joint_4_lower_limit" value="${-J_PI - J_PI/2}" />
   <xacro:property name="joint_4_upper_limit" value="${J_PI + J_PI/2}" />
-  <xacro:property name="joint_4_limit_vel" value="${xacro.arg('forearm_rotation_limit_vel')}" />
-  <xacro:property name="joint_4_limit_effort" value="${xacro.arg('forearm_rotation_limit_effort')}" />
+  <xacro:property name="joint_4_limit_vel_default" value="${duadrive_T40_limit_vel}" />
+  <xacro:property name="joint_4_limit_effort_default" value="${duadrive_T40_limit_effort}" />
   <xacro:property name="joint_5_name" value="${tf_prefix}wrist_flexion" />
   <xacro:property name="joint_5_joint_type" value="revolute" />
@@ -113,6 +100,6 @@
   <xacro:property name="joint_5_lower_limit" value="${-J_PI/2 -0.25}" />
   <xacro:property name="joint_5_upper_limit" value="${J_PI/2 + 0.25}" />
-  <xacro:property name="joint_5_limit_vel" value="${xacro.arg('wrist_flexion_limit_vel')}" />
-  <xacro:property name="joint_5_limit_effort" value="${xacro.arg('wrist_flexion_limit_effort')}" />
+  <xacro:property name="joint_5_limit_vel_default" value="${duadrive_T40_limit_vel}" />
+  <xacro:property name="joint_5_limit_effort_default" value="${duadrive_T40_limit_effort}" />
   <xacro:property name="joint_5_cam_name" value="${tf_prefix}wrist_flexion_camera" />
   <xacro:property name="joint_5_cam_joint_type" value="fixed" />
@@ -127,6 +114,6 @@
   <xacro:property name="joint_6_lower_limit" value="${-J_PI/2}" />
   <xacro:property name="joint_6_upper_limit" value="${J_PI + J_PI/2}" />
-  <xacro:property name="joint_6_limit_vel" value="${xacro.arg('wrist_rotation_limit_vel')}" />
-  <xacro:property name="joint_6_limit_effort" value="${xacro.arg('wrist_rotation_limit_effort')}" />
+  <xacro:property name="joint_6_limit_vel_default" value="${duadrive_T40_limit_vel}" />
+  <xacro:property name="joint_6_limit_effort_default" value="${duadrive_T40_limit_effort}" />
   <xacro:property name="joint_ee_name" value="${tf_prefix}flange_fix_joint" />
   <xacro:property name="joint_ee_xyz" value="0.0 0.0 0.009" />

File: duatic_dynaarm_description/urdf/dynaarm.urdf.xacro (robot description, xacro)
@@ -26,5 +26,19 @@
   <!-- -->
   <xacro:macro name="dynaarm_description"
-    params="tf_prefix parent_link collision:='simple' version *origin">
+    params="tf_prefix parent_link
+      collision:='simple'
+      joint_1_limit_vel=''
+      joint_2_limit_vel=''
+      joint_3_limit_vel=''
+      joint_4_limit_vel=''
+      joint_5_limit_vel=''
+      joint_6_limit_vel=''
+      joint_1_limit_effort=''
+      joint_2_limit_effort=''
+      joint_3_limit_effort=''
+      joint_4_limit_effort=''
+      joint_5_limit_effort=''
+      joint_6_limit_effort=''
+      version *origin">
     <!-- Set ee_parent -->
     <xacro:property name="ee_parent" value="${base}" />
@@ -73,6 +87,6 @@
       joint_lower_limit="${joint_1_lower_limit}"
       joint_upper_limit="${joint_1_upper_limit}"
-      joint_limit_vel="${joint_1_limit_vel}"
-      joint_limit_effort="${joint_1_limit_effort}"
+      joint_limit_vel="${joint_1_limit_vel_default if joint_1_limit_vel == '' else joint_1_limit_vel}"
+      joint_limit_effort="${joint_1_limit_effort_default if joint_1_limit_effort == '' else joint_1_limit_effort}"
       joint_type="${joint_1_joint_type}">
       <origin xyz="${joint_1_origin_xyz}" rpy="${joint_1_origin_rpy}" />
@@ -94,6 +108,6 @@
       joint_lower_limit="${joint_2_lower_limit}"
       joint_upper_limit="${joint_2_upper_limit}"
-      joint_limit_vel="${joint_2_limit_vel}"
-      joint_limit_effort="${joint_2_limit_effort}"
+      joint_limit_vel="${joint_2_limit_vel_default if joint_2_limit_vel == '' else joint_2_limit_vel}"
+      joint_limit_effort="${joint_2_limit_effort_default if joint_2_limit_effort == '' else joint_2_limit_effort}"
       joint_type="${joint_2_joint_type}">
       <origin xyz="${joint_2_origin_xyz}" rpy="${joint_2_origin_rpy}" />
@@ -115,6 +129,6 @@
       joint_lower_limit="${joint_3_lower_limit}"
       joint_upper_limit="${joint_3_upper_limit}"
-      joint_limit_vel="${joint_3_limit_vel}"
-      joint_limit_effort="${joint_3_limit_effort}"
+      joint_limit_vel="${joint_3_limit_vel_default if joint_3_limit_vel == '' else joint_3_limit_vel}"
+      joint_limit_effort="${joint_3_limit_effort_default if joint_3_limit_effort == '' else joint_3_limit_effort}"
       joint_type="${joint_3_joint_type}">
       <origin xyz="${joint_3_origin_xyz}" rpy="${joint_3_origin_rpy}" />
@@ -143,6 +157,6 @@
       joint_lower_limit="${joint_4_lower_limit}"
       joint_upper_limit="${joint_4_upper_limit}"
-      joint_limit_vel="${joint_4_limit_vel}"
-      joint_limit_effort="${joint_4_limit_effort}"
+      joint_limit_vel="${joint_4_limit_vel_default if joint_4_limit_vel == '' else joint_4_limit_vel}"
+      joint_limit_effort="${joint_4_limit_effort_default if joint_4_limit_effort == '' else joint_4_limit_effort}"
       joint_type="${joint_4_joint_type}">
       <origin xyz="${joint_4_origin_xyz}" rpy="${joint_4_origin_rpy}" />
@@ -163,6 +177,6 @@
       joint_lower_limit="${joint_5_lower_limit}"
       joint_upper_limit="${joint_5_upper_limit}"
-      joint_limit_vel="${joint_5_limit_vel}"
-      joint_limit_effort="${joint_5_limit_effort}"
+      joint_limit_vel="${joint_5_limit_vel_default if joint_5_limit_vel == '' else joint_5_limit_vel}"
+      joint_limit_effort="${joint_5_limit_effort_default if joint_5_limit_effort == '' else joint_5_limit_effort}"
       joint_type="${joint_5_joint_type}">
       <origin xyz="${joint_5_origin_xyz}" rpy="${joint_5_origin_rpy}" />
@@ -191,6 +205,6 @@
       joint_lower_limit="${joint_6_lower_limit}"
       joint_upper_limit="${joint_6_upper_limit}"
-      joint_limit_vel="${joint_6_limit_vel}"
-      joint_limit_effort="${joint_6_limit_effort}"
+      joint_limit_vel="${joint_6_limit_vel_default if joint_6_limit_vel == '' else joint_6_limit_vel}"
+      joint_limit_effort="${joint_6_limit_effort_default if joint_6_limit_effort == '' else joint_6_limit_effort}"
       joint_type="${joint_6_joint_type}">
       <origin xyz="${joint_6_origin_xyz}" rpy="${joint_6_origin_rpy}" />

File: duatic_dynaarm_driver/urdf/dynaarm.urdf.xacro (robot description, xacro)
@@ -33,4 +33,16 @@
                          drive_parameter_folder:=''
                          version
+                         joint_1_limit_vel=''
+                         joint_2_limit_vel=''
+                         joint_3_limit_vel=''
+                         joint_4_limit_vel=''
+                         joint_5_limit_vel=''
+                         joint_6_limit_vel=''
+                         joint_1_limit_effort=''
+                         joint_2_limit_effort=''
+                         joint_3_limit_effort=''
+                         joint_4_limit_effort=''
+                         joint_5_limit_effort=''
+                         joint_6_limit_effort=''
                          *origin">
         <xacro:include filename="$(find duatic_dynaarm_description)/urdf/dynaarm.urdf.xacro" />
@@ -46,5 +58,17 @@
                 parent_link="${parent_link}"
                 collision="${collision}"
-                version="${version}">
+                version="${version}"
+                joint_1_limit_vel="${joint_1_limit_vel}"
+                joint_2_limit_vel="${joint_2_limit_vel}"
+                joint_3_limit_vel="${joint_3_limit_vel}"
+                joint_4_limit_vel="${joint_4_limit_vel}"
+                joint_5_limit_vel="${joint_5_limit_vel}"
+                joint_6_limit_vel="${joint_6_limit_vel}"
+                joint_1_limit_effort="${joint_1_limit_effort}"
+                joint_2_limit_effort="${joint_2_limit_effort}"
+                joint_3_limit_effort="${joint_3_limit_effort}"
+                joint_4_limit_effort="${joint_4_limit_effort}"
+                joint_5_limit_effort="${joint_5_limit_effort}"
+                joint_6_limit_effort="${joint_6_limit_effort}">
             <xacro:insert_block name="origin" />
         </xacro:dynaarm_description>
