Commit message: Feat/new meshes (#33)
* Added new meshes

* fixed wrist2 mesh origin

* fixed shoulder

* fix

* Removed unused meshes

* Added base mesh for standalone dynaarm

* Removed collision files

* Fixed orientation

* Removed texture

* feat: widen simple collision mesh of base

---------

Co-authored-by: mbloechli <mbloechlinger@duatic.com>

File: duatic_dynaarm_demo/duatic_dynaarm_single_example/duatic_dynaarm_single_example_description/urdf/dynaarm_single_example.urdf.xacro (robot description, xacro)
@@ -58,5 +58,5 @@
                 ethercat_bus="$(arg ethercat_bus)"
                 version="$(arg version)">
-    <origin xyz="0 0 0" rpy="0.0 0.0 0.0" />
+    <origin xyz="0 0 0.025" rpy="0.0 0.0 0.0" />
   </xacro:dynaarm>
   <!-- Include the control plugin -->

File: duatic_dynaarm_description/urdf/common/baracuda12/dynaarm_parameters.urdf.xacro (robot description, xacro)
@@ -40,11 +40,11 @@
   <xacro:property name="end_effector" value="${tf_prefix}flange" />
   <!-- Meshes -->
-  <xacro:property name="base_mesh" value="base_mesh.dae" />
-  <xacro:property name="link01_mesh" value="shoulder_mesh.dae" />
-  <xacro:property name="link02_mesh" value="upperarm_mesh.dae" />
-  <xacro:property name="link03_mesh" value="elbow_mesh.dae" />
-  <xacro:property name="link04_mesh" value="forearm_mesh.dae" />
-  <xacro:property name="link05_mesh" value="wrist1_mesh.dae" />
-  <xacro:property name="link06_mesh" value="wrist2_mesh.dae" />
+  <xacro:property name="base_mesh" value="${'base_mesh_standalone.glb' if standalone else 'base_mesh_attached.glb'}" />
+  <xacro:property name="link01_mesh" value="shoulder_mesh.glb" />
+  <xacro:property name="link02_mesh" value="upperarm_mesh.glb" />
+  <xacro:property name="link03_mesh" value="elbow_mesh.glb" />
+  <xacro:property name="link04_mesh" value="forearm_mesh.glb" />
+  <xacro:property name="link05_mesh" value="wrist1_mesh.glb" />
+  <xacro:property name="link06_mesh" value="wrist2_mesh.glb" />
   <!-- Joint properties -->
   <xacro:property name="joint_base_name" value="${tf_prefix}joint_base" />
@@ -212,5 +212,5 @@
         <collision>
             <geometry>
-                <cylinder length='0.1' radius='0.05'/>
+                <cylinder length='0.1' radius='0.075'/>
             </geometry>
             <origin xyz='0 0 0.05' rpy='0 0 0'/>
@@ -267,5 +267,6 @@
   </xacro:if>
   <xacro:if value="${collision == 'complex'}">
-    <!-- Collision properties -->
+    <!-- Collision properties: reuse the visual meshes (base_mesh already resolves to the
+         standalone/attached variant) instead of the separate collision_meshes/*.stl files -->
     <xacro:property name="base_collision">
       <collision>
@@ -273,5 +274,5 @@
         <geometry>
           <mesh
-            filename="package://duatic_dynaarm_description/meshes/baracuda12/collision_meshes/base_collision_mesh.stl"
+            filename="package://duatic_dynaarm_description/meshes/${version}/${base_mesh}"
             scale="1 1 1" />
         </geometry>
@@ -283,5 +284,5 @@
         <geometry>
           <mesh
-            filename="package://duatic_dynaarm_description/meshes/baracuda12/collision_meshes/shoulder_collision_mesh.stl"
+            filename="package://duatic_dynaarm_description/meshes/${version}/${link01_mesh}"
             scale="1 1 1" />
         </geometry>
@@ -293,5 +294,5 @@
         <geometry>
           <mesh
-            filename="package://duatic_dynaarm_description/meshes/baracuda12/collision_meshes/upperarm_collision_mesh.stl"
+            filename="package://duatic_dynaarm_description/meshes/${version}/${link02_mesh}"
             scale="1 1 1" />
         </geometry>
@@ -303,5 +304,5 @@
         <geometry>
           <mesh
-            filename="package://duatic_dynaarm_description/meshes/baracuda12/collision_meshes/elbow_collision_mesh.stl"
+            filename="package://duatic_dynaarm_description/meshes/${version}/${link03_mesh}"
             scale="1 1 1" />
         </geometry>
@@ -313,5 +314,5 @@
         <geometry>
           <mesh
-            filename="package://duatic_dynaarm_description/meshes/baracuda12/collision_meshes/forearm_collision_mesh.stl"
+            filename="package://duatic_dynaarm_description/meshes/${version}/${link04_mesh}"
             scale="1 1 1" />
         </geometry>
@@ -323,5 +324,5 @@
         <geometry>
           <mesh
-            filename="package://duatic_dynaarm_description/meshes/baracuda12/collision_meshes/wrist1_collision_mesh.stl"
+            filename="package://duatic_dynaarm_description/meshes/${version}/${link05_mesh}"
             scale="1 1 1" />
         </geometry>
@@ -333,5 +334,5 @@
         <geometry>
           <mesh
-            filename="package://duatic_dynaarm_description/meshes/baracuda12/collision_meshes/wrist2_collision_mesh.stl"
+            filename="package://duatic_dynaarm_description/meshes/${version}/${link06_mesh}"
             scale="1 1 1" />
         </geometry>

File: duatic_dynaarm_description/urdf/common/corydoras12/dynaarm_parameters.urdf.xacro (robot description, xacro)
@@ -40,11 +40,11 @@
   <xacro:property name="end_effector" value="${tf_prefix}flange" />
   <!-- Meshes -->
-  <xacro:property name="base_mesh" value="base_mesh.dae" />
-  <xacro:property name="link01_mesh" value="shoulder_mesh.dae" />
-  <xacro:property name="link02_mesh" value="upperarm_mesh.dae" />
-  <xacro:property name="link03_mesh" value="elbow_mesh.dae" />
-  <xacro:property name="link04_mesh" value="forearm_mesh.dae" />
-  <xacro:property name="link05_mesh" value="wrist1_mesh.dae" />
-  <xacro:property name="link06_mesh" value="wrist2_mesh.dae" />
+  <xacro:property name="base_mesh" value="${'base_mesh_standalone.glb' if standalone else 'base_mesh_attached.glb'}" />
+  <xacro:property name="link01_mesh" value="shoulder_mesh.glb" />
+  <xacro:property name="link02_mesh" value="upperarm_mesh.glb" />
+  <xacro:property name="link03_mesh" value="elbow_mesh.glb" />
+  <xacro:property name="link04_mesh" value="forearm_mesh.glb" />
+  <xacro:property name="link05_mesh" value="wrist1_mesh.glb" />
+  <xacro:property name="link06_mesh" value="wrist2_mesh.glb" />
   <!-- Joint properties -->
   <xacro:property name="joint_base_name" value="${tf_prefix}joint_base" />
@@ -212,5 +212,5 @@
         <collision>
             <geometry>
-                <cylinder length='0.1' radius='0.05'/>
+                <cylinder length='0.1' radius='0.075'/>
             </geometry>
             <origin xyz='0 0 0.05' rpy='0 0 0'/>
@@ -267,5 +267,6 @@
   </xacro:if>
   <xacro:if value="${collision == 'complex'}">
-    <!-- Collision properties -->
+    <!-- Collision properties: reuse the visual meshes (base_mesh already resolves to the
+         standalone/attached variant) instead of the separate collision_meshes/*.stl files -->
     <xacro:property name="base_collision">
       <collision>
@@ -273,5 +274,5 @@
         <geometry>
           <mesh
-            filename="package://duatic_dynaarm_description/meshes/baracuda12/collision_meshes/base_collision_mesh.stl"
+            filename="package://duatic_dynaarm_description/meshes/${version}/${base_mesh}"
             scale="1 1 1" />
         </geometry>
@@ -283,5 +284,5 @@
         <geometry>
           <mesh
-            filename="package://duatic_dynaarm_description/meshes/baracuda12/collision_meshes/shoulder_collision_mesh.stl"
+            filename="package://duatic_dynaarm_description/meshes/${version}/${link01_mesh}"
             scale="1 1 1" />
         </geometry>
@@ -293,5 +294,5 @@
         <geometry>
           <mesh
-            filename="package://duatic_dynaarm_description/meshes/baracuda12/collision_meshes/upperarm_collision_mesh.stl"
+            filename="package://duatic_dynaarm_description/meshes/${version}/${link02_mesh}"
             scale="1 1 1" />
         </geometry>
@@ -303,5 +304,5 @@
         <geometry>
           <mesh
-            filename="package://duatic_dynaarm_description/meshes/baracuda12/collision_meshes/elbow_collision_mesh.stl"
+            filename="package://duatic_dynaarm_description/meshes/${version}/${link03_mesh}"
             scale="1 1 1" />
         </geometry>
@@ -313,5 +314,5 @@
         <geometry>
           <mesh
-            filename="package://duatic_dynaarm_description/meshes/baracuda12/collision_meshes/forearm_collision_mesh.stl"
+            filename="package://duatic_dynaarm_description/meshes/${version}/${link04_mesh}"
             scale="1 1 1" />
         </geometry>
@@ -323,5 +324,5 @@
         <geometry>
           <mesh
-            filename="package://duatic_dynaarm_description/meshes/baracuda12/collision_meshes/wrist1_collision_mesh.stl"
+            filename="package://duatic_dynaarm_description/meshes/${version}/${link05_mesh}"
             scale="1 1 1" />
         </geometry>
@@ -333,5 +334,5 @@
         <geometry>
           <mesh
-            filename="package://duatic_dynaarm_description/meshes/baracuda12/collision_meshes/wrist2_collision_mesh.stl"
+            filename="package://duatic_dynaarm_description/meshes/${version}/${link06_mesh}"
             scale="1 1 1" />
         </geometry>

File: duatic_dynaarm_description/urdf/dynaarm_standalone.urdf.xacro (robot description, xacro)
@@ -37,5 +37,6 @@
                 parent_link="base_link"
                 collision="$(arg collision)"
-                version="$(arg version)">
+                version="$(arg version)"
+                standalone="true">
     <origin xyz="0 0 0" rpy="0.0 0.0 0.0" />
   </xacro:dynaarm_description>

Commit message: introduce limits yaml file

File: duatic_dynaarm_demo/duatic_dynaarm_single_example/duatic_dynaarm_single_example_description/urdf/dynaarm_single_example.urdf.xacro (robot description, xacro)
@@ -35,17 +35,4 @@
   <xacro:arg name="namespace" default="" />
   <xacro:arg name="controller_manager_yaml" default="" />
-  <!-- example definition of custom control limits; remove if not needed -->
-  <xacro:arg name="shoulder_rotation_limit_vel" default="" />
-  <xacro:arg name="shoulder_flexion_limit_vel" default="" />
-  <xacro:arg name="elbow_flexion_limit_vel" default="" />
-  <xacro:arg name="forearm_rotation_limit_vel" default="" />
-  <xacro:arg name="wrist_flexion_limit_vel" default="" />
-  <xacro:arg name="wrist_rotation_limit_vel" default="" />
-  <xacro:arg name="shoulder_rotation_limit_effort" default="" />
-  <xacro:arg name="shoulder_flexion_limit_effort" default="" />
-  <xacro:arg name="elbow_flexion_limit_effort" default="" />
-  <xacro:arg name="forearm_rotation_limit_effort" default="" />
-  <xacro:arg name="wrist_flexion_limit_effort" default="" />
-  <xacro:arg name="wrist_rotation_limit_effort" default="" />
   <!-- load robot description -->
   <xacro:include filename="$(find duatic_dynaarm_driver)/urdf/dynaarm.urdf.xacro" />
@@ -84,17 +71,5 @@
     mode="$(arg mode)"
     ethercat_bus="$(arg ethercat_bus)"
-    version="$(arg version)"
-    joint_1_limit_vel="$(arg shoulder_rotation_limit_vel)"
-    joint_2_limit_vel="$(arg shoulder_flexion_limit_vel)"
-    joint_3_limit_vel="$(arg elbow_flexion_limit_vel)"
-    joint_4_limit_vel="$(arg forearm_rotation_limit_vel)"
-    joint_5_limit_vel="$(arg wrist_flexion_limit_vel)"
-    joint_6_limit_vel="$(arg wrist_rotation_limit_vel)"
-    joint_1_limit_effort="$(arg shoulder_rotation_limit_effort)"
-    joint_2_limit_effort="$(arg shoulder_flexion_limit_effort)"
-    joint_3_limit_effort="$(arg elbow_flexion_limit_effort)"
-    joint_4_limit_effort="$(arg forearm_rotation_limit_effort)"
-    joint_5_limit_effort="$(arg wrist_flexion_limit_effort)"
-    joint_6_limit_effort="$(arg wrist_rotation_limit_effort)">
+    version="$(arg version)">
     <origin xyz="0 0 0" rpy="0.0 0.0 0.0" />
   </xacro:dynaarm>

File: duatic_dynaarm_description/urdf/common/corydoras12/dynaarm_parameters.urdf.xacro (robot description, xacro)
@@ -55,6 +55,4 @@
   <xacro:property name="joint_1_lower_limit" value="${-J_PI - J_PI/2 + 0.4}" />
   <xacro:property name="joint_1_upper_limit" value="${J_PI + J_PI/2 - 0.4}" />
-  <xacro:property name="joint_1_limit_vel_default" value="10.64" />
-  <xacro:property name="joint_1_limit_effort_default" value="120.0" />
   <xacro:property name="joint_2_name" value="${tf_prefix}shoulder_flexion" />
   <xacro:property name="joint_2_joint_type" value="revolute" />
@@ -64,6 +62,4 @@
   <xacro:property name="joint_2_lower_limit" value="${-J_PI/2 - 0.15}" />
   <xacro:property name="joint_2_upper_limit" value="${J_PI/2 + 0.15}" />
-  <xacro:property name="joint_2_limit_vel_default" value="10.64" />
-  <xacro:property name="joint_2_limit_effort_default" value="120.0" />
   <xacro:property name="joint_3_name" value="${tf_prefix}elbow_flexion" />
   <xacro:property name="joint_3_joint_type" value="revolute" />
@@ -73,6 +69,4 @@
   <xacro:property name="joint_3_lower_limit" value="0.00" />
   <xacro:property name="joint_3_upper_limit" value="${J_PI - 0.05}" />
-  <xacro:property name="joint_3_limit_vel_default" value="10.64" />
-  <xacro:property name="joint_3_limit_effort_default" value="120.0" />
   <xacro:property name="joint_3_cam_name" value="${tf_prefix}elbow_camera" />
   <xacro:property name="joint_3_cam_joint_type" value="fixed" />
@@ -87,6 +81,4 @@
   <xacro:property name="joint_4_lower_limit" value="${-J_PI - J_PI/2}" />
   <xacro:property name="joint_4_upper_limit" value="${J_PI + J_PI/2}" />
-  <xacro:property name="joint_4_limit_vel_default" value="13.647" />
-  <xacro:property name="joint_4_limit_effort_default" value="40.0" />
   <xacro:property name="joint_5_name" value="${tf_prefix}wrist_flexion" />
   <xacro:property name="joint_5_joint_type" value="revolute" />
@@ -96,6 +88,4 @@
   <xacro:property name="joint_5_lower_limit" value="${-J_PI/2 -0.25}" />
   <xacro:property name="joint_5_upper_limit" value="${J_PI/2 + 0.25}" />
-  <xacro:property name="joint_5_limit_vel_default" value="13.647" />
-  <xacro:property name="joint_5_limit_effort_default" value="40.0" />
   <xacro:property name="joint_5_cam_name" value="${tf_prefix}wrist_flexion_camera" />
   <xacro:property name="joint_5_cam_joint_type" value="fixed" />
@@ -110,6 +100,4 @@
   <xacro:property name="joint_6_lower_limit" value="${-J_PI/2}" />
   <xacro:property name="joint_6_upper_limit" value="${J_PI + J_PI/2}" />
-  <xacro:property name="joint_6_limit_vel_default" value="13.647" />
-  <xacro:property name="joint_6_limit_effort_default" value="40.0" />
   <xacro:property name="joint_ee_name" value="${tf_prefix}flange_fix_joint" />
   <xacro:property name="joint_ee_xyz" value="0.0 0.0 0.009" />

File: duatic_dynaarm_description/urdf/dynaarm.urdf.xacro (robot description, xacro)
@@ -30,16 +30,5 @@
       version
       standalone:='true'
-      joint_1_limit_vel=''
-      joint_2_limit_vel=''
-      joint_3_limit_vel=''
-      joint_4_limit_vel=''
-      joint_5_limit_vel=''
-      joint_6_limit_vel=''
-      joint_1_limit_effort=''
-      joint_2_limit_effort=''
-      joint_3_limit_effort=''
-      joint_4_limit_effort=''
-      joint_5_limit_effort=''
-      joint_6_limit_effort=''
+      joint_limits:=${xacro.load_yaml('$(find duatic_dynaarm_description)/config/limits/limits.yaml')}
       *origin">
     <!-- Set ee_parent -->
@@ -89,6 +78,6 @@
       joint_lower_limit="${joint_1_lower_limit}"
       joint_upper_limit="${joint_1_upper_limit}"
-      joint_limit_vel="${joint_1_limit_vel_default if joint_1_limit_vel == '' else joint_1_limit_vel}"
-      joint_limit_effort="${joint_1_limit_effort_default if joint_1_limit_effort == '' else joint_1_limit_effort}"
+      joint_limit_vel="${joint_limits['shoulder_rotation']['max_joint_velocity']}"
+      joint_limit_effort="${joint_limits['shoulder_rotation']['max_joint_effort']}"
       joint_type="${joint_1_joint_type}">
       <origin xyz="${joint_1_origin_xyz}" rpy="${joint_1_origin_rpy}" />
@@ -110,6 +99,6 @@
       joint_lower_limit="${joint_2_lower_limit}"
       joint_upper_limit="${joint_2_upper_limit}"
-      joint_limit_vel="${joint_2_limit_vel_default if joint_2_limit_vel == '' else joint_2_limit_vel}"
-      joint_limit_effort="${joint_2_limit_effort_default if joint_2_limit_effort == '' else joint_2_limit_effort}"
+      joint_limit_vel="${joint_limits['shoulder_flexion']['max_joint_velocity']}"
+      joint_limit_effort="${joint_limits['shoulder_flexion']['max_joint_effort']}"
       joint_type="${joint_2_joint_type}">
       <origin xyz="${joint_2_origin_xyz}" rpy="${joint_2_origin_rpy}" />
@@ -131,6 +120,6 @@
       joint_lower_limit="${joint_3_lower_limit}"
       joint_upper_limit="${joint_3_upper_limit}"
-      joint_limit_vel="${joint_3_limit_vel_default if joint_3_limit_vel == '' else joint_3_limit_vel}"
-      joint_limit_effort="${joint_3_limit_effort_default if joint_3_limit_effort == '' else joint_3_limit_effort}"
+      joint_limit_vel="${joint_limits['elbow_flexion']['max_joint_velocity']}"
+      joint_limit_effort="${joint_limits['elbow_flexion']['max_joint_effort']}"
       joint_type="${joint_3_joint_type}">
       <origin xyz="${joint_3_origin_xyz}" rpy="${joint_3_origin_rpy}" />
@@ -159,6 +148,6 @@
       joint_lower_limit="${joint_4_lower_limit}"
       joint_upper_limit="${joint_4_upper_limit}"
-      joint_limit_vel="${joint_4_limit_vel_default if joint_4_limit_vel == '' else joint_4_limit_vel}"
-      joint_limit_effort="${joint_4_limit_effort_default if joint_4_limit_effort == '' else joint_4_limit_effort}"
+      joint_limit_vel="${joint_limits['forearm_rotation']['max_joint_velocity']}"
+      joint_limit_effort="${joint_limits['forearm_rotation']['max_joint_effort']}"
       joint_type="${joint_4_joint_type}">
       <origin xyz="${joint_4_origin_xyz}" rpy="${joint_4_origin_rpy}" />
@@ -179,6 +168,6 @@
       joint_lower_limit="${joint_5_lower_limit}"
       joint_upper_limit="${joint_5_upper_limit}"
-      joint_limit_vel="${joint_5_limit_vel_default if joint_5_limit_vel == '' else joint_5_limit_vel}"
-      joint_limit_effort="${joint_5_limit_effort_default if joint_5_limit_effort == '' else joint_5_limit_effort}"
+      joint_limit_vel="${joint_limits['wrist_flexion']['max_joint_velocity']}"
+      joint_limit_effort="${joint_limits['wrist_flexion']['max_joint_effort']}"
       joint_type="${joint_5_joint_type}">
       <origin xyz="${joint_5_origin_xyz}" rpy="${joint_5_origin_rpy}" />
@@ -207,6 +196,6 @@
       joint_lower_limit="${joint_6_lower_limit}"
       joint_upper_limit="${joint_6_upper_limit}"
-      joint_limit_vel="${joint_6_limit_vel_default if joint_6_limit_vel == '' else joint_6_limit_vel}"
-      joint_limit_effort="${joint_6_limit_effort_default if joint_6_limit_effort == '' else joint_6_limit_effort}"
+      joint_limit_vel="${joint_limits['wrist_rotation']['max_joint_velocity']}"
+      joint_limit_effort="${joint_limits['wrist_rotation']['max_joint_effort']}"
       joint_type="${joint_6_joint_type}">
       <origin xyz="${joint_6_origin_xyz}" rpy="${joint_6_origin_rpy}" />

File: duatic_dynaarm_driver/urdf/dynaarm.urdf.xacro (robot description, xacro)
@@ -33,16 +33,5 @@
                          drive_parameter_folder:=''
                          version
-                         joint_1_limit_vel=''
-                         joint_2_limit_vel=''
-                         joint_3_limit_vel=''
-                         joint_4_limit_vel=''
-                         joint_5_limit_vel=''
-                         joint_6_limit_vel=''
-                         joint_1_limit_effort=''
-                         joint_2_limit_effort=''
-                         joint_3_limit_effort=''
-                         joint_4_limit_effort=''
-                         joint_5_limit_effort=''
-                         joint_6_limit_effort=''
+                         joint_limits:=${xacro.load_yaml('$(find duatic_dynaarm_description)/config/limits/limits.yaml')}
                          *origin">
         <xacro:include filename="$(find duatic_dynaarm_description)/urdf/dynaarm.urdf.xacro" />
@@ -59,16 +48,5 @@
                 collision="${collision}"
                 version="${version}"
-                joint_1_limit_vel="${joint_1_limit_vel}"
-                joint_2_limit_vel="${joint_2_limit_vel}"
-                joint_3_limit_vel="${joint_3_limit_vel}"
-                joint_4_limit_vel="${joint_4_limit_vel}"
-                joint_5_limit_vel="${joint_5_limit_vel}"
-                joint_6_limit_vel="${joint_6_limit_vel}"
-                joint_1_limit_effort="${joint_1_limit_effort}"
-                joint_2_limit_effort="${joint_2_limit_effort}"
-                joint_3_limit_effort="${joint_3_limit_effort}"
-                joint_4_limit_effort="${joint_4_limit_effort}"
-                joint_5_limit_effort="${joint_5_limit_effort}"
-                joint_6_limit_effort="${joint_6_limit_effort}">
+                joint_limits="${joint_limits}">
             <xacro:insert_block name="origin" />
         </xacro:dynaarm_description>
