Commit message: revert: seperate out indent change not to be done in this PR

File: duatic_dynaarm_demo/duatic_dynaarm_single_example/duatic_dynaarm_single_example_description/urdf/dynaarm_single_example.urdf.xacro (robot description, xacro)
@@ -2,25 +2,12 @@
 <!--
 Copyright 2025 Duatic AG
-Redistribution and use in source and binary forms, with or without modification, are permitted
-provided that the following conditions are met:
-1. Redistributions of source code must retain the above copyright notice, this list of conditions
-and the following disclaimer.
-2. Redistributions in binary form must reproduce the above copyright notice, this list of
-conditions and the following disclaimer in the documentation and/or other materials provided with
-the distribution.
-3. Neither the name of the copyright holder nor the names of its contributors may be used to
-endorse or promote products derived from this software without specific prior written permission.
-THIS SOFTWARE IS PROVIDED BY THE COPYRIGHT HOLDERS AND CONTRIBUTORS “AS IS” AND ANY EXPRESS OR
-IMPLIED WARRANTIES, INCLUDING, BUT NOT LIMITED TO, THE IMPLIED WARRANTIES OF MERCHANTABILITY AND
-FITNESS FOR A PARTICULAR PURPOSE ARE DISCLAIMED. IN NO EVENT SHALL THE COPYRIGHT HOLDER OR
-CONTRIBUTORS BE LIABLE FOR ANY DIRECT, INDIRECT, INCIDENTAL, SPECIAL, EXEMPLARY, OR CONSEQUENTIAL
-DAMAGES (INCLUDING, BUT NOT LIMITED TO, PROCUREMENT OF SUBSTITUTE GOODS OR SERVICES; LOSS OF USE,
-DATA, OR PROFITS; OR BUSINESS INTERRUPTION) HOWEVER CAUSED AND ON ANY THEORY OF LIABILITY, WHETHER
-IN CONTRACT, STRICT LIABILITY, OR TORT (INCLUDING NEGLIGENCE OR OTHERWISE) ARISING IN ANY WAY OUT
-OF
-THE USE OF THIS SOFTWARE, EVEN IF ADVISED OF THE POSSIBILITY OF SUCH DAMAGE.
+Redistribution and use in source and binary forms, with or without modification, are permitted provided that the following conditions are met:
+1. Redistributions of source code must retain the above copyright notice, this list of conditions and the following disclaimer.
+2. Redistributions in binary form must reproduce the above copyright notice, this list of conditions and the following disclaimer in the documentation and/or other materials provided with the distribution.
+3. Neither the name of the copyright holder nor the names of its contributors may be used to endorse or promote products derived from this software without specific prior written permission.
+THIS SOFTWARE IS PROVIDED BY THE COPYRIGHT HOLDERS AND CONTRIBUTORS “AS IS” AND ANY EXPRESS OR IMPLIED WARRANTIES, INCLUDING, BUT NOT LIMITED TO, THE IMPLIED WARRANTIES OF MERCHANTABILITY AND FITNESS FOR A PARTICULAR PURPOSE ARE DISCLAIMED. IN NO EVENT SHALL THE COPYRIGHT HOLDER OR CONTRIBUTORS BE LIABLE FOR ANY DIRECT, INDIRECT, INCIDENTAL, SPECIAL, EXEMPLARY, OR CONSEQUENTIAL DAMAGES (INCLUDING, BUT NOT LIMITED TO, PROCUREMENT OF SUBSTITUTE GOODS OR SERVICES; LOSS OF USE, DATA, OR PROFITS; OR BUSINESS INTERRUPTION) HOWEVER CAUSED AND ON ANY THEORY OF LIABILITY, WHETHER IN CONTRACT, STRICT LIABILITY, OR TORT (INCLUDING NEGLIGENCE OR OTHERWISE) ARISING IN ANY WAY OUT OF THE USE OF THIS SOFTWARE, EVEN IF ADVISED OF THE POSSIBILITY OF SUCH DAMAGE.
 -->
 <robot name="dynaarm" xmlns:xacro="http://www.ros.org/wiki/xacro">
-  <!-- Example single arm setup -->
+  <!--Example single arm setup-->
   <xacro:arg name="tf_prefix" default="" />
   <!-- simple, complex -->
@@ -35,41 +22,40 @@
   <xacro:arg name="namespace" default="" />
   <xacro:arg name="controller_manager_yaml" default="" />
-  <!-- load robot description -->
   <xacro:include filename="$(find duatic_dynaarm_driver)/urdf/dynaarm.urdf.xacro" />
-  <link name="base_link" />
+<link name="base_link" />
   <link name="table">
     <visual>
       <origin xyz="0 0 0" rpy="0 0 0" />
       <geometry>
-        <box size="1.0 1.0 0.05" />
+          <box size="1.0 1.0 0.05"/>
       </geometry>
       <material name="Wood">
-        <color rgba="0.9 0.83 0.733 1.0" />
+        <color rgba="0.9 0.83 0.733 1.0"/>
       </material>
     </visual>
     <collision>
-      <origin xyz="0 0 0" rpy="0 0 0" />
+      <origin xyz="0 0 0" rpy="0 0 0"/>
       <geometry>
-        <box size="1.0 1.0 0.05" />
+          <box size="1.0 1.0 0.05"/>
       </geometry>
     </collision>
     <inertial>
-      <mass value="10.0" />
-      <origin xyz="0 0 0" />
-      <inertia ixx="1.0" ixy="0.0" ixz="0.0" iyy="1.0" iyz="0.0" izz="1.0" />
+      <mass value="10.0"/>
+      <origin xyz="0 0 0"/>
+      <inertia ixx="1.0" ixy="0.0" ixz="0.0" iyy="1.0" iyz="0.0" izz="1.0"/>
     </inertial>
   </link>
   <joint name="table_joint" type="fixed">
-    <parent link="base_link" />
-    <child link="table" />
-    <origin xyz="0 0 -0.025" rpy="0 0 0" />
+    <parent link="base_link"/>
+    <child link="table"/>
+    <origin xyz="0 0 -0.025" rpy="0 0 0"/>
   </joint>
   <!-- create an instance of the dynaarm and fix its base-->
   <xacro:dynaarm tf_prefix="$(arg tf_prefix)"
-    parent_link="table"
-    collision="$(arg collision)"
-    mode="$(arg mode)"
-    ethercat_bus="$(arg ethercat_bus)"
-    version="$(arg version)">
+                parent_link="table"
+                collision="$(arg collision)"
+                mode="$(arg mode)"
+                ethercat_bus="$(arg ethercat_bus)"
+                version="$(arg version)">
     <origin xyz="0 0 0" rpy="0.0 0.0 0.0" />
   </xacro:dynaarm>
@@ -77,4 +63,4 @@
   <xacro:include filename="$(find duatic_control)/urdf/plugins.urdf.xacro" />
   <xacro:control namespace="$(arg namespace)"
-    controller_manager_yaml="$(arg controller_manager_yaml)" />
+                controller_manager_yaml="$(arg controller_manager_yaml)" />
 </robot>

Commit message: feat(description): override joint limits from an optional yaml file
The joint velocity and effort limits came from a single limits.yaml
that had to list every joint and replaced the per-version values.
Add a joint_limits_override parameter to the dynaarm and
dynaarm_description macros that takes the path of a yaml file. Values
it sets replace the version defaults, and joints or values it leaves
out keep them. Remove limits.yaml and add an example override file to
the single example, which exposes the path as a xacro arg.

File: duatic_dynaarm_demo/duatic_dynaarm_single_example/duatic_dynaarm_single_example_description/urdf/dynaarm_single_example.urdf.xacro (robot description, xacro)
@@ -19,4 +19,6 @@
   <!-- v1, v2, ... -->
   <xacro:arg name="version" default="corydoras12" />
+  <!-- path to a yaml file to override joint velocity and effort limits -->
+  <xacro:arg name="joint_limits_override" default="" />
   <!-- Only relevant for Gazebo -->
   <xacro:arg name="namespace" default="" />
@@ -57,5 +59,6 @@
                 mode="$(arg mode)"
                 ethercat_bus="$(arg ethercat_bus)"
-                version="$(arg version)">
+                version="$(arg version)"
+                joint_limits_override="$(arg joint_limits_override)">
     <origin xyz="0 0 0" rpy="0.0 0.0 0.0" />
   </xacro:dynaarm>

File: duatic_dynaarm_description/urdf/dynaarm.urdf.xacro (robot description, xacro)
@@ -27,5 +27,5 @@
   <xacro:macro name="dynaarm_description"
     params="tf_prefix parent_link collision:='simple' version standalone:=true
-      joint_limits:=${xacro.load_yaml('$(find duatic_dynaarm_description)/config/limits/limits.yaml')}
+      joint_limits_override:=''
       *origin">
     <!-- Set ee_parent -->
@@ -34,4 +34,6 @@
     <!-- Include the version specific information and also load the ethercat addresses from the drive file -->
     <xacro:include filename="$(find duatic_dynaarm_description)/urdf/common/${version}/dynaarm_parameters.urdf.xacro" />
+    <!-- Per joint velocity and effort limits that replace the version defaults -->
+    <xacro:property name="joint_limits" value="${xacro.load_yaml(joint_limits_override) if joint_limits_override else dict()}" />
     <xacro:dynaarm_joint_fixed joint_name="${joint_base_name}"
       parent="${parent_link}"
@@ -72,6 +74,6 @@
       joint_lower_limit="${joint_1_lower_limit}"
       joint_upper_limit="${joint_1_upper_limit}"
-      joint_limit_vel="${joint_limits['shoulder_rotation']['max_joint_velocity']}"
-      joint_limit_effort="${joint_limits['shoulder_rotation']['max_joint_effort']}"
+      joint_limit_vel="${joint_limits.get('shoulder_rotation', dict()).get('max_velocity', joint_1_limit_vel)}"
+      joint_limit_effort="${joint_limits.get('shoulder_rotation', dict()).get('max_effort', joint_1_limit_effort)}"
       joint_type="${joint_1_joint_type}">
       <origin xyz="${joint_1_origin_xyz}" rpy="${joint_1_origin_rpy}" />
@@ -93,6 +95,6 @@
       joint_lower_limit="${joint_2_lower_limit}"
       joint_upper_limit="${joint_2_upper_limit}"
-      joint_limit_vel="${joint_limits['shoulder_flexion']['max_joint_velocity']}"
-      joint_limit_effort="${joint_limits['shoulder_flexion']['max_joint_effort']}"
+      joint_limit_vel="${joint_limits.get('shoulder_flexion', dict()).get('max_velocity', joint_2_limit_vel)}"
+      joint_limit_effort="${joint_limits.get('shoulder_flexion', dict()).get('max_effort', joint_2_limit_effort)}"
       joint_type="${joint_2_joint_type}">
       <origin xyz="${joint_2_origin_xyz}" rpy="${joint_2_origin_rpy}" />
@@ -114,6 +116,6 @@
       joint_lower_limit="${joint_3_lower_limit}"
       joint_upper_limit="${joint_3_upper_limit}"
-      joint_limit_vel="${joint_limits['elbow_flexion']['max_joint_velocity']}"
-      joint_limit_effort="${joint_limits['elbow_flexion']['max_joint_effort']}"
+      joint_limit_vel="${joint_limits.get('elbow_flexion', dict()).get('max_velocity', joint_3_limit_vel)}"
+      joint_limit_effort="${joint_limits.get('elbow_flexion', dict()).get('max_effort', joint_3_limit_effort)}"
       joint_type="${joint_3_joint_type}">
       <origin xyz="${joint_3_origin_xyz}" rpy="${joint_3_origin_rpy}" />
@@ -142,6 +144,6 @@
       joint_lower_limit="${joint_4_lower_limit}"
       joint_upper_limit="${joint_4_upper_limit}"
-      joint_limit_vel="${joint_limits['forearm_rotation']['max_joint_velocity']}"
-      joint_limit_effort="${joint_limits['forearm_rotation']['max_joint_effort']}"
+      joint_limit_vel="${joint_limits.get('forearm_rotation', dict()).get('max_velocity', joint_4_limit_vel)}"
+      joint_limit_effort="${joint_limits.get('forearm_rotation', dict()).get('max_effort', joint_4_limit_effort)}"
       joint_type="${joint_4_joint_type}">
       <origin xyz="${joint_4_origin_xyz}" rpy="${joint_4_origin_rpy}" />
@@ -162,6 +164,6 @@
       joint_lower_limit="${joint_5_lower_limit}"
       joint_upper_limit="${joint_5_upper_limit}"
-      joint_limit_vel="${joint_limits['wrist_flexion']['max_joint_velocity']}"
-      joint_limit_effort="${joint_limits['wrist_flexion']['max_joint_effort']}"
+      joint_limit_vel="${joint_limits.get('wrist_flexion', dict()).get('max_velocity', joint_5_limit_vel)}"
+      joint_limit_effort="${joint_limits.get('wrist_flexion', dict()).get('max_effort', joint_5_limit_effort)}"
       joint_type="${joint_5_joint_type}">
       <origin xyz="${joint_5_origin_xyz}" rpy="${joint_5_origin_rpy}" />
@@ -190,6 +192,6 @@
       joint_lower_limit="${joint_6_lower_limit}"
       joint_upper_limit="${joint_6_upper_limit}"
-      joint_limit_vel="${joint_limits['wrist_rotation']['max_joint_velocity']}"
-      joint_limit_effort="${joint_limits['wrist_rotation']['max_joint_effort']}"
+      joint_limit_vel="${joint_limits.get('wrist_rotation', dict()).get('max_velocity', joint_6_limit_vel)}"
+      joint_limit_effort="${joint_limits.get('wrist_rotation', dict()).get('max_effort', joint_6_limit_effort)}"
       joint_type="${joint_6_joint_type}">
       <origin xyz="${joint_6_origin_xyz}" rpy="${joint_6_origin_rpy}" />

File: duatic_dynaarm_driver/urdf/dynaarm.urdf.xacro (robot description, xacro)
@@ -33,5 +33,5 @@
                          drive_parameter_folder:=''
                          version
-                         joint_limits:=${xacro.load_yaml('$(find duatic_dynaarm_description)/config/limits/limits.yaml')}
+                         joint_limits_override:=''
                          *origin">
         <xacro:include filename="$(find duatic_dynaarm_description)/urdf/dynaarm.urdf.xacro" />
@@ -48,5 +48,5 @@
                 collision="${collision}"
                 version="${version}"
-                joint_limits="${joint_limits}">
+                joint_limits_override="${joint_limits_override}">
             <xacro:insert_block name="origin" />
         </xacro:dynaarm_description>

Commit message: refactor(description): rename joint_limits_override to joint_limits_yaml

File: duatic_dynaarm_demo/duatic_dynaarm_single_example/duatic_dynaarm_single_example_description/urdf/dynaarm_single_example.urdf.xacro (robot description, xacro)
@@ -19,6 +19,6 @@
   <!-- v1, v2, ... -->
   <xacro:arg name="version" default="corydoras12" />
-  <!-- path to a yaml file to override joint velocity and effort limits -->
-  <xacro:arg name="joint_limits_override" default="" />
+  <!-- path to a yaml file to use custom joint velocity and effort limits -->
+  <xacro:arg name="joint_limits_yaml" default="" />
   <!-- Only relevant for Gazebo -->
   <xacro:arg name="namespace" default="" />
@@ -60,5 +60,5 @@
                 ethercat_bus="$(arg ethercat_bus)"
                 version="$(arg version)"
-                joint_limits_override="$(arg joint_limits_override)">
+                joint_limits_yaml="$(arg joint_limits_yaml)">
     <origin xyz="0 0 0" rpy="0.0 0.0 0.0" />
   </xacro:dynaarm>

File: duatic_dynaarm_description/urdf/dynaarm.urdf.xacro (robot description, xacro)
@@ -27,5 +27,5 @@
   <xacro:macro name="dynaarm_description"
     params="tf_prefix parent_link collision:='simple' version standalone:=true
-      joint_limits_override:=''
+      joint_limits_yaml:=''
       *origin">
     <!-- Set ee_parent -->
@@ -34,6 +34,6 @@
     <!-- Include the version specific information and also load the ethercat addresses from the drive file -->
     <xacro:include filename="$(find duatic_dynaarm_description)/urdf/common/${version}/dynaarm_parameters.urdf.xacro" />
-    <!-- Per joint velocity and effort limits that replace the version defaults -->
-    <xacro:property name="joint_limits" value="${xacro.load_yaml(joint_limits_override) if joint_limits_override else dict()}" />
+    <!-- Per joint velocity and effort limits that replace the defaults -->
+    <xacro:property name="joint_limits" value="${xacro.load_yaml(joint_limits_yaml) if joint_limits_yaml else dict()}" />
     <xacro:dynaarm_joint_fixed joint_name="${joint_base_name}"
       parent="${parent_link}"

File: duatic_dynaarm_driver/urdf/dynaarm.urdf.xacro (robot description, xacro)
@@ -33,5 +33,5 @@
                          drive_parameter_folder:=''
                          version
-                         joint_limits_override:=''
+                         joint_limits_yaml:=''
                          *origin">
         <xacro:include filename="$(find duatic_dynaarm_description)/urdf/dynaarm.urdf.xacro" />
@@ -48,5 +48,5 @@
                 collision="${collision}"
                 version="${version}"
-                joint_limits_override="${joint_limits_override}">
+                joint_limits_yaml="${joint_limits_yaml}">
             <xacro:insert_block name="origin" />
         </xacro:dynaarm_description>
