Commit message: feat(control): Read and apply joint limits from the URDF (#25)
Co-authored-by: Lennart Nachtigall <mail@firesurfer.de>
Co-authored-by: Patrick Vonwirth <pvonwirth@duatic.com>
Co-authored-by: Marc Blöchlinger <mbloechlinger@duatic.com>

File: duatic_dynaarm_demo/duatic_dynaarm_single_example/duatic_dynaarm_single_example_description/urdf/dynaarm_single_example.urdf.xacro (robot description, xacro)
@@ -19,4 +19,6 @@
   <!-- v1, v2, ... -->
   <xacro:arg name="version" default="corydoras12" />
+  <!-- path to a yaml file to use custom joint velocity and effort limits -->
+  <xacro:arg name="joint_limits_yaml" default="" />
   <!-- Only relevant for Gazebo -->
   <xacro:arg name="namespace" default="" />
@@ -57,6 +59,7 @@
                 mode="$(arg mode)"
                 ethercat_bus="$(arg ethercat_bus)"
-                version="$(arg version)">
-    <origin xyz="0 0 0.025" rpy="0.0 0.0 0.0" />
+                version="$(arg version)"
+                joint_limits_yaml="$(arg joint_limits_yaml)">
+    <origin xyz="0 0 0" rpy="0.0 0.0 0.0" />
   </xacro:dynaarm>
   <!-- Include the control plugin -->

File: duatic_dynaarm_description/urdf/common/baracuda12/dynaarm_parameters.urdf.xacro (robot description, xacro)
@@ -22,8 +22,5 @@
 -->
 <robot xmlns:xacro="http://www.ros.org/wiki/xacro">
-  <xacro:property name="arm_version_name" value="baracuda12"/>
   <xacro:property name="J_PI" value="3.14159265359" />
-  <xacro:property name="baboon_peak_torque" value="40" />
-  <xacro:property name="baboon_max_speed" value="4" />
   <xacro:property name="mm2_to_m2" value="0.000001" />
   <xacro:property name="mm_to_m" value="0.001" />
@@ -60,4 +57,6 @@
   <xacro:property name="joint_1_lower_limit" value="${-J_PI - J_PI/2 + 0.4}" />
   <xacro:property name="joint_1_upper_limit" value="${J_PI + J_PI/2 - 0.4}" />
+  <xacro:property name="joint_1_limit_vel" value="10.64" />
+  <xacro:property name="joint_1_limit_effort" value="120.0" />
   <xacro:property name="joint_2_name" value="${tf_prefix}shoulder_flexion" />
   <xacro:property name="joint_2_joint_type" value="revolute" />
@@ -67,4 +66,6 @@
   <xacro:property name="joint_2_lower_limit" value="${-J_PI/2 - 0.15}" />
   <xacro:property name="joint_2_upper_limit" value="${J_PI/2 + 0.15}" />
+  <xacro:property name="joint_2_limit_vel" value="10.64" />
+  <xacro:property name="joint_2_limit_effort" value="120.0" />
   <xacro:property name="joint_3_name" value="${tf_prefix}elbow_flexion" />
   <xacro:property name="joint_3_joint_type" value="revolute" />
@@ -74,4 +75,6 @@
   <xacro:property name="joint_3_lower_limit" value="0.00" />
   <xacro:property name="joint_3_upper_limit" value="${J_PI - 0.05}" />
+  <xacro:property name="joint_3_limit_vel" value="10.64" />
+  <xacro:property name="joint_3_limit_effort" value="120.0" />
   <xacro:property name="joint_3_cam_name" value="${tf_prefix}elbow_camera" />
   <xacro:property name="joint_3_cam_joint_type" value="fixed" />
@@ -86,4 +89,6 @@
   <xacro:property name="joint_4_lower_limit" value="${-J_PI - J_PI/2}" />
   <xacro:property name="joint_4_upper_limit" value="${J_PI + J_PI/2}" />
+  <xacro:property name="joint_4_limit_vel" value="13.647" />
+  <xacro:property name="joint_4_limit_effort" value="40.0" />
   <xacro:property name="joint_5_name" value="${tf_prefix}wrist_flexion" />
   <xacro:property name="joint_5_joint_type" value="revolute" />
@@ -93,4 +98,6 @@
   <xacro:property name="joint_5_lower_limit" value="${-J_PI/2 -0.25}" />
   <xacro:property name="joint_5_upper_limit" value="${J_PI/2 + 0.25}" />
+  <xacro:property name="joint_5_limit_vel" value="13.647" />
+  <xacro:property name="joint_5_limit_effort" value="40.0" />
   <xacro:property name="joint_5_cam_name" value="${tf_prefix}wrist_flexion_camera" />
   <xacro:property name="joint_5_cam_joint_type" value="fixed" />
@@ -105,4 +112,6 @@
   <xacro:property name="joint_6_lower_limit" value="${-J_PI/2}" />
   <xacro:property name="joint_6_upper_limit" value="${J_PI + J_PI/2}" />
+  <xacro:property name="joint_6_limit_vel" value="13.647" />
+  <xacro:property name="joint_6_limit_effort" value="40.0" />
   <xacro:property name="joint_ee_name" value="${tf_prefix}flange_fix_joint" />
   <xacro:property name="joint_ee_xyz" value="0.0 0.0 0.009" />

File: duatic_dynaarm_description/urdf/dynaarm.urdf.xacro (robot description, xacro)
@@ -26,5 +26,7 @@
   <!-- -->
   <xacro:macro name="dynaarm_description"
-    params="tf_prefix parent_link collision:='simple' version standalone:=true *origin">
+    params="tf_prefix parent_link collision:='simple' version standalone:=true
+      joint_limits_yaml:=''
+      *origin">
     <!-- Set ee_parent -->
     <xacro:property name="ee_parent" value="${base}" />
@@ -32,4 +34,6 @@
     <!-- Include the version specific information and also load the ethercat addresses from the drive file -->
     <xacro:include filename="$(find duatic_dynaarm_description)/urdf/common/${version}/dynaarm_parameters.urdf.xacro" />
+    <!-- Per joint velocity and effort limits that replace the defaults -->
+    <xacro:property name="joint_limits" value="${xacro.load_yaml(joint_limits_yaml) if joint_limits_yaml else dict()}" />
     <xacro:dynaarm_joint_fixed joint_name="${joint_base_name}"
       parent="${parent_link}"
@@ -70,6 +74,6 @@
       joint_lower_limit="${joint_1_lower_limit}"
       joint_upper_limit="${joint_1_upper_limit}"
-      joint_limit_vel="${baboon_max_speed}"
-      joint_limit_effort="${baboon_peak_torque}"
+      joint_limit_vel="${joint_limits.get(joint_1_name, dict()).get('max_velocity', joint_1_limit_vel)}"
+      joint_limit_effort="${joint_limits.get(joint_1_name, dict()).get('max_effort', joint_1_limit_effort)}"
       joint_type="${joint_1_joint_type}">
       <origin xyz="${joint_1_origin_xyz}" rpy="${joint_1_origin_rpy}" />
@@ -91,6 +95,6 @@
       joint_lower_limit="${joint_2_lower_limit}"
       joint_upper_limit="${joint_2_upper_limit}"
-      joint_limit_vel="${baboon_max_speed}"
-      joint_limit_effort="${baboon_peak_torque}"
+      joint_limit_vel="${joint_limits.get(joint_2_name, dict()).get('max_velocity', joint_2_limit_vel)}"
+      joint_limit_effort="${joint_limits.get(joint_2_name, dict()).get('max_effort', joint_2_limit_effort)}"
       joint_type="${joint_2_joint_type}">
       <origin xyz="${joint_2_origin_xyz}" rpy="${joint_2_origin_rpy}" />
@@ -112,6 +116,6 @@
       joint_lower_limit="${joint_3_lower_limit}"
       joint_upper_limit="${joint_3_upper_limit}"
-      joint_limit_vel="${baboon_max_speed}"
-      joint_limit_effort="${baboon_peak_torque}"
+      joint_limit_vel="${joint_limits.get(joint_3_name, dict()).get('max_velocity', joint_3_limit_vel)}"
+      joint_limit_effort="${joint_limits.get(joint_3_name, dict()).get('max_effort', joint_3_limit_effort)}"
       joint_type="${joint_3_joint_type}">
       <origin xyz="${joint_3_origin_xyz}" rpy="${joint_3_origin_rpy}" />
@@ -140,6 +144,6 @@
       joint_lower_limit="${joint_4_lower_limit}"
       joint_upper_limit="${joint_4_upper_limit}"
-      joint_limit_vel="${baboon_max_speed}"
-      joint_limit_effort="${baboon_peak_torque}"
+      joint_limit_vel="${joint_limits.get(joint_4_name, dict()).get('max_velocity', joint_4_limit_vel)}"
+      joint_limit_effort="${joint_limits.get(joint_4_name, dict()).get('max_effort', joint_4_limit_effort)}"
       joint_type="${joint_4_joint_type}">
       <origin xyz="${joint_4_origin_xyz}" rpy="${joint_4_origin_rpy}" />
@@ -160,6 +164,6 @@
       joint_lower_limit="${joint_5_lower_limit}"
       joint_upper_limit="${joint_5_upper_limit}"
-      joint_limit_vel="${baboon_max_speed}"
-      joint_limit_effort="${baboon_peak_torque}"
+      joint_limit_vel="${joint_limits.get(joint_5_name, dict()).get('max_velocity', joint_5_limit_vel)}"
+      joint_limit_effort="${joint_limits.get(joint_5_name, dict()).get('max_effort', joint_5_limit_effort)}"
       joint_type="${joint_5_joint_type}">
       <origin xyz="${joint_5_origin_xyz}" rpy="${joint_5_origin_rpy}" />
@@ -188,6 +192,6 @@
       joint_lower_limit="${joint_6_lower_limit}"
       joint_upper_limit="${joint_6_upper_limit}"
-      joint_limit_vel="${baboon_max_speed}"
-      joint_limit_effort="${baboon_peak_torque}"
+      joint_limit_vel="${joint_limits.get(joint_6_name, dict()).get('max_velocity', joint_6_limit_vel)}"
+      joint_limit_effort="${joint_limits.get(joint_6_name, dict()).get('max_effort', joint_6_limit_effort)}"
       joint_type="${joint_6_joint_type}">
       <origin xyz="${joint_6_origin_xyz}" rpy="${joint_6_origin_rpy}" />

File: duatic_dynaarm_driver/urdf/dynaarm.urdf.xacro (robot description, xacro)
@@ -33,4 +33,5 @@
                          drive_parameter_folder:=''
                          version
+                         joint_limits_yaml:=''
                          *origin">
         <xacro:include filename="$(find duatic_dynaarm_description)/urdf/dynaarm.urdf.xacro" />
@@ -46,5 +47,6 @@
                 parent_link="${parent_link}"
                 collision="${collision}"
-                version="${version}">
+                version="${version}"
+                joint_limits_yaml="${joint_limits_yaml}">
             <xacro:insert_block name="origin" />
         </xacro:dynaarm_description>
