Commit message: refactor(description): remove unused dynaarm_link macro
No caller exists in this repo or any other Duatic repository; every
link uses dynaarm_link_w_collision instead. Rendered URDFs for both
versions and collision modes are byte-identical before and after.

File: duatic_dynaarm_description/urdf/common/dynaarm_common.urdf.xacro (robot description, xacro)
@@ -40,20 +40,4 @@
             <xacro:insert_block name="base_collision" />
             <xacro:insert_block name="base_inertia" />
-        </link>
-    </xacro:macro>
-    <!-- -->
-    <!-- DynaArm Link Macro -->
-    <!-- -->
-    <xacro:macro name="dynaarm_link"
-        params="link_name file_name **link_inertia">
-        <link name="${link_name}">
-            <visual>
-                <geometry>
-                    <mesh
-                        filename="package://duatic_dynaarm_description/meshes/${version}/${file_name}"
-                        scale="1.0 1.0 1.0" />
-                </geometry>
-            </visual>
-            <xacro:insert_block name="link_inertia" />
         </link>
     </xacro:macro>

Commit message: refactor(description): inline single-use macros and centralize limit overrides
dynaarm_main_body and dynaarm_tool were each called once, from
dynaarm_description, so their bodies now live there directly. The
joint_limits lookup was repeated for velocity and effort on every
revolute joint call; dynaarm_revolute_joint now applies it once and
callers pass only the defaults. Rendered URDFs are byte-identical,
both without a limits file and with one overriding velocity, effort,
and both.

File: duatic_dynaarm_description/urdf/common/dynaarm_common.urdf.xacro (robot description, xacro)
@@ -108,10 +108,14 @@
                 joint_type
                 *origin">
+        <!-- joint_limits overrides the default velocity and effort per joint -->
+        <xacro:property name="limits" value="${joint_limits.get(joint_name, dict())}" />
+        <xacro:property name="effort" value="${limits.get('max_effort', joint_limit_effort)}" />
+        <xacro:property name="velocity" value="${limits.get('max_velocity', joint_limit_vel)}" />
         <joint name="${joint_name}" type="${joint_type}">
             <parent link="${parent}" />
             <child link="${child}" />
             <axis xyz="${joint_axis_xyz}" />
-            <limit effort="${joint_limit_effort}" command_effort="${joint_limit_effort}"
-                current="10" gear_velocity="${joint_limit_vel}" velocity="${joint_limit_vel}"
+            <limit effort="${effort}" command_effort="${effort}"
+                current="10" gear_velocity="${velocity}" velocity="${velocity}"
                 lower="${joint_lower_limit}" upper="${joint_upper_limit}" />
             <!-- limit effort also defines torque limit and freeze controller gains -->

File: duatic_dynaarm_description/urdf/dynaarm.urdf.xacro (robot description, xacro)
@@ -39,12 +39,4 @@
       <xacro:insert_block name="origin" />
     </xacro:dynaarm_joint_fixed>
-    <!-- DynaArm-->
-    <xacro:dynaarm_main_body />
-    <xacro:dynaarm_tool />
-  </xacro:macro>
-  <!-- -->
-  <!-- DynaArm Main Body-->
-  <!-- -->
-  <xacro:macro name="dynaarm_main_body">
     <!-- Link: Base -->
     <xacro:dynaarm_baselink link_name="${base}" file_name="${base_mesh}">
@@ -72,6 +64,6 @@
       joint_lower_limit="${joint_1_lower_limit}"
       joint_upper_limit="${joint_1_upper_limit}"
-      joint_limit_vel="${joint_limits.get(joint_1_name, dict()).get('max_velocity', joint_1_limit_vel)}"
-      joint_limit_effort="${joint_limits.get(joint_1_name, dict()).get('max_effort', joint_1_limit_effort)}"
+      joint_limit_vel="${joint_1_limit_vel}"
+      joint_limit_effort="${joint_1_limit_effort}"
       joint_type="${joint_1_joint_type}">
       <origin xyz="${joint_1_origin_xyz}" rpy="${joint_1_origin_rpy}" />
@@ -93,6 +85,6 @@
       joint_lower_limit="${joint_2_lower_limit}"
       joint_upper_limit="${joint_2_upper_limit}"
-      joint_limit_vel="${joint_limits.get(joint_2_name, dict()).get('max_velocity', joint_2_limit_vel)}"
-      joint_limit_effort="${joint_limits.get(joint_2_name, dict()).get('max_effort', joint_2_limit_effort)}"
+      joint_limit_vel="${joint_2_limit_vel}"
+      joint_limit_effort="${joint_2_limit_effort}"
       joint_type="${joint_2_joint_type}">
       <origin xyz="${joint_2_origin_xyz}" rpy="${joint_2_origin_rpy}" />
@@ -114,6 +106,6 @@
       joint_lower_limit="${joint_3_lower_limit}"
       joint_upper_limit="${joint_3_upper_limit}"
-      joint_limit_vel="${joint_limits.get(joint_3_name, dict()).get('max_velocity', joint_3_limit_vel)}"
-      joint_limit_effort="${joint_limits.get(joint_3_name, dict()).get('max_effort', joint_3_limit_effort)}"
+      joint_limit_vel="${joint_3_limit_vel}"
+      joint_limit_effort="${joint_3_limit_effort}"
       joint_type="${joint_3_joint_type}">
       <origin xyz="${joint_3_origin_xyz}" rpy="${joint_3_origin_rpy}" />
@@ -142,6 +134,6 @@
       joint_lower_limit="${joint_4_lower_limit}"
       joint_upper_limit="${joint_4_upper_limit}"
-      joint_limit_vel="${joint_limits.get(joint_4_name, dict()).get('max_velocity', joint_4_limit_vel)}"
-      joint_limit_effort="${joint_limits.get(joint_4_name, dict()).get('max_effort', joint_4_limit_effort)}"
+      joint_limit_vel="${joint_4_limit_vel}"
+      joint_limit_effort="${joint_4_limit_effort}"
       joint_type="${joint_4_joint_type}">
       <origin xyz="${joint_4_origin_xyz}" rpy="${joint_4_origin_rpy}" />
@@ -162,6 +154,6 @@
       joint_lower_limit="${joint_5_lower_limit}"
       joint_upper_limit="${joint_5_upper_limit}"
-      joint_limit_vel="${joint_limits.get(joint_5_name, dict()).get('max_velocity', joint_5_limit_vel)}"
-      joint_limit_effort="${joint_limits.get(joint_5_name, dict()).get('max_effort', joint_5_limit_effort)}"
+      joint_limit_vel="${joint_5_limit_vel}"
+      joint_limit_effort="${joint_5_limit_effort}"
       joint_type="${joint_5_joint_type}">
       <origin xyz="${joint_5_origin_xyz}" rpy="${joint_5_origin_rpy}" />
@@ -190,20 +182,16 @@
       joint_lower_limit="${joint_6_lower_limit}"
       joint_upper_limit="${joint_6_upper_limit}"
-      joint_limit_vel="${joint_limits.get(joint_6_name, dict()).get('max_velocity', joint_6_limit_vel)}"
-      joint_limit_effort="${joint_limits.get(joint_6_name, dict()).get('max_effort', joint_6_limit_effort)}"
+      joint_limit_vel="${joint_6_limit_vel}"
+      joint_limit_effort="${joint_6_limit_effort}"
       joint_type="${joint_6_joint_type}">
       <origin xyz="${joint_6_origin_xyz}" rpy="${joint_6_origin_rpy}" />
     </xacro:dynaarm_revolute_joint>
-  </xacro:macro>
-  <!-- -->
-  <!-- DynaArm Tool-->
-  <!-- -->
-  <xacro:macro name="dynaarm_tool">
-      <xacro:virtual_link link_name="${end_effector}" />
-      <xacro:dynaarm_joint_fixed joint_name="${joint_ee_name}"
-          parent="${ee_parent}"
-          child="${end_effector}">
-          <origin xyz="${joint_ee_origin_xyz}" rpy="${joint_ee_origin_rpy}" />
-      </xacro:dynaarm_joint_fixed>
+    <!-- Link: Flange -->
+    <xacro:virtual_link link_name="${end_effector}" />
+    <xacro:dynaarm_joint_fixed joint_name="${joint_ee_name}"
+      parent="${ee_parent}"
+      child="${end_effector}">
+      <origin xyz="${joint_ee_origin_xyz}" rpy="${joint_ee_origin_rpy}" />
+    </xacro:dynaarm_joint_fixed>
   </xacro:macro>
 </robot>

Commit message: refactor(description): merge base and arm link macros into dynaarm_link
dynaarm_baselink and dynaarm_link_w_collision differed only in the
carbon fiber material on the base visual and in the order of the
inertial and collision elements. One dynaarm_link macro with a
carbon_fiber flag now builds every link. The rendered base link lists
inertial before collision; all URDFs are otherwise identical, and
equivalent once element order is ignored.

File: duatic_dynaarm_description/urdf/common/dynaarm_common.urdf.xacro (robot description, xacro)
@@ -23,8 +23,8 @@
 <robot xmlns:xacro="http://www.ros.org/wiki/xacro">
     <!-- -->
-    <!-- DynaArm Base Link Macro -->
+    <!-- DynaArm Link Macro -->
     <!-- -->
-    <xacro:macro name="dynaarm_baselink"
-        params="link_name file_name **base_inertia **base_collision">
+    <xacro:macro name="dynaarm_link"
+        params="link_name file_name carbon_fiber:=false **link_inertia **link_collision">
         <link name="${link_name}">
             <visual>
@@ -34,24 +34,9 @@
                         scale="1.0 1.0 1.0" />
                 </geometry>
-                <material name="carbon_fiber">
-                    <color rgba="0.792156862745098 0.819607843137255 0.933333333333333 1" />
-                </material>
-            </visual>
-            <xacro:insert_block name="base_collision" />
-            <xacro:insert_block name="base_inertia" />
-        </link>
-    </xacro:macro>
-    <!-- -->
-    <!-- DynaArm Link With Collision Macro -->
-    <!-- -->
-    <xacro:macro name="dynaarm_link_w_collision"
-        params="link_name file_name **link_inertia **link_collision">
-        <link name="${link_name}">
-            <visual>
-                <geometry>
-                    <mesh
-                        filename="package://duatic_dynaarm_description/meshes/${version}/${file_name}"
-                        scale="1.0 1.0 1.0" />
-                </geometry>
+                <xacro:if value="${carbon_fiber}">
+                    <material name="carbon_fiber">
+                        <color rgba="0.792156862745098 0.819607843137255 0.933333333333333 1" />
+                    </material>
+                </xacro:if>
             </visual>
             <xacro:insert_block name="link_inertia" />

File: duatic_dynaarm_description/urdf/dynaarm.urdf.xacro (robot description, xacro)
@@ -39,14 +39,14 @@
     </xacro:dynaarm_joint_fixed>
     <!-- Link: Base -->
-    <xacro:dynaarm_baselink link_name="${base}" file_name="${base_mesh}">
-      <base_inertia>
+    <xacro:dynaarm_link link_name="${base}" file_name="${base_mesh}" carbon_fiber="true">
+      <link_inertia>
         <xacro:insert_block name="base_inertial" />
-      </base_inertia>
-      <base_collision>
+      </link_inertia>
+      <link_collision>
         <xacro:insert_block name="base_collision" />
-      </base_collision>
-    </xacro:dynaarm_baselink>
+      </link_collision>
+    </xacro:dynaarm_link>
     <!-- Link: Shoulder -->
-    <xacro:dynaarm_link_w_collision link_name="${link01}" file_name="${link01_mesh}">
+    <xacro:dynaarm_link link_name="${link01}" file_name="${link01_mesh}">
       <link_inertia>
         <xacro:insert_block name="link01_inertial" />
@@ -55,5 +55,5 @@
         <xacro:insert_block name="link01_collision" />
       </link_collision>
-    </xacro:dynaarm_link_w_collision>
+    </xacro:dynaarm_link>
     <!-- Joint: Shoulder Rotation -->
     <xacro:dynaarm_revolute_joint joint_name="${joint_1_name}"
@@ -69,5 +69,5 @@
     </xacro:dynaarm_revolute_joint>
     <!-- Link: Upperarm -->
-    <xacro:dynaarm_link_w_collision link_name="${link02}" file_name="${link02_mesh}">
+    <xacro:dynaarm_link link_name="${link02}" file_name="${link02_mesh}">
       <link_inertia>
         <xacro:insert_block name="link02_inertial" />
@@ -76,5 +76,5 @@
         <xacro:insert_block name="link02_collision" />
       </link_collision>
-    </xacro:dynaarm_link_w_collision>
+    </xacro:dynaarm_link>
     <!-- Joint: Shoulder Flexion -->
     <xacro:dynaarm_revolute_joint joint_name="${joint_2_name}"
@@ -90,5 +90,5 @@
     </xacro:dynaarm_revolute_joint>
     <!-- Link: Elbow -->
-    <xacro:dynaarm_link_w_collision link_name="${link03}" file_name="${link03_mesh}">
+    <xacro:dynaarm_link link_name="${link03}" file_name="${link03_mesh}">
       <link_inertia>
         <xacro:insert_block name="link03_inertial" />
@@ -97,5 +97,5 @@
         <xacro:insert_block name="link03_collision" />
       </link_collision>
-    </xacro:dynaarm_link_w_collision>
+    </xacro:dynaarm_link>
     <!-- Joint: Elbow Flexion -->
     <xacro:dynaarm_revolute_joint joint_name="${joint_3_name}"
@@ -119,5 +119,5 @@
     </xacro:dynaarm_joint_fixed>
     <!-- Link: Forearm -->
-    <xacro:dynaarm_link_w_collision link_name="${link04}" file_name="${link04_mesh}">
+    <xacro:dynaarm_link link_name="${link04}" file_name="${link04_mesh}">
       <link_inertia>
         <xacro:insert_block name="link04_inertial" />
@@ -126,5 +126,5 @@
         <xacro:insert_block name="link04_collision" />
       </link_collision>
-    </xacro:dynaarm_link_w_collision>
+    </xacro:dynaarm_link>
     <!-- Joint: Forearm Rotation -->
     <xacro:dynaarm_revolute_joint joint_name="${joint_4_name}" parent="${link03}"
@@ -139,5 +139,5 @@
     </xacro:dynaarm_revolute_joint>
     <!-- Link: Wrist 1 -->
-    <xacro:dynaarm_link_w_collision link_name="${link05}" file_name="${link05_mesh}">
+    <xacro:dynaarm_link link_name="${link05}" file_name="${link05_mesh}">
       <link_inertia>
         <xacro:insert_block name="link05_inertial" />
@@ -146,5 +146,5 @@
         <xacro:insert_block name="link05_collision" />
       </link_collision>
-    </xacro:dynaarm_link_w_collision>
+    </xacro:dynaarm_link>
     <!-- Joint: Wrist Flexion -->
     <xacro:dynaarm_revolute_joint joint_name="${joint_5_name}" parent="${link04}"
@@ -167,5 +167,5 @@
     </xacro:dynaarm_joint_fixed>
     <!-- Link: Wrist 2 -->
-    <xacro:dynaarm_link_w_collision link_name="${link06}" file_name="${link06_mesh}">
+    <xacro:dynaarm_link link_name="${link06}" file_name="${link06_mesh}">
       <link_inertia>
         <xacro:insert_block name="link06_inertial" />
@@ -174,5 +174,5 @@
         <xacro:insert_block name="link06_collision" />
       </link_collision>
-    </xacro:dynaarm_link_w_collision>
+    </xacro:dynaarm_link>
     <!-- Joint: Wrist Rotation -->
     <xacro:dynaarm_revolute_joint joint_name="${joint_6_name}" parent="${link05}"

Commit message: refactor(description): drop default mesh scale attributes
The link meshes set scale to 1 1 1, which is the URDF default, spelled
two different ways in the same macro. The rendered URDFs differ from
the previous commit only by the removed scale attributes.

File: duatic_dynaarm_description/urdf/common/dynaarm_common.urdf.xacro (robot description, xacro)
@@ -30,7 +30,5 @@
             <visual>
                 <geometry>
-                    <mesh
-                        filename="package://duatic_dynaarm_description/meshes/${version}/${file_name}"
-                        scale="1.0 1.0 1.0" />
+                    <mesh filename="package://duatic_dynaarm_description/meshes/${version}/${file_name}" />
                 </geometry>
                 <xacro:if value="${carbon_fiber}">
@@ -48,7 +46,5 @@
                     <origin xyz="0 0 0" rpy="0 0 0" />
                     <geometry>
-                        <mesh
-                            filename="package://duatic_dynaarm_description/meshes/${version}/${file_name}"
-                            scale="1 1 1" />
+                        <mesh filename="package://duatic_dynaarm_description/meshes/${version}/${file_name}" />
                     </geometry>
                 </collision>

Commit message: refactor(description): drop the limit element from fixed joints
URDF only defines joint limits for revolute and prismatic joints. The
effort=2000 velocity=0 limit on the base, camera mount and flange joints
was never read: ros2_control and the DuaDrive interface only take limits
for the joints listed in ros2_control, which are the six revolute ones.
The mock bringup loads the same controllers and logs the same per-joint
limits with and without it.

File: duatic_dynaarm_description/urdf/common/dynaarm_common.urdf.xacro (robot description, xacro)
@@ -118,5 +118,4 @@
             <parent link="${parent}" />
             <child link="${child}" />
-            <limit effort="2000" velocity="0" lower="0" upper="0" />
             <xacro:insert_block name="origin" />
         </joint>

Commit message: refactor(description): drop the carbon_fiber option from dynaarm_link
Only the base link set carbon_fiber, and the tinted material it added
is no longer wanted. Removing the parameter leaves dynaarm_link with no
conditional visual, and no link in the generated URDF carries a
material anymore.

File: duatic_dynaarm_description/urdf/common/dynaarm_common.urdf.xacro (robot description, xacro)
@@ -26,5 +26,5 @@
     <!-- -->
     <xacro:macro name="dynaarm_link"
-        params="link_name file_name carbon_fiber:=false **link_inertia **link_collision">
+        params="link_name file_name **link_inertia **link_collision">
         <link name="${link_name}">
             <visual>
@@ -32,9 +32,4 @@
                     <mesh filename="package://duatic_dynaarm_description/meshes/${version}/${file_name}" />
                 </geometry>
-                <xacro:if value="${carbon_fiber}">
-                    <material name="carbon_fiber">
-                        <color rgba="0.792156862745098 0.819607843137255 0.933333333333333 1" />
-                    </material>
-                </xacro:if>
             </visual>
             <xacro:insert_block name="link_inertia" />

File: duatic_dynaarm_description/urdf/dynaarm.urdf.xacro (robot description, xacro)
@@ -39,5 +39,5 @@
     </xacro:dynaarm_joint_fixed>
     <!-- Link: Base -->
-    <xacro:dynaarm_link link_name="${base}" file_name="${base_mesh}" carbon_fiber="true">
+    <xacro:dynaarm_link link_name="${base}" file_name="${base_mesh}">
       <link_inertia>
         <xacro:insert_block name="base_inertial" />

Commit message: refactor(description): drop unused elements from the DynaArm model (#50)

File: duatic_dynaarm_description/urdf/common/dynaarm_common.urdf.xacro (robot description, xacro)
@@ -94,5 +94,4 @@
                 joint_limit_vel
                 joint_limit_effort
-                joint_type
                 *origin">
         <!-- joint_limits overrides the default velocity and effort per joint -->
@@ -100,5 +99,5 @@
         <xacro:property name="effort" value="${limits.get('max_effort', joint_limit_effort)}" />
         <xacro:property name="velocity" value="${limits.get('max_velocity', joint_limit_vel)}" />
-        <joint name="${joint_name}" type="${joint_type}">
+        <joint name="${joint_name}" type="revolute">
             <parent link="${parent}" />
             <child link="${child}" />
@@ -119,5 +118,4 @@
             <parent link="${parent}" />
             <child link="${child}" />
-            <limit effort="2000" velocity="0" lower="0" upper="0" />
             <xacro:insert_block name="origin" />
         </joint>
